File: sa800u-baseboard-hw/HDMI.sch (KiCad schematic (older format))
At the start: 0 parts

Commit message: added HDMI converter
Parts:
- added C?: C_1u_0402, antmicro-footprints:0402-cap, symbol antmicroCapacitors0402:C_1u_0402
- added C? (x2): C_10p_0402, antmicro-footprints:0402-cap, symbol antmicroCapacitors0402:C_10p_0402
- added R?: R_10k_0603, antmicro-footprints:0603-res, symbol antmicroResistors0603:R_10k_0603
- added R? (x3): R_4k7_0402, antmicro-footprints:0402-res, symbol antmicroResistors0402:R_4k7_0402
- added R?: R_1k_0402, antmicro-footprints:0402-res, symbol antmicroResistors0402:R_1k_0402
- added R? (x2): R_0R_0402, antmicro-footprints:0402-res, symbol antmicroResistors0402:R_0R_0402
- added R? (x2): R_2k2_0402, antmicro-footprints:0402-res, symbol antmicroResistors0402:R_2k2_0402
- added R?: R_20k_0402, antmicro-footprints:0402-res, symbol antmicroResistors0402:R_20k_0402
- added R?: R_7k68_0603, antmicro-footprints:0603-res, symbol antmicroResistors0603:R_7k68_0603
- added R?: R_1M0_0402, antmicro-footprints:0402-res, symbol antmicroResistors0402:R_1M0_0402
- added U?: LT9611, symbol HDMI:LT9611
- added Y?: ECS-1618-250-BN-TR, symbol Oscillators:ECS-1618-250-BN-TR
Connections:
- new net: R?.1, R?.1, U?.35 (HTX_HPD)
- new net: C?.1, R?.2, U?.49 (XTALI), Y?.4 (VDD)
- new net: C?.1, R?.1, U?.50 (XTALO), Y?.3 (OUT)
- new net: R?.2, U?.52 (REXT)
- new net +1V8: Y?.1 (EN)
- new net +5V: R?.1, R?.1
- new net CEC_GPIO6: U?.24 (CEC_GPIO6)
- new net DETECT_HDMI: R?.2
- new net DSI1_CLK_N: U?.9 (MC_N0)
- new net DSI1_CLK_P: U?.10 (MC_P0)
- new net DSI1_LN0_N: U?.13 (M0_N0)
- new net DSI1_LN1_N: U?.11 (M1_N0)
- new net DSI1_LN1_P: U?.12 (M1_P0), U?.14 (M0_P0)
- new net DSI1_LN2_N: U?.7 (M2_N0)
- new net DSI1_LN2_P: U?.8 (M2_P0)
- new net DSI1_LN3_N: U?.5 (M3_N0)
- new net DSI1_LN3_P: U?.6 (M3_P0)
- new net GND: C?.2, C?.2, C?.2, R?.1, R?.2, R?.2, U?.65 (GND), Y?.2 (GND)
- new net HDMIOUT_SCL: R?.2, U?.18 (CSCL_GPIO10)
- new net HDMIOUT_SDA: R?.2, U?.19 (CSDA_GPIO11)
- new net I2C_ADDR: R?.1, R?.2, U?.25 (I2C_ADDR)
- new net I2S_D0_SPDIF: U?.30 (I2S_D0_SPDIF)
- new net I2S_MCLK: U?.29 (I2S_MCLK_GPIO9)
- new net I2S_SCLK: U?.28 (I2S_SCLK_GPIO8)
- new net I2S_WS: U?.27 (I2S_WS_GPIO7)
- new net INTO_GPIO5: R?.2, U?.23 (INTIO_GPIO5)
- new net LKT9611_VDD12: U?.53 (VCC12_SYSPLL), U?.54 (VDD)
- new net LT9611VCC12_RX: U?.56 (VCC12_MRX23)
- new net LT9611_VCC12_RX: U?.4 (VCC12_MRX01)
- new net LT9611_VCC12_TX: U?.44 (VCC12_HTX)
- new net LT9611_VCC33_IO: U?.26 (VC33_IO), U?.34 (VCC33_IO)
- new net LT9611_VCC33_RX: U?.3 (VCC33_MRX01), U?.55 (VCC33_MRX23)
- new net LT9611_VCC33_TX: U?.43 (VCC33_HTX)
- new net LT9611_VCC_RX: U?.51 (VCC33_BG)
- new net LT9611_VDD12: U?.15 (VDD1), U?.16 (VDD2), U?.31 (VDD3)
- new net RST_N: C?.1, R?.2, U?.17 (RST_N)
- new net SCL_HDMI: R?.2, U?.37 (HTX_DSCL)
- new net SDA_HDMI: R?.2, U?.36 (HTX_DSDA)
- new net TX_CLKM: U?.38 (HTX_C-)
- new net TX_CLKP: U?.39 (HTX_C+)
- new net TX_D0M: U?.40 (HTX_D0-)
- new net TX_D0P: U?.41 (HTX_D0+)
- new net TX_D1M: U?.45 (HTX_D1-)
- new net TX_D1P: U?.46 (HTX_D1+)
- new net TX_D2M: U?.47 (HTX_D2-)
- new net TX_D2P: U?.48 (HTX_D2+)
- new net VCOM: U?.42 (VCOM)
- new net VDD33: R?.1, R?.1, R?.1, R?.1, R?.1
- no-connect marks 0 -> 11
Other:
- note added: "Why is this 1M resistor here? \n"
