File: sa800u-baseboard-hw/LCM.sch (KiCad schematic (older format))
At the start: 14 parts, among them J2 FFC-1mm-20pin, U3 FFC-1mm-30pin

Commit message: Review - Add geeral remarks
Other:
- note added: "REMARK:These pull-ups are doubled"
Changed lines of the file:
@@
 Wire Wire Line
 	5600 2550 7100 2550
+Text Notes 2950 3025 0    50   ~ 0
+REMARK:These pull-ups are doubled
+Wire Notes Line
+	4425 3000 5275 3000
+Wire Notes Line
+	2875 3000 2400 3000
+Wire Notes Line
+	2400 3000 2400 2400
+Wire Notes Line
+	2400 2400 2275 2400
 $EndSCHEMATC

Commit message: fixed doubled pullups for I2C in DSI, changed connectors antmicro lib connectors
Parts:
- removed J2: FFC-1mm-20pin, symbol Connectors:FFC-1mm-20pin
- removed U3: FFC-1mm-30pin, symbol Connectors:FFC-1mm-30pin
- added J?: 3-84952-0, symbol antmicroFCCConnectors:3-84952-0
- added J?: 68612014122, antmicro-footprints:68612014122, symbol antmicroFCCConnectors:68612014122
Connections:
- wire segments 109 -> 110
- no-connect marks 0 -> 15
Other:
- note added: "Compatible with generic raspberry pi LCDs."
- note added: "General purpose DSI for LCD"
- note added: "Is this connector right? 30 instead of 15?\n"
- note removed: "REMARK:These pull-ups are doubled"
- moved on the sheet: L1, L2, L3, L4, L5, L6, L7, L8, R28, R29, R30, R31
