File: sa800u-baseboard-hw/Ethernet Controller.sch (KiCad schematic (older format))
At the start: 33 parts, among them T1 749020010A, U1 RTL8111H, Y1 ECS-1618-250-BN-TR

Commit message: Review - Add geeral remarks
Other:
- note added: "REMARK: Add components to our repository \n(antmicro-kicad-components)"
- note added: "REMARK: Please use _P _N at the end of the labels \n(eg. LAN0_RJ45_D1P -->LAN0_RJ45_D1_P)"
- note added: "REMARK: Please, fill the background \nof the symbol"
- note added: "REMARK: This GND's should be isolated. \nUse EARTH symbol instead of GND at HV side."
Changed lines of the file:
@@
 Wire Wire Line
 	6000 6400 7500 6400
+Text Notes 875  5250 0    50   ~ 0
+REMARK: Add components to our repository \n(antmicro-kicad-components)
+Text Notes 5750 925  0    50   ~ 0
+REMARK: Please use _P _N at the end of the labels \n(eg. LAN0_RJ45_D1P -->LAN0_RJ45_D1_P)
+Text Notes 6200 3300 0    50   ~ 0
+REMARK: This GND's should be isolated. \nUse EARTH symbol instead of GND at HV side.
+Wire Notes Line
+	5425 4300 6750 4300
+Wire Notes Line
+	6750 4300 6750 3350
+Wire Notes Line
+	6750 3350 6775 3350
+Wire Notes Line
+	7650 3075 7650 2900
+Wire Notes Line
+	6800 3000 6800 2350
+Wire Notes Line
+	6800 2350 6825 2350
+Text Notes 575  5500 0    50   ~ 0
+REMARK: Please, fill the background \nof the symbol
 $EndSCHEMATC

Commit message: fixed doubled pullups for I2C in DSI, changed connectors antmicro lib connectors
Connections:
- net labels added: Earth
- wire segments 136 -> 139
Changed lines of the file:
@@
 	8200 2650 8200 2400
-Wire Wire Line
-	7050 2650 7650 2650
 Wire Wire Line
 	7050 2400 7050 2650
 Text GLabel 6850 2150 0    50   Input ~ 0
 3V3
-$Comp
-L power:GND #PWR0105
-U 1 1 6199FB11
-P 6900 2250
-F 0 "#PWR0105" H 6900 2000 50  0001 C CNN
-F 1 "GND" V 6905 2122 50  0000 R CNN
-F 2 "" H 6900 2250 50  0001 C CNN
-F 3 "" H 6900 2250 50  0001 C CNN
-	1    6900 2250
-	0    1    1    0
-$EndComp
 Text Label 9850 1950 0    50   ~ 0
 ETH_LED2
@@
 	-1   0    0    1
 $EndComp
-$Comp
-L power:GND #PWR0111
-U 1 1 61BDF244
-P 5200 4200
-F 0 "#PWR0111" H 5200 3950 50  0001 C CNN
-F 1 "GND" H 5205 4027 50  0000 C CNN
-F 2 "" H 5200 4200 50  0001 C CNN
-F 3 "" H 5200 4200 50  0001 C CNN
-	1    5200 4200
-	1    0    0    -1
-$EndComp
 Wire Wire Line
 	8750 1950 9850 1950
@@
 Wire Wire Line
 	2050 1500 2800 1500
-$Comp
-L power:GND #PWR01
-U 1 1 61C6A237
-P 7650 2650
-F 0 "#PWR01" H 7650 2400 50  0001 C CNN
-F 1 "GND" H 7655 2477 50  0000 C CNN
-F 2 "" H 7650 2650 50  0001 C CNN
-F 3 "" H 7650 2650 50  0001 C CNN
-	1    7650 2650
-	1    0    0    -1
-$EndComp
-Connection ~ 7650 2650
-Wire Wire Line
-	7650 2650 8200 2650
 $Comp
 L power:GND #PWR02
@@
 Text Notes 575  5500 0    50   ~ 0
 REMARK: Please, fill the background \nof the symbol
+$Comp
+L power:Earth #PWR?
+U 1 1 619F1D72
+P 5200 4300
+F 0 "#PWR?" H 5200 4050 50  0001 C CNN
+F 1 "Earth" H 5200 4150 50  0001 C CNN
+F 2 "" H 5200 4300 50  0001 C CNN
+F 3 "~" H 5200 4300 50  0001 C CNN
+	1    5200 4300
+	1    0    0    -1
+$EndComp
+$Comp
+L power:Earth #PWR?
+U 1 1 619F2B63
+P 6900 2350
+F 0 "#PWR?" H 6900 2100 50  0001 C CNN
+F 1 "Earth" H 6900 2200 50  0001 C CNN
+F 2 "" H 6900 2350 50  0001 C CNN
+F 3 "~" H 6900 2350 50  0001 C CNN
+	1    6900 2350
+	1    0    0    -1
+$EndComp
+$Comp
+L power:Earth #PWR?
+U 1 1 619F3D25
+P 7650 2700
+F 0 "#PWR?" H 7650 2450 50  0001 C CNN
+F 1 "Earth" H 7650 2550 50  0001 C CNN
+F 2 "" H 7650 2700 50  0001 C CNN
+F 3 "~" H 7650 2700 50  0001 C CNN
+	1    7650 2700
+	1    0    0    -1
+$EndComp
+Wire Wire Line
+	7050 2650 7650 2650
+Wire Wire Line
+	7650 2700 7650 2650
+Connection ~ 7650 2650
+Wire Wire Line
+	7650 2650 8200 2650
+Wire Wire Line
+	6900 2250 6900 2350
+Wire Wire Line
+	5200 4200 5200 4300
 $EndSCHEMATC

Commit message: fixed ethernet controller symbol
Other:
- note removed: "REMARK: This GND's should be isolated. \nUse EARTH symbol instead of GND at HV side."
Changed lines of the file:
@@
 Text Notes 5750 925  0    50   ~ 0
 REMARK: Please use _P _N at the end of the labels \n(eg. LAN0_RJ45_D1P -->LAN0_RJ45_D1_P)
-Text Notes 6200 3300 0    50   ~ 0
-REMARK: This GND's should be isolated. \nUse EARTH symbol instead of GND at HV side.
-Wire Notes Line
-	5425 4300 6750 4300
-Wire Notes Line
-	6750 4300 6750 3350
-Wire Notes Line
-	6750 3350 6775 3350
-Wire Notes Line
-	7650 3075 7650 2900
-Wire Notes Line
-	6800 3000 6800 2350
-Wire Notes Line
-	6800 2350 6825 2350
 Text Notes 575  5500 0    50   ~ 0
 REMARK: Please, fill the background \nof the symbol

Commit message: fixed labels for differential pairs
Connections:
- net labels added: LAN0_MDI0_N, LAN0_MDI0_P, LAN0_MDI1_N, LAN0_MDI1_P, LAN0_MDI2_N, LAN0_MDI2_P, LAN0_MDI3_N, LAN0_MDI3_P, LAN0_RJ45_D1_N, LAN0_RJ45_D1_P, LAN0_RJ45_D2_N, LAN0_RJ45_D2_P, LAN0_RJ45_D3_N, LAN0_RJ45_D3_P, LAN0_RJ45_D4_N, LAN0_RJ45_D4_P, PCIE1_REFCLK_N, PCIE1_RX_N, PCIE1_TX_N
- net labels removed: LAN0_MDI0N, LAN0_MDI0P, LAN0_MDI1N, LAN0_MDI1P, LAN0_MDI2N, LAN0_MDI2P, LAN0_MDI3N, LAN0_MDI3P, LAN0_RJ45_D1M, LAN0_RJ45_D1P, LAN0_RJ45_D2M, LAN0_RJ45_D2P, LAN0_RJ45_D3M, LAN0_RJ45_D3P, LAN0_RJ45_D4M, LAN0_RJ45_D4P, PCIE1_REFCLK_M, PCIE1_RX_M, PCIE1_TX_M
Other:
- note removed: "REMARK: Add components to our repository \n(antmicro-kicad-components)"
- note removed: "REMARK: Please, fill the background \nof the symbol"
Changed lines of the file:
@@
 	-1   0    0    -1
 $EndComp
-Text Label 2050 1100 0    50   ~ 0
-LAN0_MDI0P
 Text Label 2050 1300 0    50   ~ 0
-LAN0_MDI0N
+LAN0_MDI0_N
 Text Label 2050 1500 0    50   ~ 0
-LAN0_MDI1P
+LAN0_MDI1_P
 Text Label 2050 1700 0    50   ~ 0
-LAN0_MDI1N
+LAN0_MDI1_N
 Text Label 2050 1900 0    50   ~ 0
-LAN0_MDI2P
+LAN0_MDI2_P
 Text Label 2050 2100 0    50   ~ 0
-LAN0_MDI2N
+LAN0_MDI2_N
 Text Label 2050 2300 0    50   ~ 0
-LAN0_MDI3P
+LAN0_MDI3_P
 Text Label 2050 2500 0    50   ~ 0
-LAN0_MDI3N
+LAN0_MDI3_N
 Text Label 3750 2500 0    50   ~ 0
-LAN0_RJ45_D4M
+LAN0_RJ45_D4_N
 Wire Wire Line
 	3650 2500 3750 2500
 Text Label 3750 2300 0    50   ~ 0
-LAN0_RJ45_D4P
+LAN0_RJ45_D4_P
 Text Label 3750 2100 0    50   ~ 0
-LAN0_RJ45_D3M
+LAN0_RJ45_D3_N
 Text Label 3750 1900 0    50   ~ 0
-LAN0_RJ45_D3P
+LAN0_RJ45_D3_P
 Text Label 3750 1700 0    50   ~ 0
-LAN0_RJ45_D2M
+LAN0_RJ45_D2_N
 Text Label 3750 1500 0    50   ~ 0
-LAN0_RJ45_D2P
-Text Label 3750 1300 0    50   ~ 0
-LAN0_RJ45_D1M
+LAN0_RJ45_D2_P
 Text Label 3750 1100 0    50   ~ 0
-LAN0_RJ45_D1P
+LAN0_RJ45_D1_P
 Wire Wire Line
 	3650 2300 3750 2300
@@
 PCIE1_RST_N
 Text Label 4550 6500 3    50   ~ 0
-PCIE1_RX_M
+PCIE1_RX_N
 Text Label 4300 6500 3    50   ~ 0
 PCIE1_RX_P
@@
 1V0A
 Text Label 2000 6100 0    50   ~ 0
-LAN0_MDI2N
+LAN0_MDI2_N
 Text Label 2000 6000 0    50   ~ 0
-LAN0_MDI2P
+LAN0_MDI2_P
 Text Label 2000 5900 0    50   ~ 0
-LAN0_MDI1N
+LAN0_MDI1_N
 Text Label 2000 5800 0    50   ~ 0
-LAN0_MDI1P
+LAN0_MDI1_P
 Wire Wire Line
 	2500 6100 2000 6100
@@
 	2500 6000 2000 6000
 Text Label 2000 5600 0    50   ~ 0
-LAN0_MDI0N
+LAN0_MDI0_N
 Wire Wire Line
 	2500 5900 2000 5900
@@
 	2000 5500 2500 5500
 Text Label 2000 5500 0    50   ~ 0
-LAN0_MDI0P
+LAN0_MDI0_P
 Wire Wire Line
 	3000 6700 3000 7400
@@
 	3700 6700 3700 7400
 Text Label 3700 7400 1    50   ~ 0
-PCIE1_REFCLK_M
+PCIE1_REFCLK_N
 Wire Wire Line
 	3600 6700 3600 7400
@@
 PCIE1_REFCLK_P
 Text Label 3500 7400 1    50   ~ 0
-PCIE1_TX_M
+PCIE1_TX_N
 Text Label 3400 7400 1    50   ~ 0
 PCIE1_TX_P
@@
 3V3
 Text Label 3100 7400 1    50   ~ 0
-LAN0_MDI3N
+LAN0_MDI3_N
 Text Label 3000 7400 1    50   ~ 0
-LAN0_MDI3P
+LAN0_MDI3_P
 $Comp
 L RTL8111Hx:RTL8111H U1
@@
 	7000 1450 6350 1450
 Text Label 6350 2050 0    50   ~ 0
-LAN0_RJ45_D4M
+LAN0_RJ45_D4_N
 Text Label 6350 1950 0    50   ~ 0
-LAN0_RJ45_D4P
+LAN0_RJ45_D4_P
 Text Label 6350 1850 0    50   ~ 0
-LAN0_RJ45_D3M
+LAN0_RJ45_D3_N
 Text Label 6350 1750 0    50   ~ 0
-LAN0_RJ45_D3P
+LAN0_RJ45_D3_P
 Text Label 6350 1650 0    50   ~ 0
-LAN0_RJ45_D2M
+LAN0_RJ45_D2_N
 Text Label 6350 1550 0    50   ~ 0
-LAN0_RJ45_D2P
+LAN0_RJ45_D2_P
 Text Label 6350 1450 0    50   ~ 0
-LAN0_RJ45_D1M
+LAN0_RJ45_D1_N
 Wire Wire Line
 	7000 1350 6350 1350
 Text Label 6350 1350 0    50   ~ 0
-LAN0_RJ45_D1P
+LAN0_RJ45_D1_P
 $Comp
 L antmicroModularConnectorsJacksWithMagnetics:WE-RJ45_7499111121A J?1
@@
 Wire Wire Line
 	6000 6400 7500 6400
-Text Notes 875  5250 0    50   ~ 0
-REMARK: Add components to our repository \n(antmicro-kicad-components)
 Text Notes 5750 925  0    50   ~ 0
 REMARK: Please use _P _N at the end of the labels \n(eg. LAN0_RJ45_D1P -->LAN0_RJ45_D1_P)
-Text Notes 575  5500 0    50   ~ 0
-REMARK: Please, fill the background \nof the symbol
 $Comp
 L power:Earth #PWR?
@@
 Wire Wire Line
 	5200 4200 5200 4300
+Text Label 3750 1300 0    50   ~ 0
+LAN0_RJ45_D1_N
+Text Label 2050 1100 0    50   ~ 0
+LAN0_MDI0_P
 $EndSCHEMATC

Commit message: fixed part of labels
Other:
- note removed: "REMARK: Please use _P _N at the end of the labels \n(eg. LAN0_RJ45_D1P -->LAN0_RJ45_D1_P)"
Changed lines of the file:
@@
 Text Label 4300 5500 0    50   ~ 0
 REG_1V0
-Text Label 4300 5800 0    50   ~ 0
-PCIE1_WAKE_N
 Wire Wire Line
 	4200 5800 4300 5800
-Text Label 4300 5900 0    50   ~ 0
-ETH_ISOLATEB
 Wire Wire Line
 	4200 5900 4300 5900
@@
 Wire Wire Line
 	4200 6200 4300 6200
-Text Label 4300 6000 0    50   ~ 0
-PCIE1_RST_N
-Text Label 4550 6500 3    50   ~ 0
-PCIE1_RX_N
-Text Label 4300 6500 3    50   ~ 0
-PCIE1_RX_P
 Text GLabel 1750 5700 0    50   Input ~ 0
 1V0A
@@
 Wire Wire Line
 	3700 6700 3700 7400
-Text Label 3700 7400 1    50   ~ 0
-PCIE1_REFCLK_N
 Wire Wire Line
 	3600 6700 3600 7400
-Text Label 3600 7400 1    50   ~ 0
-PCIE1_REFCLK_P
-Text Label 3500 7400 1    50   ~ 0
-PCIE1_TX_N
-Text Label 3400 7400 1    50   ~ 0
-PCIE1_TX_P
 Wire Wire Line
 	3300 6700 3300 7400
 Wire Wire Line
 	3200 6700 3200 7450
-Text Label 3300 7400 1    50   ~ 0
-PCIE1_CLKREQ_N
 Text GLabel 3200 7450 3    50   Input ~ 0
 3V3
@@
 	1    0    0    -1
 $EndComp
-Text Label 6000 6250 0    50   ~ 0
-PCIE1_CLKREQ_N
-Text Label 6000 6400 0    50   ~ 0
-ETH_ISOLATEB
-Text Label 6000 6100 0    50   ~ 0
-PCIE1_RST_N
-Text Label 6000 5950 0    50   ~ 0
-PCIE1_WAKE_N
 Wire Wire Line
 	6000 5950 6550 5950
@@
 Wire Wire Line
 	6000 6400 7500 6400
-Text Notes 5750 925  0    50   ~ 0
-REMARK: Please use _P _N at the end of the labels \n(eg. LAN0_RJ45_D1P -->LAN0_RJ45_D1_P)
 $Comp
 L power:Earth #PWR?
@@
 Text Label 2050 1100 0    50   ~ 0
 LAN0_MDI0_P
+Text GLabel 3300 7400 3    50   Input ~ 0
+PCIE1_CLKREQ_N
+Text GLabel 3400 7400 3    50   Input ~ 0
+PCIE1_TX_P
+Text GLabel 3500 7400 3    50   Input ~ 0
+PCIE1_TX_N
+Text GLabel 3600 7400 3    50   Input ~ 0
+PCIE1_REFCLK_P
+Text GLabel 3700 7400 3    50   Input ~ 0
+PCIE1_REFCLK_N
+Text GLabel 4300 6500 3    50   Input ~ 0
+PCIE1_RX_P
+Text GLabel 4550 6500 3    50   Input ~ 0
+PCIE1_RX_N
+Text GLabel 4300 6000 2    50   Input ~ 0
+PCIE1_RST_N
+Text GLabel 4300 5900 2    50   Input ~ 0
+ETH_ISOLATEB
+Text GLabel 4300 5800 2    50   Input ~ 0
+PCIE1_WAKE_N
+Text GLabel 6000 6400 0    50   Input ~ 0
+ETH_ISOLATEB
+Text GLabel 6000 6250 0    50   Input ~ 0
+PCIE1_CLKREQ_N
+Text GLabel 6000 6100 0    50   Input ~ 0
+PCIE1_RST_N
+Text GLabel 6000 5950 0    50   Input ~ 0
+PCIE1_WAKE_N
 $EndSCHEMATC

Commit message: introducing minor genreal improvements
Parts:
- removed R15: R_2k49_0402, antmicro-footprints:0402-res, symbol antmicroResistors0402:R_2k49_0402
- removed Y1: ECS-1618-250-BN-TR, symbol Oscillators:ECS-1618-250-BN-TR
- added R?: R_2k49_1%_0402, antmicro-footprints:0402-res, symbol antmicroResistors0402:R_2k49_1%_0402
- added Y?: ECS-1618-250-BN-TR, antmicro-footprints:OSC_ECS-1618-250-BN-TR, symbol antmicroOscillators:ECS-1618-250-BN-TR
Other:
- note added: "Review Oscillator connection."
- moved on the sheet: C7, C8, R19
Changed lines of the file:
@@
 	3000 4650 2750 4650
-$Comp
-L antmicroResistors0402:R_2k49_0402 R15
-U 1 1 618F9273
-P 3200 4850
-F 0 "R15" V 2950 4800 60  0000 L CNN
-F 1 "R_2k49_0402" H 3200 4700 60  0001 C CNN
-F 2 "antmicro-footprints:0402-res" H 3400 5050 60  0001 L CNN
-F 3 "" H 3200 4850 50  0001 C CNN
-F 4 "YAGEO" H 3400 5250 60  0001 L CNN "Manufacturer"
-F 5 "RC0402FR-132K49L" H 3400 5150 60  0001 L CNN "MPN"
-F 6 "2k49" V 2850 4750 50  0000 L CNN "Val"
-	1    3200 4850
-	0    1    1    0
-$EndComp
 $Comp
 L power:GND #PWR0101
@@
 Text Notes 1600 950  0    50   ~ 0
 Choke is on secondary side.\n(Where only data is passed through)
-$Comp
-L Oscillators:ECS-1618-250-BN-TR Y1
-U 1 1 61995322
-P 8000 4500
-F 0 "Y1" H 8250 4665 50  0000 C CNN
-F 1 "ECS-1618-250-BN-TR" H 8250 4574 50  0000 C CNN
-F 2 "" H 8200 4550 50  0001 C CNN
-F 3 "" H 8200 4550 50  0001 C CNN
-	1    8000 4500
-	1    0    0    -1
-$EndComp
-Wire Wire Line
-	7900 4600 7450 4600
-Wire Wire Line
-	7450 4600 7450 4450
+Wire Wire Line
+	6800 4600 6350 4600
+Wire Wire Line
+	6350 4600 6350 4450
 $Comp
 L power:+1V8 #PWR04
 U 1 1 61999203
-P 7450 4450
-F 0 "#PWR04" H 7450 4300 50  0001 C CNN
-F 1 "+1V8" H 7465 4623 50  0000 C CNN
-F 2 "" H 7450 4450 50  0001 C CNN
-F 3 "" H 7450 4450 50  0001 C CNN
-	1    7450 4450
-	1    0    0    -1
-$EndComp
-Wire Wire Line
-	7900 4700 7450 4700
-Wire Wire Line
-	7450 4700 7450 4850
+P 6350 4450
+F 0 "#PWR04" H 6350 4300 50  0001 C CNN
+F 1 "+1V8" H 6365 4623 50  0000 C CNN
+F 2 "" H 6350 4450 50  0001 C CNN
+F 3 "" H 6350 4450 50  0001 C CNN
+	1    6350 4450
+	1    0    0    -1
+$EndComp
+Wire Wire Line
+	8400 4800 8400 4950
 $Comp
 L power:GND #PWR05
 U 1 1 6199D143
-P 7450 4850
-F 0 "#PWR05" H 7450 4600 50  0001 C CNN
-F 1 "GND" H 7455 4677 50  0000 C CNN
-F 2 "" H 7450 4850 50  0001 C CNN
-F 3 "" H 7450 4850 50  0001 C CNN
-	1    7450 4850
-	1    0    0    -1
-$EndComp
-Wire Wire Line
-	8600 4700 8850 4700
-Wire Wire Line
-	8850 4700 8850 4800
-$Comp
-L antmicroCapacitors0402:C_10p_0402 C7
-U 1 1 619A5032
-P 8850 5000
-F 0 "C7" H 8965 5045 60  0000 L CNN
-F 1 "C_10p_0402" H 8850 4850 60  0001 C CNN
-F 2 "antmicro-footprints:0402-cap" H 9050 5200 60  0001 L CNN
-F 3 "" H 8850 5000 50  0001 C CNN
-F 4 "MULTICOMP" H 9050 5400 60  0001 L CNN "Manufacturer"
-F 5 "MC0402N100D500CT" H 9050 5300 60  0001 L CNN "MPN"
-F 6 "10p" H 8965 4947 50  0000 L CNN "Val"
-	1    8850 5000
-	1    0    0    -1
-$EndComp
-$Comp
-L power:GND #PWR011
-U 1 1 619A53C6
-P 8850 5150
-F 0 "#PWR011" H 8850 4900 50  0001 C CNN
-F 1 "GND" H 8855 4977 50  0000 C CNN
-F 2 "" H 8850 5150 50  0001 C CNN
-F 3 "" H 8850 5150 50  0001 C CNN
-	1    8850 5150
-	1    0    0    -1
-$EndComp
-Wire Wire Line
-	8600 4600 9400 4600
-Wire Wire Line
-	9400 4600 9400 4800
-$Comp
-L antmicroCapacitors0402:C_10p_0402 C8
-U 1 1 619A945F
-P 9400 5000
-F 0 "C8" H 9515 5045 60  0000 L CNN
-F 1 "C_10p_0402" H 9400 4850 60  0001 C CNN
-F 2 "antmicro-footprints:0402-cap" H 9600 5200 60  0001 L CNN
-F 3 "" H 9400 5000 50  0001 C CNN
-F 4 "MULTICOMP" H 9600 5400 60  0001 L CNN "Manufacturer"
-F 5 "MC0402N100D500CT" H 9600 5300 60  0001 L CNN "MPN"
-F 6 "10p" H 9515 4947 50  0000 L CNN "Val"
-	1    9400 5000
-	1    0    0    -1
-$EndComp
-$Comp
-L power:GND #PWR012
-U 1 1 619A95EF
-P 9400 5150
-F 0 "#PWR012" H 9400 4900 50  0001 C CNN
-F 1 "GND" H 9405 4977 50  0000 C CNN
-F 2 "" H 9400 5150 50  0001 C CNN
-F 3 "" H 9400 5150 50  0001 C CNN
-	1    9400 5150
-	1    0    0    -1
-$EndComp
-Connection ~ 8850 4800
-Wire Wire Line
-	8850 4800 8850 4850
-$Comp
-L antmicroResistors0402:R_1M0_0402 R19
-U 1 1 619ADB78
-P 9150 4800
-F 0 "R19" H 9150 5013 60  0000 C CNN
-F 1 "R_1M0_0402" H 9150 4650 60  0001 C CNN
-F 2 "antmicro-footprints:0402-res" H 9350 5000 60  0001 L CNN
-F 3 "" H 9150 4800 50  0001 C CNN
-F 4 "TE CONNECTIVITY" H 9350 5200 60  0001 L CNN "Manufacturer"
-F 5 "CRG0402F1M0" H 9350 5100 60  0001 L CNN "MPN"
-F 6 "1M0" H 9150 4915 50  0000 C CNN "Val"
-	1    9150 4800
-	1    0    0    -1
-$EndComp
-Wire Wire Line
-	8850 4800 9000 4800
-Wire Wire Line
-	9300 4800 9400 4800
-Connection ~ 9400 4800
-Wire Wire Line
-	9400 4800 9400 4850
-Text Label 8600 4800 0    50   ~ 0
-XTAL1
-Wire Wire Line
-	8600 4800 8850 4800
-Wire Wire Line
-	9400 4800 9650 4800
-Text Label 9650 4800 0    50   ~ 0
-XTAL2
-Text Notes 8850 4500 0    50   ~ 0
-Why is this 1M resistor here? \n
+P 8400 4950
+F 0 "#PWR05" H 8400 4700 50  0001 C CNN
+F 1 "GND" H 8405 4777 50  0000 C CNN
+F 2 "" H 8400 4950 50  0001 C CNN
+F 3 "" H 8400 4950 50  0001 C CNN
+	1    8400 4950
+	1    0    0    -1
+$EndComp
 $Comp
 L power:+1V8 #PWR013
@@
 Text GLabel 6000 5950 0    50   Input ~ 0
 PCIE1_WAKE_N
+$Comp
+L antmicroOscillators:ECS-1618-250-BN-TR Y?
+U 1 1 61A23266
+P 7000 4200
+F 0 "Y?" H 7600 4549 50  0000 C CNN
+F 1 "ECS-1618-250-BN-TR" H 7600 4458 50  0000 C CNN
+F 2 "antmicro-footprints:OSC_ECS-1618-250-BN-TR" H 7000 4200 50  0001 C CNN
+F 3 "https://ecsxtal.com/store/pdf/ECS_1618.pdf" H 7000 4200 50  0001 C CNN
+F 4 "ECS-1618-250-BN-TR" H 7600 4367 50  0000 C CNN "MPN"
+F 5 "ECSXTAL" H 7600 4276 50  0000 C CNN "Manufacturer"
+	1    7000 4200
+	1    0    0    -1
+$EndComp
+Text Notes 9950 4750 0    50   ~ 0
+Review Oscillator connection.
+Text Label 9750 4500 0    50   ~ 0
+XTAL2
+Wire Wire Line
+	9500 4500 9750 4500
+Wire Wire Line
+	8700 4500 8950 4500
+Text Label 8700 4500 0    50   ~ 0
+XTAL1
+Wire Wire Line
+	9500 4500 9500 4550
+Connection ~ 9500 4500
+Wire Wire Line
+	9400 4500 9500 4500
+Wire Wire Line
+	8950 4500 9100 4500
+$Comp
+L antmicroResistors0402:R_1M0_0402 R19
+U 1 1 619ADB78
+P 9250 4500
+F 0 "R19" H 9250 4713 60  0000 C CNN
+F 1 "R_1M0_0402" H 9250 4350 60  0001 C CNN
+F 2 "antmicro-footprints:0402-res" H 9450 4700 60  0001 L CNN
+F 3 "" H 9250 4500 50  0001 C CNN
+F 4 "TE CONNECTIVITY" H 9450 4900 60  0001 L CNN "Manufacturer"
+F 5 "CRG0402F1M0" H 9450 4800 60  0001 L CNN "MPN"
+F 6 "1M0" H 9250 4615 50  0000 C CNN "Val"
+	1    9250 4500
+	1    0    0    -1
+$EndComp
+Wire Wire Line
+	8950 4500 8950 4550
+Connection ~ 8950 4500
+$Comp
+L power:GND #PWR012
+U 1 1 619A95EF
+P 9500 4850
+F 0 "#PWR012" H 9500 4600 50  0001 C CNN
+F 1 "GND" H 9505 4677 50  0000 C CNN
+F 2 "" H 9500 4850 50  0001 C CNN
+F 3 "" H 9500 4850 50  0001 C CNN
+	1    9500 4850
+	1    0    0    -1
+$EndComp
+$Comp
+L antmicroCapacitors0402:C_10p_0402 C8
+U 1 1 619A945F
+P 9500 4700
+F 0 "C8" H 9615 4745 60  0000 L CNN
+F 1 "C_10p_0402" H 9500 4550 60  0001 C CNN
+F 2 "antmicro-footprints:0402-cap" H 9700 4900 60  0001 L CNN
+F 3 "" H 9500 4700 50  0001 C CNN
+F 4 "MULTICOMP" H 9700 5100 60  0001 L CNN "Manufacturer"
+F 5 "MC0402N100D500CT" H 9700 5000 60  0001 L CNN "MPN"
+F 6 "10p" H 9615 4647 50  0000 L CNN "Val"
+	1    9500 4700
+	1    0    0    -1
+$EndComp
+$Comp
+L power:GND #PWR011
+U 1 1 619A53C6
+P 8950 4850
+F 0 "#PWR011" H 8950 4600 50  0001 C CNN
+F 1 "GND" H 8955 4677 50  0000 C CNN
+F 2 "" H 8950 4850 50  0001 C CNN
+F 3 "" H 8950 4850 50  0001 C CNN
+	1    8950 4850
+	1    0    0    -1
+$EndComp
+$Comp
+L antmicroCapacitors0402:C_10p_0402 C7
+U 1 1 619A5032
+P 8950 4700
+F 0 "C7" H 9065 4745 60  0000 L CNN
+F 1 "C_10p_0402" H 8950 4550 60  0001 C CNN
+F 2 "antmicro-footprints:0402-cap" H 9150 4900 60  0001 L CNN
+F 3 "" H 8950 4700 50  0001 C CNN
+F 4 "MULTICOMP" H 9150 5100 60  0001 L CNN "Manufacturer"
+F 5 "MC0402N100D500CT" H 9150 5000 60  0001 L CNN "MPN"
+F 6 "10p" H 9065 4647 50  0000 L CNN "Val"
+	1    8950 4700
+	1    0    0    -1
+$EndComp
+Wire Wire Line
+	8950 4400 8950 4500
+Text Notes 8950 4200 0    50   ~ 0
+Why is this 1M resistor here? \n
+Wire Wire Line
+	9500 3850 6800 3850
+Wire Wire Line
+	6800 3850 6800 4400
+Wire Wire Line
+	9500 3850 9500 4500
+Wire Wire Line
+	8400 4400 8950 4400
+$Comp
+L antmicroResistors0402:R_2k49_1%_0402 R?
+U 1 1 61B0F054
+P 3200 4850
+F 0 "R?" V 2800 4700 60  0000 L CNN
+F 1 "R_2k49_1%_0402" H 3200 4700 60  0001 C CNN
+F 2 "antmicro-footprints:0402-res" H 3400 5050 60  0001 L CNN
+F 3 "" H 3200 4850 50  0001 C CNN
+F 4 "Bourns" H 3400 5250 60  0001 L CNN "Manufacturer"
+F 5 "CR0502-FX-2491GLF" H 3400 5150 60  0001 L CNN "MPN"
+F 6 "2k49_1%" H 2750 4900 50  0000 L CNN "Val"
+	1    3200 4850
+	0    1    1    0
+$EndComp
 $EndSCHEMATC
