File: sa800u-baseboard-hw/sa800u-baseboard-hw.sch (KiCad schematic (older format))
At the start: 0 parts

Commit message: Review - Add geeral remarks
Other:
- note added: "GENERAL REMARKS:\n-Nice sheet separation\n-Nice and clear signal labeling\n-Use "kmake get-ignore" inside the repo to make git ignore backup\n files\n-Make folder structure flat - move files ../ \n-Make all the sheets A3 format\n-Avoid "space" in file names use "_" instead"
Changed lines of the file:
@@
 F1 "Level_shift_HDMI.sch" 50
 $EndSheet
+Text Notes 625  6150 0    50   ~ 0
+GENERAL REMARKS:\n-Nice sheet separation\n-Nice and clear signal labeling\n-Use "kmake get-ignore" inside the repo to make git ignore backup\n files\n-Make folder structure flat - move files ../ \n-Make all the sheets A3 format\n-Avoid "space" in file names use "_" instead
 $EndSCHEMATC
