File: SoM.sch (KiCad schematic (older format))
At the start: 0 parts

Commit message: added Cameras interface and finished SoM model and symbol
Parts:
- added U?: SA800U-WF-J1, symbol SA800U-WF:SA800U-WF-J1
- added U?: SA800U-WF-J2, symbol SA800U-WF:SA800U-WF-J2
- added U?: SA800U-WF-J3, symbol SA800U-WF:SA800U-WF-J3
- added U?: SA800U-WF-J4, symbol SA800U-WF:SA800U-WF-J4
Connections:
- net labels added: CAM0_AFVDD_EN, CAM0_AVDD_EN, CAM0_DVDD_EN, CAM0_PWDN, CAM0_RST, CAM1_AFVDD_EN, CAM1_AVDD_EN, CAM1_DVDD_EN, CAM1_PWDN, CAM1_RST, CAM3_RST, CAM3_TRIGGER_OUT, CAM3_VCC_EN, CCI0_I2C_SCL, CCI0_I2C_SDA, CCI1_I2C_SCL, CCI1_I2C_SDA, CSI0_CLK_N, CSI0_CLK_P, CSI0_LN0_N, CSI0_LN0_P, CSI0_LN1_N, CSI0_LN1_P, CSI0_LN2_N, CSI0_LN2_P, CSI0_LN3_N, CSI0_LN3_P, CSI1_CLK_N, CSI1_CLK_P, CSI1_LN0_N, CSI1_LN0_P, CSI1_LN1_N, CSI1_LN1_P, CSI1_LN2_N, CSI1_LN2_P, CSI1_LN3_N, CSI1_LN3_P, CSI2_LN1_N, CSI2_LN1_P, CSI2_LN2_N, CSI2_LN2_P, CSI2_LN3_N, CSI2_LN3_P, GND, HDMI1_INTO, LT6911_3V3_EN, LT6911_RST, PWR_OFF, RESET_USBHUB, VBAT
- wire segments 0 -> 76
- no-connect marks 0 -> 14
Other:
- note added: "SPI may be exposed on a connector?"
