File: SoM.sch (KiCad schematic (older format))
At the start: 4 parts

Commit message: work in progress, added usb hub, connectors, and m2 connector
Parts:
- removed U?: SA800U-WF-J1, symbol SA800U-WF:SA800U-WF-J1
- removed U?: SA800U-WF-J2, symbol SA800U-WF:SA800U-WF-J2
- removed U?: SA800U-WF-J3, symbol SA800U-WF:SA800U-WF-J3
- removed U?: SA800U-WF-J4, symbol SA800U-WF:SA800U-WF-J4
- added U? (x4): SA800U-WF, antmicro-footprints:SA800U-WF, symbol antmicroMicrocontrollers:SA800U-WF
Changed lines of the file:
@@
 $Descr A3 16535 11693
 encoding utf-8
-Sheet 8 9
+Sheet 7 9
 Title ""
 Date ""
@@
 Comment4 ""
 $EndDescr
-$Comp
-L SA800U-WF:SA800U-WF-J1 U?
-U 1 1 61A8EF71
-P 1750 1650
-F 0 "U?" H 2475 1815 50  0000 C CNN
-F 1 "SA800U-WF-J1" H 2475 1724 50  0000 C CNN
-F 2 "" H 1850 1450 50  0001 C CNN
-F 3 "" H 1850 1450 50  0001 C CNN
-	1    1750 1650
-	1    0    0    -1
-$EndComp
-$Comp
-L SA800U-WF:SA800U-WF-J2 U?
-U 1 1 61A93EC2
-P 6150 1650
-F 0 "U?" H 6388 1815 50  0000 C CNN
-F 1 "SA800U-WF-J2" H 6388 1724 50  0000 C CNN
-F 2 "" H 6450 1000 50  0001 C CNN
-F 3 "" H 6450 1000 50  0001 C CNN
-	1    6150 1650
-	1    0    0    -1
-$EndComp
-$Comp
-L SA800U-WF:SA800U-WF-J3 U?
-U 1 1 61A9F40B
-P 11000 1700
-F 0 "U?" H 11650 1865 50  0000 C CNN
-F 1 "SA800U-WF-J3" H 11650 1774 50  0000 C CNN
-F 2 "" H 11050 1700 50  0001 C CNN
-F 3 "" H 11050 1700 50  0001 C CNN
-	1    11000 1700
-	1    0    0    -1
-$EndComp
-$Comp
-L SA800U-WF:SA800U-WF-J4 U?
-U 1 1 61AA09E5
-P 11000 5900
-F 0 "U?" H 11650 6065 50  0000 C CNN
-F 1 "SA800U-WF-J4" H 11650 5974 50  0000 C CNN
-F 2 "" H 11000 5850 50  0001 C CNN
-F 3 "" H 11000 5850 50  0001 C CNN
-	1    11000 5900
-	1    0    0    -1
-$EndComp
 $Comp
 L power:GND #PWR?
@@
 Wire Wire Line
 	1650 9550 1300 9550
-Connection ~ 1650 9550
 Wire Wire Line
 	1550 9650 1650 9650
@@
 Wire Wire Line
 	1300 10150 1650 10150
+$Comp
+L antmicroMicrocontrollers:SA800U-WF U?
+U 1 1 61B940C3
+P 1750 1650
+F 0 "U?" H 2475 1997 50  0000 C CNN
+F 1 "SA800U-WF" H 2475 1906 50  0000 C CNN
+F 2 "antmicro-footprints:SA800U-WF" H 1750 1650 50  0001 C CNN
+F 3 "https://www.quectel.com/wp-content/uploads/2021/05/Quectel_SA800U-WF_Hardware_Design_V1.0.pdf" H 1750 1650 50  0001 C CNN
+F 4 "SA800U-WF" H 2475 1815 50  0000 C CNN "MPN"
+F 5 "QUECTEL" H 2475 1724 50  0000 C CNN "Manufacturer"
+	1    1750 1650
+	1    0    0    -1
+$EndComp
+Connection ~ 1650 9550
+$Comp
+L antmicroMicrocontrollers:SA800U-WF U?
+U 2 1 61BAF70E
+P 5150 1750
+F 0 "U?" H 5875 2097 50  0000 C CNN
+F 1 "SA800U-WF" H 5875 2006 50  0000 C CNN
+F 2 "antmicro-footprints:SA800U-WF" H 5150 1750 50  0001 C CNN
+F 3 "https://www.quectel.com/wp-content/uploads/2021/05/Quectel_SA800U-WF_Hardware_Design_V1.0.pdf" H 5150 1750 50  0001 C CNN
+F 4 "SA800U-WF" H 5875 1915 50  0000 C CNN "MPN"
+F 5 "QUECTEL" H 5875 1824 50  0000 C CNN "Manufacturer"
+	2    5150 1750
+	1    0    0    -1
+$EndComp
+$Comp
+L antmicroMicrocontrollers:SA800U-WF U?
+U 3 1 61BB5D93
+P 9600 2250
+F 0 "U?" H 10250 2597 50  0000 C CNN
+F 1 "SA800U-WF" H 10250 2506 50  0000 C CNN
+F 2 "antmicro-footprints:SA800U-WF" H 9600 2250 50  0001 C CNN
+F 3 "https://www.quectel.com/wp-content/uploads/2021/05/Quectel_SA800U-WF_Hardware_Design_V1.0.pdf" H 9600 2250 50  0001 C CNN
+F 4 "SA800U-WF" H 10250 2415 50  0000 C CNN "MPN"
+F 5 "QUECTEL" H 10250 2324 50  0000 C CNN "Manufacturer"
+	3    9600 2250
+	1    0    0    -1
+$EndComp
+$Comp
+L antmicroMicrocontrollers:SA800U-WF U?
+U 4 1 61BBA563
+P 9500 7200
+F 0 "U?" H 10150 7547 50  0000 C CNN
+F 1 "SA800U-WF" H 10150 7456 50  0000 C CNN
+F 2 "antmicro-footprints:SA800U-WF" H 9500 7200 50  0001 C CNN
+F 3 "https://www.quectel.com/wp-content/uploads/2021/05/Quectel_SA800U-WF_Hardware_Design_V1.0.pdf" H 9500 7200 50  0001 C CNN
+F 4 "SA800U-WF" H 10150 7365 50  0000 C CNN "MPN"
+F 5 "QUECTEL" H 10150 7274 50  0000 C CNN "Manufacturer"
+	4    9500 7200
+	1    0    0    -1
+$EndComp
 $EndSCHEMATC

Commit message: added sd card, buttons, rtc battery - work in progress
Parts:
- added BAT?: BLP2032SM-GCT-ND, antmicro-footprints:BLP2032SM-GCT-ND, symbol antmicroBatteryHoldersClipsContacts:BLP2032SM-GCT-ND
- added S? (x4): TL3340AF160QG, antmicro-footprints:TL3340AF160QG, symbol antmicroPushbuttonSwitches:TL3340AF160QG
Other:
- note added: "Work in progress."
Changed lines of the file:
@@
 $Descr A3 16535 11693
 encoding utf-8
-Sheet 7 9
+Sheet 7 10
 Title ""
 Date ""
@@
 	1    0    0    -1
 $EndComp
+$Comp
+L antmicroBatteryHoldersClipsContacts:BLP2032SM-GCT-ND BAT?
+U 1 1 61C092A2
+P 11600 8050
+AR Path="/61C092A2" Ref="BAT?"  Part="1"
+AR Path="/61A4BC4F/61C092A2" Ref="BAT?"  Part="1"
+F 0 "BAT?" H 11730 8053 60  0000 L CNN
+F 1 "BLP2032SM-GCT-ND" H 11730 7947 60  0000 L CNN
+F 2 "antmicro-footprints:BLP2032SM-GCT-ND" H 11600 8050 60  0001 C CNN
+F 3 "" H 11600 8050 60  0001 C CNN
+F 4 "MPD" H 11600 8050 50  0001 C CNN "Manufacturer"
+F 5 "BLP2032SM-GCT-ND" H 11600 8050 50  0001 C CNN "MPN"
+	1    11600 8050
+	1    0    0    -1
+$EndComp
+$Comp
+L antmicroPushbuttonSwitches:TL3340AF160QG S?
+U 1 1 61C126F3
+P 12550 8100
+F 0 "S?" H 12650 8547 50  0000 C CNN
+F 1 "TL3340AF160QG" H 12650 8456 50  0000 C CNN
+F 2 "antmicro-footprints:TL3340AF160QG" H 12550 8100 50  0001 C CNN
+F 3 "https://pl.mouser.com/datasheet/2/140/TL3340-2065742.pdf" H 12550 8100 50  0001 C CNN
+F 4 "TL3340AF160QG" H 12650 8365 50  0000 C CNN "MPN"
+F 5 "" H 12550 8100 50  0000 C CNN "Manufacturer"
+	1    12550 8100
+	1    0    0    -1
+$EndComp
+$Comp
+L antmicroPushbuttonSwitches:TL3340AF160QG S?
+U 1 1 61C145CA
+P 12550 8850
+F 0 "S?" H 12650 9297 50  0000 C CNN
+F 1 "TL3340AF160QG" H 12650 9206 50  0000 C CNN
+F 2 "antmicro-footprints:TL3340AF160QG" H 12550 8850 50  0001 C CNN
+F 3 "https://pl.mouser.com/datasheet/2/140/TL3340-2065742.pdf" H 12550 8850 50  0001 C CNN
+F 4 "TL3340AF160QG" H 12650 9115 50  0000 C CNN "MPN"
+F 5 "" H 12550 8850 50  0000 C CNN "Manufacturer"
+	1    12550 8850
+	1    0    0    -1
+$EndComp
+$Comp
+L antmicroPushbuttonSwitches:TL3340AF160QG S?
+U 1 1 61C150DA
+P 12550 7400
+F 0 "S?" H 12650 7847 50  0000 C CNN
+F 1 "TL3340AF160QG" H 12650 7756 50  0000 C CNN
+F 2 "antmicro-footprints:TL3340AF160QG" H 12550 7400 50  0001 C CNN
+F 3 "https://pl.mouser.com/datasheet/2/140/TL3340-2065742.pdf" H 12550 7400 50  0001 C CNN
+F 4 "TL3340AF160QG" H 12650 7665 50  0000 C CNN "MPN"
+F 5 "" H 12550 7400 50  0000 C CNN "Manufacturer"
+	1    12550 7400
+	1    0    0    -1
+$EndComp
+$Comp
+L antmicroPushbuttonSwitches:TL3340AF160QG S?
+U 1 1 61C1584E
+P 12550 9550
+F 0 "S?" H 12650 9997 50  0000 C CNN
+F 1 "TL3340AF160QG" H 12650 9906 50  0000 C CNN
+F 2 "antmicro-footprints:TL3340AF160QG" H 12550 9550 50  0001 C CNN
+F 3 "https://pl.mouser.com/datasheet/2/140/TL3340-2065742.pdf" H 12550 9550 50  0001 C CNN
+F 4 "TL3340AF160QG" H 12650 9815 50  0000 C CNN "MPN"
+F 5 "" H 12550 9550 50  0000 C CNN "Manufacturer"
+	1    12550 9550
+	1    0    0    -1
+$EndComp
+Text Notes 11550 7700 0    50   ~ 0
+Work in progress.
 $EndSCHEMATC

Commit message: added some usb connectors, goldpins for GPIO and I2C, fixed buttons
Parts:
- removed S? (x4): TL3340AF160QG, antmicro-footprints:TL3340AF160QG, symbol antmicroPushbuttonSwitches:TL3340AF160QG
- added S? (x4): KMR2, antmicro-footprints:SW_SPST_4.2x2.8, symbol antmicroPushbuttonSwitches:KMR2
Changed lines of the file:
@@
-	1    0    0    -1
-$EndComp
-$Comp
-L antmicroPushbuttonSwitches:TL3340AF160QG S?
-U 1 1 61C126F3
-P 12550 8100
-F 0 "S?" H 12650 8547 50  0000 C CNN
-F 1 "TL3340AF160QG" H 12650 8456 50  0000 C CNN
-F 2 "antmicro-footprints:TL3340AF160QG" H 12550 8100 50  0001 C CNN
-F 3 "https://pl.mouser.com/datasheet/2/140/TL3340-2065742.pdf" H 12550 8100 50  0001 C CNN
-F 4 "TL3340AF160QG" H 12650 8365 50  0000 C CNN "MPN"
-F 5 "" H 12550 8100 50  0000 C CNN "Manufacturer"
-	1    12550 8100
-	1    0    0    -1
-$EndComp
-$Comp
-L antmicroPushbuttonSwitches:TL3340AF160QG S?
-U 1 1 61C145CA
-P 12550 8850
-F 0 "S?" H 12650 9297 50  0000 C CNN
-F 1 "TL3340AF160QG" H 12650 9206 50  0000 C CNN
-F 2 "antmicro-footprints:TL3340AF160QG" H 12550 8850 50  0001 C CNN
-F 3 "https://pl.mouser.com/datasheet/2/140/TL3340-2065742.pdf" H 12550 8850 50  0001 C CNN
-F 4 "TL3340AF160QG" H 12650 9115 50  0000 C CNN "MPN"
-F 5 "" H 12550 8850 50  0000 C CNN "Manufacturer"
-	1    12550 8850
-	1    0    0    -1
-$EndComp
-$Comp
-L antmicroPushbuttonSwitches:TL3340AF160QG S?
-U 1 1 61C150DA
-P 12550 7400
-F 0 "S?" H 12650 7847 50  0000 C CNN
-F 1 "TL3340AF160QG" H 12650 7756 50  0000 C CNN
-F 2 "antmicro-footprints:TL3340AF160QG" H 12550 7400 50  0001 C CNN
-F 3 "https://pl.mouser.com/datasheet/2/140/TL3340-2065742.pdf" H 12550 7400 50  0001 C CNN
-F 4 "TL3340AF160QG" H 12650 7665 50  0000 C CNN "MPN"
-F 5 "" H 12550 7400 50  0000 C CNN "Manufacturer"
-	1    12550 7400
-	1    0    0    -1
-$EndComp
-$Comp
-L antmicroPushbuttonSwitches:TL3340AF160QG S?
-U 1 1 61C1584E
-P 12550 9550
-F 0 "S?" H 12650 9997 50  0000 C CNN
-F 1 "TL3340AF160QG" H 12650 9906 50  0000 C CNN
-F 2 "antmicro-footprints:TL3340AF160QG" H 12550 9550 50  0001 C CNN
-F 3 "https://pl.mouser.com/datasheet/2/140/TL3340-2065742.pdf" H 12550 9550 50  0001 C CNN
-F 4 "TL3340AF160QG" H 12650 9815 50  0000 C CNN "MPN"
-F 5 "" H 12550 9550 50  0000 C CNN "Manufacturer"
-	1    12550 9550
 	1    0    0    -1
 $EndComp
 Text Notes 11550 7700 0    50   ~ 0
 Work in progress.
+$Comp
+L antmicroPushbuttonSwitches:KMR2 S?
+U 1 1 61C94E75
+P 14000 7350
+F 0 "S?" H 14000 7625 50  0000 C CNN
+F 1 "KMR2" H 14000 7534 50  0000 C CNN
+F 2 "antmicro-footprints:SW_SPST_4.2x2.8" H 14200 7550 50  0001 L CNN
+F 3 "http://www.farnell.com/datasheets/2631211.pdf" H 14200 7650 60  0001 L CNN
+F 4 "KMR211NGLFS" H 14196 7743 60  0001 L CNN "MPN"
+F 5 "C&K Components" H 14200 7822 60  0001 L CNN "Manufacturer"
+	1    14000 7350
+	1    0    0    -1
+$EndComp
+$Comp
+L antmicroPushbuttonSwitches:KMR2 S?
+U 1 1 61CA28EE
+P 14000 7850
+F 0 "S?" H 14000 8125 50  0000 C CNN
+F 1 "KMR2" H 14000 8034 50  0000 C CNN
+F 2 "antmicro-footprints:SW_SPST_4.2x2.8" H 14200 8050 50  0001 L CNN
+F 3 "http://www.farnell.com/datasheets/2631211.pdf" H 14200 8150 60  0001 L CNN
+F 4 "KMR211NGLFS" H 14196 8243 60  0001 L CNN "MPN"
+F 5 "C&K Components" H 14200 8322 60  0001 L CNN "Manufacturer"
+	1    14000 7850
+	1    0    0    -1
+$EndComp
+$Comp
+L antmicroPushbuttonSwitches:KMR2 S?
+U 1 1 61CA563B
+P 14000 8400
+F 0 "S?" H 14000 8675 50  0000 C CNN
+F 1 "KMR2" H 14000 8584 50  0000 C CNN
+F 2 "antmicro-footprints:SW_SPST_4.2x2.8" H 14200 8600 50  0001 L CNN
+F 3 "http://www.farnell.com/datasheets/2631211.pdf" H 14200 8700 60  0001 L CNN
+F 4 "KMR211NGLFS" H 14196 8793 60  0001 L CNN "MPN"
+F 5 "C&K Components" H 14200 8872 60  0001 L CNN "Manufacturer"
+	1    14000 8400
+	1    0    0    -1
+$EndComp
+$Comp
+L antmicroPushbuttonSwitches:KMR2 S?
+U 1 1 61CA8515
+P 14000 8900
+F 0 "S?" H 14000 9175 50  0000 C CNN
+F 1 "KMR2" H 14000 9084 50  0000 C CNN
+F 2 "antmicro-footprints:SW_SPST_4.2x2.8" H 14200 9100 50  0001 L CNN
+F 3 "http://www.farnell.com/datasheets/2631211.pdf" H 14200 9200 60  0001 L CNN
+F 4 "KMR211NGLFS" H 14196 9293 60  0001 L CNN "MPN"
+F 5 "C&K Components" H 14200 9372 60  0001 L CNN "Manufacturer"
+	1    14000 8900
+	1    0    0    -1
+$EndComp
 $EndSCHEMATC
