File: SoM.sch (KiCad schematic (older format))
At the start: 12 parts, among them J5 MC-HVT1-S04-G, U8 SA800U-WF

Commit message: add decoupling capacitors and tvs to som
Parts:
- added C?: C_100u_0805, antmicro-footprints:0805-cap, symbol antmicroCapacitorsmisc:C_100u_0805
- added C?: C_100n_0402, antmicro-footprints:0402-cap, symbol antmicroCapacitors0402:C_100n_0402
- added C?: C_33p_0402, antmicro-footprints:0402-cap, symbol antmicroCapacitors0402:C_33p_0402
- added C?: C_10p_0402, antmicro-footprints:0402-cap, symbol antmicroCapacitors0402:C_10p_0402
- added D?: STS321045B502, antmicro-footprints:STS321045B502, symbol antmicroTVSDiodes:STS321045B502
Connections:
- wire segments 397 -> 412
Changed lines of the file:
@@
 Wire Wire Line
 	12650 5950 12650 6250
-Text Label 11500 7850 0    50   ~ 0
+Text Label 11500 7400 0    50   ~ 0
 VOL_UP_TVS
 $Comp
 L power:GND #PWR0177
 U 1 1 61F2FF9D
-P 15300 7650
-F 0 "#PWR0177" H 15300 7400 50  0001 C CNN
-F 1 "GND" V 15305 7522 50  0000 R CNN
-F 2 "" H 15300 7650 50  0001 C CNN
-F 3 "" H 15300 7650 50  0001 C CNN
-	1    15300 7650
+P 15300 7200
+F 0 "#PWR0177" H 15300 6950 50  0001 C CNN
+F 1 "GND" V 15305 7072 50  0000 R CNN
+F 2 "" H 15300 7200 50  0001 C CNN
+F 3 "" H 15300 7200 50  0001 C CNN
+	1    15300 7200
 	0    -1   -1   0
 $EndComp
 Wire Wire Line
-	15000 7650 15300 7650
+	15000 7200 15300 7200
 Wire Wire Line
-	15300 8050 15000 8050
+	15300 7600 15000 7600
 Wire Wire Line
-	15000 7850 15300 7850
-Text Label 15300 7850 0    50   ~ 0
+	15000 7400 15300 7400
+Text Label 15300 7400 0    50   ~ 0
 VOL_DOWN_TVS
-Text Label 15300 8050 0    50   ~ 0
+Text Label 15300 7600 0    50   ~ 0
 HOME_TVS
 Wire Wire Line
-	12000 7850 11500 7850
+	12000 7400 11500 7400
 Wire Wire Line
-	11500 7650 12000 7650
-Text Label 11500 7650 0    50   ~ 0
+	11500 7200 12000 7200
+Text Label 11500 7200 0    50   ~ 0
 PWRKEY_TVS
 $Comp
 L antmicroTVSDiodes:RCLAMP2504N.TCT D18
 U 1 1 61D0B3AA
-P 13500 7900
-F 0 "D18" H 13500 8697 50  0000 C CNN
-F 1 "RCLAMP2504N.TCT" H 13500 8606 50  0000 C CNN
-F 2 "antmicro-footprints:RCLAMP2504N.TCT" H 13500 7900 50  0001 C CNN
-F 3 "https://pl.mouser.com/datasheet/2/761/SEMTS05345_1-2575174.pdf" H 13500 7900 50  0001 C CNN
-F 4 "RCLAMP2504N.TCT" H 13500 8515 50  0000 C CNN "MPN"
-F 5 "SEMTECH" H 13500 8424 50  0000 C CNN "Manufacturer"
-	1    13500 7900
+P 13500 7450
+F 0 "D18" H 13500 8247 50  0000 C CNN
+F 1 "RCLAMP2504N.TCT" H 13500 8156 50  0000 C CNN
+F 2 "antmicro-footprints:RCLAMP2504N.TCT" H 13500 7450 50  0001 C CNN
+F 3 "https://pl.mouser.com/datasheet/2/761/SEMTS05345_1-2575174.pdf" H 13500 7450 50  0001 C CNN
+F 4 "RCLAMP2504N.TCT" H 13500 8065 50  0000 C CNN "MPN"
+F 5 "SEMTECH" H 13500 7974 50  0000 C CNN "Manufacturer"
+	1    13500 7450
 	1    0    0    -1
 $EndComp
@@
 Wire Wire Line
 	8100 5400 7600 5400
+Text GLabel 12350 8700 0    50   Input ~ 0
+VBAT
+Wire Wire Line
+	12350 8700 12600 8700
+$Comp
+L antmicroCapacitorsmisc:C_100u_0805 C?
+U 1 1 61F3DBE1
+P 12600 9050
+F 0 "C?" H 12715 9095 60  0000 L CNN
+F 1 "C_100u_0805" H 12600 8900 60  0001 C CNN
+F 2 "antmicro-footprints:0805-cap" H 12800 9250 60  0001 L CNN
+F 3 "" H 12600 9050 50  0001 C CNN
+F 4 "MURATA" H 12800 9450 60  0001 L CNN "Manufacturer"
+F 5 "GRM21BR60J107ME15L" H 12800 9350 60  0001 L CNN "MPN"
+F 6 "100u" H 12715 8997 50  0000 L CNN "Val"
+	1    12600 9050
+	1    0    0    -1
+$EndComp
+$Comp
+L antmicroCapacitors0402:C_100n_0402 C?
+U 1 1 61F40427
+P 13050 9050
+F 0 "C?" H 13165 9095 60  0000 L CNN
+F 1 "C_100n_0402" H 13050 8900 60  0001 C CNN
+F 2 "antmicro-footprints:0402-cap" H 13250 9250 60  0001 L CNN
+F 3 "" H 13050 9050 50  0001 C CNN
+F 4 "Walsin" H 13250 9450 60  0001 L CNN "Manufacturer"
+F 5 "0402X104K6R3CT" H 13250 9350 60  0001 L CNN "MPN"
+F 6 "100n" H 13165 8997 50  0000 L CNN "Val"
+	1    13050 9050
+	1    0    0    -1
+$EndComp
+$Comp
+L antmicroCapacitors0402:C_33p_0402 C?
+U 1 1 61F422BA
+P 13500 9050
+F 0 "C?" H 13615 9095 60  0000 L CNN
+F 1 "C_33p_0402" H 13500 8900 60  0001 C CNN
+F 2 "antmicro-footprints:0402-cap" H 13700 9250 60  0001 L CNN
+F 3 "" H 13500 9050 50  0001 C CNN
+F 4 "MULTICOMP" H 13700 9450 60  0001 L CNN "Manufacturer"
+F 5 "MC0402N330J500CT" H 13700 9350 60  0001 L CNN "MPN"
+F 6 "33p" H 13615 8997 50  0000 L CNN "Val"
+	1    13500 9050
+	1    0    0    -1
+$EndComp
+$Comp
+L antmicroCapacitors0402:C_10p_0402 C?
+U 1 1 61F4405A
+P 13900 9050
+F 0 "C?" H 14015 9095 60  0000 L CNN
+F 1 "C_10p_0402" H 13900 8900 60  0001 C CNN
+F 2 "antmicro-footprints:0402-cap" H 14100 9250 60  0001 L CNN
+F 3 "" H 13900 9050 50  0001 C CNN
+F 4 "MULTICOMP" H 14100 9450 60  0001 L CNN "Manufacturer"
+F 5 "MC0402N100D500CT" H 14100 9350 60  0001 L CNN "MPN"
+F 6 "10p" H 14015 8997 50  0000 L CNN "Val"
+	1    13900 9050
+	1    0    0    -1
+$EndComp
+Wire Wire Line
+	12600 8700 12600 8900
+Wire Wire Line
+	13900 8900 13500 8900
+Connection ~ 12600 8900
+Connection ~ 13050 8900
+Wire Wire Line
+	13050 8900 12600 8900
+Connection ~ 13500 8900
+Wire Wire Line
+	13500 8900 13050 8900
+Wire Wire Line
+	12600 9200 12600 9300
+Wire Wire Line
+	12600 9300 13050 9300
+Wire Wire Line
+	13900 9300 13900 9200
+Wire Wire Line
+	13050 9200 13050 9300
+Connection ~ 13050 9300
+Wire Wire Line
+	13050 9300 13500 9300
+Wire Wire Line
+	13500 9200 13500 9300
+Connection ~ 13500 9300
+Wire Wire Line
+	13500 9300 13900 9300
+$Comp
+L power:GND #PWR?
+U 1 1 620569CD
+P 12600 9400
+F 0 "#PWR?" H 12600 9150 50  0001 C CNN
+F 1 "GND" V 12605 9272 50  0000 R CNN
+F 2 "" H 12600 9400 50  0001 C CNN
+F 3 "" H 12600 9400 50  0001 C CNN
+	1    12600 9400
+	1    0    0    -1
+$EndComp
+Wire Wire Line
+	12600 9400 12600 9300
+Connection ~ 12600 9300
+$Comp
+L antmicroTVSDiodes:STS321045B502 D?
+U 1 1 620E0161
+P 14650 9100
+F 0 "D?" V 14604 9328 50  0000 L CNN
+F 1 "STS321045B502" V 14695 9328 50  0000 L CNN
+F 2 "antmicro-footprints:STS321045B502" H 14650 9100 50  0001 C CNN
+F 3 "https://www.eaton.com/content/dam/eaton/products/electronic-components/resources/data-sheet/eaton-sts321045b502-tvs-diode-esd-suppressor-data-sheet.pdf" H 14650 9100 50  0001 C CNN
+F 4 "STS321045B502" H 14650 9100 50  0001 C CNN "MPN"
+F 5 "Cooper Bussmann" H 14650 9100 50  0001 C CNN "Manufacturer"
+	1    14650 9100
+	0    1    1    0
+$EndComp
+Text GLabel 14650 8050 0    50   Input ~ 0
+VBAT
+Wire Wire Line
+	14650 8050 14650 8300
+$Comp
+L power:GND #PWR?
+U 1 1 6211DF21
+P 14650 10000
+F 0 "#PWR?" H 14650 9750 50  0001 C CNN
+F 1 "GND" V 14655 9872 50  0000 R CNN
+F 2 "" H 14650 10000 50  0001 C CNN
+F 3 "" H 14650 10000 50  0001 C CNN
+	1    14650 10000
+	1    0    0    -1
+$EndComp
+Wire Wire Line
+	14650 10000 14650 9900
 $EndSCHEMATC

Commit message: annotations
Parts:
- gave numbers to parts that had none: 5
- renumbered D18 to D14, J5 to J7, R85 to R73, R86 to R74, R87 to R75, R88 to R76, S4 to S1, S1 to S2, S2 to S3, S3 to S4, U8 to U10

Commit message: added bulk 2 more capacitors to som
Parts:
- added C? (x2): C_100u_0805, antmicro-footprints:0805-cap, symbol antmicroCapacitorsmisc:C_100u_0805
Connections:
- wire segments 412 -> 418
Other:
- moved on the sheet: C93
Changed lines of the file:
@@
 L antmicroCapacitorsmisc:C_100u_0805 C92
 U 1 1 61F3DBE1
-P 12600 9050
-F 0 "C92" H 12715 9095 60  0000 L CNN
-F 1 "C_100u_0805" H 12600 8900 60  0001 C CNN
-F 2 "antmicro-footprints:0805-cap" H 12800 9250 60  0001 L CNN
-F 3 "" H 12600 9050 50  0001 C CNN
-F 4 "MURATA" H 12800 9450 60  0001 L CNN "Manufacturer"
-F 5 "GRM21BR60J107ME15L" H 12800 9350 60  0001 L CNN "MPN"
-F 6 "100u" H 12715 8997 50  0000 L CNN "Val"
-	1    12600 9050
+P 12550 9100
+F 0 "C92" H 12665 9145 60  0000 L CNN
+F 1 "C_100u_0805" H 12550 8950 60  0001 C CNN
+F 2 "antmicro-footprints:0805-cap" H 12750 9300 60  0001 L CNN
+F 3 "" H 12550 9100 50  0001 C CNN
+F 4 "MURATA" H 12750 9500 60  0001 L CNN "Manufacturer"
+F 5 "GRM21BR60J107ME15L" H 12750 9400 60  0001 L CNN "MPN"
+F 6 "100u" H 12665 9047 50  0000 L CNN "Val"
+	1    12550 9100
 	1    0    0    -1
 $EndComp
@@
 L antmicroCapacitors0402:C_100n_0402 C93
 U 1 1 61F40427
-P 13050 9050
-F 0 "C93" H 13165 9095 60  0000 L CNN
-F 1 "C_100n_0402" H 13050 8900 60  0001 C CNN
-F 2 "antmicro-footprints:0402-cap" H 13250 9250 60  0001 L CNN
-F 3 "" H 13050 9050 50  0001 C CNN
-F 4 "Walsin" H 13250 9450 60  0001 L CNN "Manufacturer"
-F 5 "0402X104K6R3CT" H 13250 9350 60  0001 L CNN "MPN"
-F 6 "100n" H 13165 8997 50  0000 L CNN "Val"
-	1    13050 9050
+P 13000 9100
+F 0 "C93" H 13115 9145 60  0000 L CNN
+F 1 "C_100n_0402" H 13000 8950 60  0001 C CNN
+F 2 "antmicro-footprints:0402-cap" H 13200 9300 60  0001 L CNN
+F 3 "" H 13000 9100 50  0001 C CNN
+F 4 "Walsin" H 13200 9500 60  0001 L CNN "Manufacturer"
+F 5 "0402X104K6R3CT" H 13200 9400 60  0001 L CNN "MPN"
+F 6 "100n" H 13115 9047 50  0000 L CNN "Val"
+	1    13000 9100
 	1    0    0    -1
 $EndComp
@@
 L antmicroCapacitors0402:C_33p_0402 C94
 U 1 1 61F422BA
-P 13500 9050
-F 0 "C94" H 13615 9095 60  0000 L CNN
-F 1 "C_33p_0402" H 13500 8900 60  0001 C CNN
-F 2 "antmicro-footprints:0402-cap" H 13700 9250 60  0001 L CNN
-F 3 "" H 13500 9050 50  0001 C CNN
-F 4 "MULTICOMP" H 13700 9450 60  0001 L CNN "Manufacturer"
-F 5 "MC0402N330J500CT" H 13700 9350 60  0001 L CNN "MPN"
-F 6 "33p" H 13615 8997 50  0000 L CNN "Val"
-	1    13500 9050
+P 13450 9100
+F 0 "C94" H 13565 9145 60  0000 L CNN
+F 1 "C_33p_0402" H 13450 8950 60  0001 C CNN
+F 2 "antmicro-footprints:0402-cap" H 13650 9300 60  0001 L CNN
+F 3 "" H 13450 9100 50  0001 C CNN
+F 4 "MULTICOMP" H 13650 9500 60  0001 L CNN "Manufacturer"
+F 5 "MC0402N330J500CT" H 13650 9400 60  0001 L CNN "MPN"
+F 6 "33p" H 13565 9047 50  0000 L CNN "Val"
+	1    13450 9100
 	1    0    0    -1
 $EndComp
@@
 L antmicroCapacitors0402:C_10p_0402 C95
 U 1 1 61F4405A
-P 13900 9050
-F 0 "C95" H 14015 9095 60  0000 L CNN
-F 1 "C_10p_0402" H 13900 8900 60  0001 C CNN
-F 2 "antmicro-footprints:0402-cap" H 14100 9250 60  0001 L CNN
-F 3 "" H 13900 9050 50  0001 C CNN
-F 4 "MULTICOMP" H 14100 9450 60  0001 L CNN "Manufacturer"
-F 5 "MC0402N100D500CT" H 14100 9350 60  0001 L CNN "MPN"
-F 6 "10p" H 14015 8997 50  0000 L CNN "Val"
-	1    13900 9050
+P 13850 9100
+F 0 "C95" H 13965 9145 60  0000 L CNN
+F 1 "C_10p_0402" H 13850 8950 60  0001 C CNN
+F 2 "antmicro-footprints:0402-cap" H 14050 9300 60  0001 L CNN
+F 3 "" H 13850 9100 50  0001 C CNN
+F 4 "MULTICOMP" H 14050 9500 60  0001 L CNN "Manufacturer"
+F 5 "MC0402N100D500CT" H 14050 9400 60  0001 L CNN "MPN"
+F 6 "10p" H 13965 9047 50  0000 L CNN "Val"
+	1    13850 9100
 	1    0    0    -1
 $EndComp
 Wire Wire Line
-	13900 8900 13500 8900
-Connection ~ 13050 8900
+	13850 8950 13450 8950
+Connection ~ 13000 8950
 Wire Wire Line
-	13050 8900 12600 8900
-Connection ~ 13500 8900
+	13000 8950 12550 8950
+Connection ~ 13450 8950
 Wire Wire Line
-	13500 8900 13050 8900
+	13450 8950 13000 8950
 Wire Wire Line
-	12600 9200 12600 9300
+	12550 9250 12550 9350
 Wire Wire Line
-	12600 9300 13050 9300
+	12550 9350 13000 9350
 Wire Wire Line
-	13900 9300 13900 9200
+	13850 9350 13850 9250
 Wire Wire Line
-	13050 9200 13050 9300
-Connection ~ 13050 9300
+	13000 9250 13000 9350
+Connection ~ 13000 9350
 Wire Wire Line
-	13050 9300 13500 9300
+	13000 9350 13450 9350
 Wire Wire Line
-	13500 9200 13500 9300
-Connection ~ 13500 9300
+	13450 9250 13450 9350
+Connection ~ 13450 9350
 Wire Wire Line
-	13500 9300 13900 9300
+	13450 9350 13850 9350
 $Comp
 L power:GND #PWR0141
 U 1 1 620569CD
-P 12600 9400
-F 0 "#PWR0141" H 12600 9150 50  0001 C CNN
-F 1 "GND" V 12605 9272 50  0000 R CNN
-F 2 "" H 12600 9400 50  0001 C CNN
-F 3 "" H 12600 9400 50  0001 C CNN
-	1    12600 9400
+P 12550 9450
+F 0 "#PWR0141" H 12550 9200 50  0001 C CNN
+F 1 "GND" V 12555 9322 50  0000 R CNN
+F 2 "" H 12550 9450 50  0001 C CNN
+F 3 "" H 12550 9450 50  0001 C CNN
+	1    12550 9450
 	1    0    0    -1
 $EndComp
 Wire Wire Line
-	12600 9400 12600 9300
-Connection ~ 12600 9300
+	12550 9450 12550 9350
+Connection ~ 12550 9350
 $Comp
 L antmicroTVSDiodes:STS321045B502 D15
@@
 Wire Wire Line
 	14650 10000 14650 9900
-Connection ~ 12600 8900
 Wire Wire Line
-	12600 8700 12600 8900
+	11750 8750 11750 8950
 Wire Wire Line
-	12350 8700 12600 8700
-Text GLabel 12350 8700 0    50   Input ~ 0
+	11500 8750 11750 8750
+Text GLabel 11500 8750 0    50   Input ~ 0
 VBAT
+$Comp
+L antmicroCapacitorsmisc:C_100u_0805 C?
+U 1 1 620055D3
+P 12150 9100
+F 0 "C?" H 12265 9145 60  0000 L CNN
+F 1 "C_100u_0805" H 12150 8950 60  0001 C CNN
+F 2 "antmicro-footprints:0805-cap" H 12350 9300 60  0001 L CNN
+F 3 "" H 12150 9100 50  0001 C CNN
+F 4 "MURATA" H 12350 9500 60  0001 L CNN "Manufacturer"
+F 5 "GRM21BR60J107ME15L" H 12350 9400 60  0001 L CNN "MPN"
+F 6 "100u" H 12265 9047 50  0000 L CNN "Val"
+	1    12150 9100
+	1    0    0    -1
+$EndComp
+$Comp
+L antmicroCapacitorsmisc:C_100u_0805 C?
+U 1 1 62006DC2
+P 11750 9100
+F 0 "C?" H 11865 9145 60  0000 L CNN
+F 1 "C_100u_0805" H 11750 8950 60  0001 C CNN
+F 2 "antmicro-footprints:0805-cap" H 11950 9300 60  0001 L CNN
+F 3 "" H 11750 9100 50  0001 C CNN
+F 4 "MURATA" H 11950 9500 60  0001 L CNN "Manufacturer"
+F 5 "GRM21BR60J107ME15L" H 11950 9400 60  0001 L CNN "MPN"
+F 6 "100u" H 11865 9047 50  0000 L CNN "Val"
+	1    11750 9100
+	1    0    0    -1
+$EndComp
+Wire Wire Line
+	11750 8950 12150 8950
+Connection ~ 11750 8950
+Connection ~ 12550 8950
+Connection ~ 12150 8950
+Wire Wire Line
+	12150 8950 12550 8950
+Wire Wire Line
+	12550 9350 12150 9350
+Wire Wire Line
+	11750 9350 11750 9250
+Wire Wire Line
+	12150 9250 12150 9350
+Connection ~ 12150 9350
+Wire Wire Line
+	12150 9350 11750 9350
 $EndSCHEMATC

Commit message: Add local libs to fix CI
Parts:
- BAT1: footprint antmicro-footprints:MS621FE-FL11E -> sa800u-baseboard-hw-footprints:MS621FE-FL11E; symbol antmicroBatteryHoldersClipsContacts:MS621FE-FL11E -> sa800u-baseboard-hw:MS621FE-FL11E
- C92, C? (x2): footprint antmicro-footprints:0805-cap -> sa800u-baseboard-hw-footprints:0805-cap; symbol antmicroCapacitorsmisc:C_100u_0805 -> sa800u-baseboard-hw:C_100u_0805
- C93: footprint antmicro-footprints:0402-cap -> sa800u-baseboard-hw-footprints:0402-cap; symbol antmicroCapacitors0402:C_100n_0402 -> sa800u-baseboard-hw:C_100n_0402
- C94: footprint antmicro-footprints:0402-cap -> sa800u-baseboard-hw-footprints:0402-cap; symbol antmicroCapacitors0402:C_33p_0402 -> sa800u-baseboard-hw:C_33p_0402
- C95: footprint antmicro-footprints:0402-cap -> sa800u-baseboard-hw-footprints:0402-cap; symbol antmicroCapacitors0402:C_10p_0402 -> sa800u-baseboard-hw:C_10p_0402
- D14: footprint antmicro-footprints:RCLAMP2504N.TCT -> sa800u-baseboard-hw-footprints:RCLAMP2504N.TCT; symbol antmicroTVSDiodes:RCLAMP2504N.TCT -> sa800u-baseboard-hw:RCLAMP2504N.TCT
- D15: footprint antmicro-footprints:STS321045B502 -> sa800u-baseboard-hw-footprints:STS321045B502; symbol antmicroTVSDiodes:STS321045B502 -> sa800u-baseboard-hw:STS321045B502
- J7: footprint antmicro-footprints:PinHeader_1x4_P1.27mm_Drill.7mm -> sa800u-baseboard-hw-footprints:PinHeader_1x4_P1.27mm_Drill.7mm; symbol antmicroRectangularConnectorsHeadersMalePins:MC-HVT1-S04-G -> sa800u-baseboard-hw:MC-HVT1-S04-G
- R73, R74, R75, R76: footprint antmicro-footprints:0402-res -> sa800u-baseboard-hw-footprints:0402-res; symbol antmicroResistors0402:R_1k_0402 -> sa800u-baseboard-hw:R_1k_0402
- S1, S2, S3, S4: footprint antmicro-footprints:SW_SPST_4.2x2.8 -> sa800u-baseboard-hw-footprints:SW_SPST_4.2x2.8; symbol antmicroPushbuttonSwitches:KMR2 -> sa800u-baseboard-hw:KMR2
- U10: footprint antmicro-footprints:SA800U-WF -> sa800u-baseboard-hw-footprints:SA800U-WF; symbol antmicroMicrocontrollers:SA800U-WF -> sa800u-baseboard-hw:SA800U-WF

Commit message: annotations
Parts:
- gave numbers to parts that had none: 2
Changed lines of the file:
@@
 VBAT
 $Comp
-L sa800u-baseboard-hw:C_100u_0805 C?
+L sa800u-baseboard-hw:C_100u_0805 C108
 U 1 1 620055D3
 P 12150 9100
-F 0 "C?" H 12265 9145 60  0000 L CNN
+F 0 "C108" H 12265 9145 60  0000 L CNN
 F 1 "C_100u_0805" H 12150 8950 60  0001 C CNN
 F 2 "sa800u-baseboard-hw-footprints:0805-cap" H 12350 9300 60  0001 L CNN
@@
 $EndComp
 $Comp
-L sa800u-baseboard-hw:C_100u_0805 C?
+L sa800u-baseboard-hw:C_100u_0805 C107
 U 1 1 62006DC2
 P 11750 9100
-F 0 "C?" H 11865 9145 60  0000 L CNN
+F 0 "C107" H 11865 9145 60  0000 L CNN
 F 1 "C_100u_0805" H 11750 8950 60  0001 C CNN
 F 2 "sa800u-baseboard-hw-footprints:0805-cap" H 11950 9300 60  0001 L CNN
