File: USB_Hub.sch (KiCad schematic (older format))
At the start: 42 parts

Commit message: added usb c controller and mux, removed hub
Parts:
- removed C? (x5): C_100n_0402, antmicro-footprints:0402-cap, symbol antmicroCapacitors0402:C_100n_0402
- removed C?: C_22u_0603, antmicro-footprints:0603-cap, symbol antmicroCapacitors0603:C_22u_0603
- removed C? (x2): C_10p_0402, antmicro-footprints:0402-cap, symbol antmicroCapacitors0402:C_10p_0402
- removed D? (x3): ESD9L5.0ST5G, antmicro-footprints:DIOM1006X40N, symbol antmicroTVSDiodes:ESD9L5.0ST5G
- removed IC? (x2): HD3SS3220, antmicro-footprints:RNH0030A, symbol antmicroInterfaceControllers:HD3SS3220
- removed J?: WE_632723300011, antmicro-footprints:WE_632723300011, symbol antmicroUSBDVIHDMIConnectors:WE_632723300011
- removed Q?: 2N7000, antmicro-footprints:TO-92-3, symbol antmicroTransistorsFETsMOSFETsSingle:2N7000
- removed R?: R_100k_0402, antmicro-footprints:0402-res, symbol antmicroResistors0402:R_100k_0402
- removed R? (x5): R_1k_0402, antmicro-footprints:0402-res, symbol antmicroResistors0402:R_1k_0402
- removed R?: R_12k_1%_0603, antmicro-footprints:0603-res, symbol antmicroResistors0603:R_12k_1%_0603
- removed R? (x4): R_200k_0402, antmicro-footprints:0402-res, symbol antmicroResistors0402:R_200k_0402
- removed R? (x2): R_4k7_0402, antmicro-footprints:0402-res, symbol antmicroResistors0402:R_4k7_0402
- removed U?: USB57442G, antmicro-footprints:QFN40P700X700X100-57N, symbol antmicroInterfaceControllers:USB57442G
- removed Y?: ECS-1618-250-BN-TR, antmicro-footprints:OSC_ECS-1618-250-BN-TR, symbol antmicroOscillators:ECS-1618-250-BN-TR
- added C? (x5): C_100n_0402, antmicro-footprints:0402-cap, symbol antmicroCapacitors0402:C_100n_0402
- added C? (x4): C_47u_0603, antmicro-footprints:0603-cap, symbol antmicroCapacitors0603:C_47u_0603
- added C?: C_10u_0402, antmicro-footprints:0402-cap, symbol antmicroCapacitors0402:C_10u_0402
- added R?: R_100k_0.5%_0402, antmicro-footprints:0402, symbol antmicroResistors0402:R_100k_0.5%_0402
- added R? (x3): R_100k_0402, antmicro-footprints:0402-res, symbol antmicroResistors0402:R_100k_0402
- added R?: R_200k_0402, antmicro-footprints:0402-res, symbol antmicroResistors0402:R_200k_0402
- added U?: TPS25820DSST, antmicro-footprints:WSON-12_2x3mm, symbol antmicroInterfaceControllers:TPS25820DSST
- added U?: CBTL02043ABQ,115, antmicro-footprints:DHVQFN20, symbol antmicroLogicSignalSwitchesMultiplexersDecoders:CBTL02043ABQ,115
- added U?: TXB0104D, antmicro-footprints:SOIC-14_W3.9mm, symbol antmicroLogicTranslatorsLevelShifters:TXB0104D
Connections:
- net labels added: 5V, USB2C_HS_D_N, USB2C_HS_D_P, USB2C_RX1_N, USB2C_RX1_P, USB2C_RX2_N, USB2C_RX2_P, USB2C_TX1_N, USB2C_TX1_P, USB2C_TX2_N, USB2C_TX2_P, USB2_5V, USB2_CC1, USB2_CC2, USB2_CC_SELECT, USB2_EN, USB2_EN_5V, USB2_FAULT, USB2_FAULT_5V, USB2_HS_D_N, USB2_HS_D_P, USB2_RX_N, USB2_RX_P, USB2_SINK, USB2_SINK_5V, USB2_TX_N, USB2_TX_P
- net labels removed: 1V2, PORT1_HS_D_N, PORT1_HS_D_P, PORT1_RX_N, PORT1_RX_P, PORT1_TX_N, PORT1_TX_P, PORT2_HS_D_N, PORT2_HS_D_P, PORT2_RX1_N, PORT2_RX1_P, PORT2_RX2_N, PORT2_RX2_P, PORT2_RX_N, PORT2_RX_P, PORT2_TX1_N, PORT2_TX1_P, PORT2_TX2_N, PORT2_TX2_P, PORT2_TX_N, PORT2_TX_P, PRT_CTL1, PRT_CTL2, RESET_USBHUB, SPI_CE_N, SPI_DI, USB2_D_N, USB2_D_P, USB2_HUB_SS_RX_N, USB2_HUB_SS_RX_P, USB2_HUB_SS_TX_N, USB2_HUB_SS_TX_P, USBHUB_RESET, USBPORT1_5V, USBPORT2_5V, XTALI_HUB, XTALO_HUB
- wire segments 197 -> 133
- no-connect marks 25 -> 4
Other:
- note removed: "Connect to overcurrent protection."
- note removed: "Data lanes for USB 2.0\n"
- note removed: "USB 3.0 Upstream"
- note removed: "USB3.0 SS RX lines Downstream \n"
- note removed: "USB3.0 SS TX lines Downstream"
- moved on the sheet: C?, D?, J?
