File: sa800u-baseboard-hw.kicad_pcb (KiCad board)
At the start: 2 copper layers, 100 x 70 mm, 171 parts, among them IC1 TPS2378DDA, J1 WE-RJ45_7499111121A, J10 2908-05WB-MG, J11 MC-HVT1-S04-G, J12 MC-HVT1-S04-G, J13 MC-HVT1-S04-G, J14 MC-HVT1-S04-G, J2 46756-1001, J4 WE_632723300011, J5 WE_632723300011, J6 WE_632723300011, J7 3-84952-0, J8 F52R-1A7H1-11020, J9 WE_68715014522, Q1 2N7000, Q2 2N7000, Q3 2N7000, T1 749020010A, U1 RTL8111H, U10 MDT580M01001, U11 AP62301Z6-7, U12 AP62301Z6-7, U13 TPS65982BB, U2 LT9611, U3 TXB0104RUT, U4 TXS0102YZPR, U5 TS3USB30EDGSR, U6 FT2232HL-REEL, U7 USB57442G, U8 SA800U-WF, U9 MAX13042EEBC+T, Y1 ECS-1618-250-BN-TR, Y2 ECS-1618-250-BN-TR

Commit message: Add local libs to fix CI
Parts:
- BAT1: footprint antmicro-footprints:MS621FE-FL11E -> sa800u-baseboard-hw-footprints:MS621FE-FL11E
- C1, C6: footprint antmicro-footprints:1210-cap -> sa800u-baseboard-hw-footprints:1210-cap
- C10, C11, C12, C13, C14, C15, C16, C17, C18, C2, C21, C22, C23, C24, C25, C26, C27, C28, C3, C34, C35, C4, C5, C7, C8, C9: footprint antmicro-footprints:0402-cap -> sa800u-baseboard-hw-footprints:0402-cap
- C19, C20, R14, R20, R25, R38, R41, R57, R58, R59, R60, R61, R62: footprint antmicro-footprints:0603-res -> sa800u-baseboard-hw-footprints:0603-res
- C29, C30, C36: footprint antmicro-footprints:CP_Elec_10x10.5 -> sa800u-baseboard-hw-footprints:CP_Elec_10x10.5
- C31, C33: footprint antmicro-footprints:0805-cap -> sa800u-baseboard-hw-footprints:0805-cap
- C32: footprint antmicro-footprints:KEMET_A -> sa800u-baseboard-hw-footprints:KEMET_A
- D1, D2: footprint antmicro-footprints:SOT-23-3 -> sa800u-baseboard-hw-footprints:SOT-23-3
- D10, D3: footprint antmicro-footprints:DO-214AC -> sa800u-baseboard-hw-footprints:DO-214AC
- D11: footprint antmicro-footprints:SOD-123 -> sa800u-baseboard-hw-footprints:SOD-123
- D4, D5: footprint antmicro-footprints:SOT95P230X110-3N -> sa800u-baseboard-hw-footprints:SOT95P230X110-3N
- D6, D7: footprint antmicro-footprints:PGB1010603MR -> sa800u-baseboard-hw-footprints:PGB1010603MR
- D8, D9: footprint antmicro-footprints:MB10S -> sa800u-baseboard-hw-footprints:MB10S
- FB1, FB2, FB3: footprint antmicro-footprints:0805-res -> sa800u-baseboard-hw-footprints:0805-res
- IC1: footprint antmicro-footprints:SOIC127P600X170-9N -> sa800u-baseboard-hw-footprints:SOIC127P600X170-9N
- J1: footprint antmicro-footprints:7499111121A -> sa800u-baseboard-hw-footprints:7499111121A
- J10: footprint antmicro-footprints:MicroSD_2908-05WB-MG -> sa800u-baseboard-hw-footprints:MicroSD_2908-05WB-MG
- J11, J12, J13, J14: footprint antmicro-footprints:PinHeader_1x4_P1.27mm_Drill.7mm -> sa800u-baseboard-hw-footprints:PinHeader_1x4_P1.27mm_Drill.7mm
- J2: footprint antmicro-footprints:HDMI_Micro-D_Molex_46765-1x01 -> sa800u-baseboard-hw-footprints:HDMI_Micro-D_Molex_46765-1x01
- J4, J5, J6: footprint antmicro-footprints:WE_632723300011 -> sa800u-baseboard-hw-footprints:WE_632723300011
- J7: footprint antmicro-footprints:TE_3-84952-0 -> sa800u-baseboard-hw-footprints:TE_3-84952-0
- J8: footprint antmicro-footprints:F52R-1A7H1-11020 -> sa800u-baseboard-hw-footprints:F52R-1A7H1-11020
- J9: footprint antmicro-footprints:WE_68715014522 -> sa800u-baseboard-hw-footprints:WE_68715014522
- L1, L10, L11, L12, L13, L14, L15, L16, L17, L18, L2, L3, L4, L5, L6, L7, L8, L9: footprint antmicro-footprints:FIL_NFP0QHB242HS2D -> sa800u-baseboard-hw-footprints:FIL_NFP0QHB242HS2D
- MP1, MP2, MP3, MP4: footprint antmicro-footprints:mounting-hole-3mm-NPTH -> sa800u-baseboard-hw-footprints:mounting-hole-3mm-NPTH
- PS1: footprint antmicro-footprints:PDQE30-Q48 -> sa800u-baseboard-hw-footprints:PDQE30-Q48
- Q1, Q2, Q3: footprint antmicro-footprints:TO-92-3 -> sa800u-baseboard-hw-footprints:TO-92-3
- R1, R10, R11, R12, R13, R15, R16, R17, R18, R19, R2, R21, R22, R23, R24, R26, R27, R28, R29, R3, R30, R31, R32, R33, R34, R35, R36, R37, R39, R4, R40, R42, R43, R44, R45, R46, R47, R5, R50, R51, R52, R53, R54, R55, R56, R6, R7, R8, R9: footprint antmicro-footprints:0402-res -> sa800u-baseboard-hw-footprints:0402-res
- S1, S2, S3, S4: footprint antmicro-footprints:SW_SPST_4.2x2.8 -> sa800u-baseboard-hw-footprints:SW_SPST_4.2x2.8
- T1: footprint antmicro-footprints:749020010A -> sa800u-baseboard-hw-footprints:749020010A
- U1: footprint antmicro-footprints:RTL8111H -> sa800u-baseboard-hw-footprints:RTL8111H
- U10: footprint antmicro-footprints:MDT580M01001 -> sa800u-baseboard-hw-footprints:MDT580M01001
- U11, U12: footprint antmicro-footprints:SOT-563 -> sa800u-baseboard-hw-footprints:SOT-563
- U13: footprint USBPD:TPS65982ABZBHR -> sa800u-baseboard-hw-footprints:TPS65982ABZBHR
- U2: footprint antmicro-footprints:LT9611 -> sa800u-baseboard-hw-footprints:LT9611
- U3: footprint antmicro-footprints:Texas_R_PUQFN-N12 -> sa800u-baseboard-hw-footprints:Texas_R_PUQFN-N12
- U4: footprint antmicro-footprints:BGA8C50P2X4_88X188X50N -> sa800u-baseboard-hw-footprints:BGA8C50P2X4_88X188X50N
- U5: footprint antmicro-footprints:MSOP-10_W3mm -> sa800u-baseboard-hw-footprints:MSOP-10_W3mm
- U6: footprint antmicro-footprints:LQFP-64_10x10mm -> sa800u-baseboard-hw-footprints:LQFP-64_10x10mm
- U7: footprint antmicro-footprints:QFN40P700X700X100-57N -> sa800u-baseboard-hw-footprints:QFN40P700X700X100-57N
- U8: footprint antmicro-footprints:SA800U-WF -> sa800u-baseboard-hw-footprints:SA800U-WF
- U9: footprint antmicro-footprints:max13042eebc&plus_t -> sa800u-baseboard-hw-footprints:max13042eebc&plus_t
- Y1, Y2: footprint antmicro-footprints:OSC_ECS-1618-250-BN-TR -> sa800u-baseboard-hw-footprints:OSC_ECS-1618-250-BN-TR
