File: sa800u-baseboard-hw.kicad_pcb (KiCad board)
At the start: 2 copper layers, 100 x 70 mm, 372 parts, among them IC1 TPS2378DDA, IC3 TPS7A0518PDBVT, J1 5-2337992-8, J10 1053091202, J11 WE_632723300011, J12 WE_632723300011, J2 46756-1001, J3 WE_632723300011, J4 WE_632723300011, J5 3-84952-0, J6 F52R-1A7H1-11020, J7 MC-HVT1-S04-G, J8 WE_68715014522, J9 2908-05WB-MG, Q1 2N7000, Q2 2N7000, Q3 2N7000, Q4 2N7000, Q5 BSS84PH6327XTSA2, Q6 IRF7416TRPBF, Q7 IRF7404TRPBF, U1 RTL8111H, U10 SA800U-WF, U11 MAX13042EEBC+T, U12 MDT580M01001, U13 AP62301WU-7, U14 AP62301WU-7, U15 AP62301WU-7, U16 LMV431IM5, U17 AP62301WU-7, U18 STUSB4500QTR, U2 LT9611, U3 TXB0104RUT, U4 TXS0102YZPR, U5 TPS25820DSST, U6 TS3USB30EDGSR, U7 TXB0104D, U8 CBTL02043ABQ,115, U9 FT232RQ-REEL, Y1 ABM8G-25.000MHZ-18-D2Y-T, Y2 ABM8G-24.000MHZ-18-D2Y-T

Commit message: Annotate parts, add 3D model of USB-C plug, update PCB
Parts:
- removed FB1: BLM21PG221SN1D, sa800u-baseboard-hw-footprints:0805-res
- removed MP1, MP2, MP3, MP4: PCB_Spacer_M2, sa800u-baseboard-hw-footprints:9774030243R
- added C126: C_100n_0402, sa800u-baseboard-hw-footprints:0402-cap, F.Cu at (8.85, 131.7)
- added C140: C_100n_0402, sa800u-baseboard-hw-footprints:0402-cap, F.Cu at (-2.66, 168.4)
- added C141: C_100n_0402, sa800u-baseboard-hw-footprints:0402-cap, F.Cu at (0.25, 166.4)
- added C142: C_100n_0402, sa800u-baseboard-hw-footprints:0402-cap, F.Cu at (-5.57, 164.4)
- added C143: C_100n_0402, sa800u-baseboard-hw-footprints:0402-cap, F.Cu at (-5.57, 162.4)
- added C144: C_1u_0402, sa800u-baseboard-hw-footprints:0402-cap, F.Cu at (-37.9, 166.1)
- added C145: C_1u_0402, sa800u-baseboard-hw-footprints:0402-cap, F.Cu at (-35.0, 166.1)
- added C146: C_1u_0402, sa800u-baseboard-hw-footprints:0402-cap, F.Cu at (-37.9, 168.1)
- added C147: C_100n_0402, sa800u-baseboard-hw-footprints:0402-cap, F.Cu at (-5.02, 124.0)
- added C148: C_100n_0402, sa800u-baseboard-hw-footprints:0402-cap, F.Cu at (-21.8, 143.0)
- added C149: C_100u_0805, sa800u-baseboard-hw-footprints:0805-cap, F.Cu at (-31.5, 138.3)
- added C150: C_4u7_0805, antmicro-footprints:0805-cap, F.Cu at (-23.8, 103.9)
- added D27: ASMB-TTF0-0A20B, sa800u-baseboard-hw-footprints:PLCC6_3.5x3.7mm, F.Cu at (32.0, 125.6)
- added D28: ESD144B1W0201E6327XTSA1, sa800u-baseboard-hw-footprints:ESD144B1W0201E6327XTSA1, F.Cu at (44.8, 124.0)
- added FB5: BLM18SG121TN1D, sa800u-baseboard-hw-footprints:0603-res, F.Cu at (3.26, 141.0)
- added FB6: BLM18SG121TN1D, sa800u-baseboard-hw-footprints:0603-res, F.Cu at (-4.45, 155.7)
- added Q10: SQS401EN-T1_BE3, sa800u-baseboard-hw-footprints:Vishay_PowerPAK_1212-8_Single, F.Cu at (-36.6, 139.2)
- added Q8: Si7223DN, sa800u-baseboard-hw-footprints:PowerPak-1212, F.Cu at (169.5, 88.0)
- added Q9: Si7223DN, sa800u-baseboard-hw-footprints:PowerPak-1212, F.Cu at (169.5, 83.0)
- added R119: R_2k_0402, sa800u-baseboard-hw-footprints:0402-res, F.Cu at (0.25, 164.4)
- added R120: R_2k_0402, sa800u-baseboard-hw-footprints:0402-res, F.Cu at (3.16, 162.4)
- added R121: R_100k_0402, sa800u-baseboard-hw-footprints:0402-res, F.Cu at (36.5, 124.0)
- added R122: R_100k_0402, sa800u-baseboard-hw-footprints:0402-res, F.Cu at (30.4, 131.1)
- added R123: R_100k_0402, sa800u-baseboard-hw-footprints:0402-res, F.Cu at (33.3, 129.1)
- added R124: R_100k_0402, sa800u-baseboard-hw-footprints:0402-res, F.Cu at (30.4, 129.1)
- added R125: R_4k7_0402, sa800u-baseboard-hw-footprints:0402-res, F.Cu at (39.4, 124.0)
- added R126: R_4k7_0402, sa800u-baseboard-hw-footprints:0402-res, F.Cu at (33.3, 131.1)
- added R127: R_4k7_0402, sa800u-baseboard-hw-footprints:0402-res, F.Cu at (36.2, 129.1)
- added R128: R_4k7_0402, sa800u-baseboard-hw-footprints:0402-res, F.Cu at (39.4, 126.0)
- added R129: R_4k7_0402, sa800u-baseboard-hw-footprints:0402-res, F.Cu at (42.3, 124.0)
- added R130: R_4k7_0402, sa800u-baseboard-hw-footprints:0402-res, F.Cu at (36.2, 131.1)
- added R131: R_100R_0402, sa800u-baseboard-hw-footprints:0402-res, F.Cu at (39.1, 128.0)
- added R132: R_150R_0402, sa800u-baseboard-hw-footprints:0402-res, F.Cu at (42.3, 126.0)
- added R133: R_590R_0402, sa800u-baseboard-hw-footprints:0402-res, F.Cu at (36.5, 126.0)
- added R134: R_510R_0402, antmicro-footprints:0402-res, F.Cu at (-1.22, 155.9)
- added R135: R_200k_0402, antmicro-footprints:0402-res, F.Cu at (-8.68, 133.5)
- added R136: R_39k_0402, antmicro-footprints:0402-res, F.Cu at (-14.5, 135.5)
- added R137: R_13k7_0402, antmicro-footprints:0402-res, F.Cu at (-18.9, 143.0)
- added R138: R_200k_0402, antmicro-footprints:0402-res, F.Cu at (-14.5, 137.5)
- added R139: R_39k_0402, antmicro-footprints:0402-res, F.Cu at (-5.02, 128.0)
- added R140: R_13k7_0402, antmicro-footprints:0402-res, F.Cu at (-11.6, 133.5)
- added R141: R_200k_0402, antmicro-footprints:0402-res, F.Cu at (-5.02, 126.0)
- added R142: R_39k_0402, antmicro-footprints:0402-res, F.Cu at (-34.0, 143.3)
- added R143: R_13k7_0402, antmicro-footprints:0402-res, F.Cu at (-24.8, 143.0)
- added R144: R_255k_0402, sa800u-baseboard-hw-footprints:0402-res, F.Cu at (-31.1, 143.3)
- added R145: R_10k_0402, sa800u-baseboard-hw-footprints:0402-res, F.Cu at (-28.2, 143.3)
- added R146: R_10k_0402, sa800u-baseboard-hw-footprints:0402-res, F.Cu at (-5.02, 130.0)
- added R147: R_10k_0402, sa800u-baseboard-hw-footprints:0402-res, F.Cu at (-14.5, 139.5)
- added R148: R_10k_0402, sa800u-baseboard-hw-footprints:0402-res, F.Cu at (-11.6, 137.5)
- added R149: R_10k_0402, sa800u-baseboard-hw-footprints:0402-res, F.Cu at (-16.0, 143.0)
- added R150: R_10k_0402, sa800u-baseboard-hw-footprints:0402-res, F.Cu at (-8.68, 135.5)
- added R151: R_10k_0402, sa800u-baseboard-hw-footprints:0402-res, F.Cu at (-5.77, 133.5)
- added R152: R_10k_0402, sa800u-baseboard-hw-footprints:0402-res, F.Cu at (-11.6, 139.5)
- added R153: R_10k_0402, sa800u-baseboard-hw-footprints:0402-res, F.Cu at (-27.6, 137.9)
- added R154: R_75k_0402, antmicro-footprints:0402-res, F.Cu at (-11.6, 135.5)
- added R155: R_0R_0603, antmicro-footprints:0603-res, F.Cu at (-19.6, 100.8)
- added R156: R_0R_0603, antmicro-footprints:0603-res, F.Cu at (-24.4, 106.6)
- added R157: R_0R_0402, sa800u-baseboard-hw-footprints:0402-res, F.Cu at (-11.7, 100.5)
- added SP2: 9774060151, antmicro-footprints:9774060151, B.Cu at (151.5, 85.5)
- added SP3: 9774060151, antmicro-footprints:9774060151, B.Cu at (151.5, 148.5)
- added SP4: 9774060151, antmicro-footprints:9774060151, B.Cu at (65.0, 148.0)
- added SP5: 9774060151, antmicro-footprints:9774060151, B.Cu at (65.0, 86.0)
- added U19: NTS0102GT, sa800u-baseboard-hw-footprints:PSON50P100X195X50-8N, F.Cu at (-8.32, 163.2)
- added U20: NTS0102GT, sa800u-baseboard-hw-footprints:PSON50P100X195X50-8N, F.Cu at (-8.32, 166.8)
- added U21: LTC4417IUF, sa800u-baseboard-hw-footprints:LTC4417IUF-TRPBF, F.Cu at (176.0, 89.5)
- added U22: AP2114H-3_3TRG1, antmicro-footprints:SOT-223, F.Cu at (-30.2, 104.5)
- C100, C121, C99: moved to F.Cu
- C106: value C_47u_ELEC_100V -> C_4u7_0805; footprint sa800u-baseboard-hw-footprints:CP_Elec_10x10.5 -> antmicro-footprints:0805-cap; moved to F.Cu
- C96: value C_1u_0402 -> C_4u7_0402
- D10, D8, D9: value ESD9L5.0ST5G -> TPD4E05U06_PASS; footprint sa800u-baseboard-hw-footprints:DIOM1006X40N -> sa800u-baseboard-hw-footprints:TPD4E05U06_PASS
- D11, D13: value TPD1E10B06DPYR -> KP-1608EC; footprint sa800u-baseboard-hw-footprints:XDFN-2_1x0.60mm -> antmicro-footprints:LED_0603
- D19: value BZT52C12 -> KP-1608EC; footprint sa800u-baseboard-hw-footprints:SOD-123 -> antmicro-footprints:LED_0603; moved to F.Cu
- D7: value ESD9L5.0ST5G -> 1N4148WS; footprint sa800u-baseboard-hw-footprints:DIOM1006X40N -> sa800u-baseboard-hw-footprints:SOD-323F
- J5: value 3-84952-0 -> 1-1734248-5; footprint sa800u-baseboard-hw-footprints:TE_3-84952-0 -> sa800u-baseboard-hw-footprints:TE_1-1734248-5; moved to F.Cu
- J6, L14, L15, L16, L17, L18, R83, R84: moved to B.Cu
- Q1, Q2, Q3, Q4: value 2N7000 -> BSS138APW; footprint sa800u-baseboard-hw-footprints:TO-92-3 -> sa800u-baseboard-hw-footprints:SC70-3
- Q6: value IRF7416TRPBF -> Si7223DN; footprint sa800u-baseboard-hw-footprints:IRF7416TRPBF -> sa800u-baseboard-hw-footprints:PowerPak-1212
- R1: value R_10k_0402 -> R_1k_0402; footprint sa800u-baseboard-hw-footprints:0402-res -> antmicro-footprints:0402-res
- R2, R3: value R_10k_0402 -> R_0R_0402; footprint sa800u-baseboard-hw-footprints:0402-res -> antmicro-footprints:0402-res
- R22: value R_10k_0603 -> R_10k_0402; footprint sa800u-baseboard-hw-footprints:0603-res -> sa800u-baseboard-hw-footprints:0402-res
- R28: value R_7k68_0603 -> R_0R_0402; footprint sa800u-baseboard-hw-footprints:0603-res -> antmicro-footprints:0402-res
- R37, R48: value R_120k_0402 -> R_2k_0402
- R38, R47: value R_10k_0603 -> R_2k_0402; footprint sa800u-baseboard-hw-footprints:0603-res -> sa800u-baseboard-hw-footprints:0402-res
- R49, R50: value R_2k2_0402 -> R_2k_0402
- R52: value R_510R_0603 -> R_7k68_0603
- R54, R56, R57, R58, R60, R61, R62: value R_510R_0603 -> R_510R_0402; footprint sa800u-baseboard-hw-footprints:0603-res -> antmicro-footprints:0402-res
- R71, R72: value R_4k7_0402 -> R_2k_0402
- R77, R79, R80, R81, R82: value R_0R_0603 -> R_2k_0402; footprint sa800u-baseboard-hw-footprints:0603-res -> sa800u-baseboard-hw-footprints:0402-res
- R78: value R_1M_0603 -> R_2k_0402; footprint sa800u-baseboard-hw-footprints:0603-res -> sa800u-baseboard-hw-footprints:0402-res
- R8: value R_25k_1%_0402 -> R_0R_0402; footprint sa800u-baseboard-hw-footprints:0402 -> antmicro-footprints:0402-res
- R87: value R_7k5_2512 -> R_7k5_0402; footprint sa800u-baseboard-hw-footprints:2512-res -> sa800u-baseboard-hw-footprints:0402-res
- U11: value MAX13042EEBC+T -> NTS0102GT; footprint sa800u-baseboard-hw-footprints:max13042eebc&plus_t -> sa800u-baseboard-hw-footprints:PSON50P100X195X50-8N
- U4: value TXS0102YZPR -> NTS0102GT; footprint sa800u-baseboard-hw-footprints:BGA8C50P2X4_88X188X50N -> sa800u-baseboard-hw-footprints:PSON50P100X195X50-8N
- U6: value TS3USB30EDGSR -> FSUSB30MUX
- moved R3 297.3 mm to (-18.0, 148.3), turned to 0 degrees
- moved R2 289.5 mm to (-23.9, 150.3), turned to 0 degrees
- moved R8 288.2 mm to (-20.9, 148.3), turned to 0 degrees
- moved R81 260.4 mm to (-5.57, 168.4)
- moved R111 260.3 mm to (262.4, 169.9)
- moved C127 260.3 mm to (255.8, 174.7)
- moved C128 260.3 mm to (254.7, 166.8)
- moved C136 260.3 mm to (255.2, 170.6)
- moved C137 260.3 mm to (255.2, 171.6)
- moved C138 260.3 mm to (255.2, 169.6)
- moved C139 260.3 mm to (264.3, 169.9)
- moved D23 260.3 mm to (258.8, 173.8)
- moved D24 260.3 mm to (252.3, 167.1)
- moved Q7 260.3 mm to (265.1, 163.6)
- moved R106 260.3 mm to (253.2, 168.6)
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Connections:
- net /SoM/GPIO_49 renamed GPIO_49
- net /SoM/I2C10_SCL renamed I2C10_SCL
- net /SoM/I2C10_SDA renamed I2C10_SDA
- net /USB-PD/STUSB4500_DISCHARGE renamed Net-(R111-Pad2)
- net 1V2 renamed 1V2_SYS
- net I2S_D0_SPDIF renamed /HDMI_converter/I2S_D0_SPDIF
- net I2S_MCLK renamed /HDMI_converter/I2S_MCLK
- net I2S_SCLK renamed /HDMI_converter/I2S_SCLK
- net I2S_WS renamed /HDMI_converter/I2S_WS
- net LT9611_VCC12_RX renamed /HDMI_converter/LT9611_VCC12_RX
- net LT9611_VCC12_TX renamed /HDMI_converter/LT9611_VCC12_TX
- net LT9611_VDD12 renamed /HDMI_converter/LT9611_VDD12
- net Net-(C101-Pad2) renamed /PoE/VSS_POE
- net Net-(C139-Pad1) renamed PD_VDD
- net Net-(C90-Pad2) renamed /USB-C_Interface /USB_SBU2_1
- net Net-(C91-Pad2) renamed /USB-C_Interface /USB_SBU_1_2
- net Net-(IC1-Pad2) renamed /PoE/DEN
- net Net-(IC1-Pad3) renamed /PoE/CLS
- net Net-(IC1-Pad6) renamed /PoE/CDB
- net Net-(PS1-Pad5) renamed /PoE/TRIM
- net Net-(R95-Pad2) renamed /PSU/5V_DC_DC_ENABLE
- net USB2_5V renamed /USB-C_Interface /USB2_5V
- C100 pad 1: Net-(C100-Pad1) -> /PoE/VDD_POE
- C102 pad 1: VDD -> 5V_POE
- C103 pad 1: VDD -> 5V_POE
- C104 pad 1: VDD -> 5V_POE
- C105 pad 1: VDD -> 5V_POE
- C106 pad 1: /PoE/VDD_POE -> 5V_SYS
- C106 pad 2: GNDD -> GND
- C11 pad 1: 5V -> VDD
- C111 pad 1: 5V -> 5V_SYS
- C112 pad 1: 5V -> 5V_SYS
- C114 pad 1: 3V3 -> 3V8_SYS
- C115 pad 1: 1V8 -> 3V3_SYS
- C117 pad 1: 3V3 -> 3V8_SYS
- C118 pad 1: 1V8 -> 3V3_SYS
- C120 pad 1: 3V3 -> 3V3_SYS
- C121 pad 1: 3V3 -> LVS1A_1V8
- C13 pad 1: 5V -> VDD
- C136 pad 1: /USB-PD/2V7 -> GND
- C136 pad 2: GND -> /USB-PD/VREG_1V2
- C137 pad 1: /USB-PD/PD_VBUS -> /USB-PD/STUSB_VDD
- C138 pad 1: Net-(C138-Pad1) -> /USB-PD/VREG_2V7
- C18 pad 1: /Ethernet_Controller/ETH_1V0 -> Net-(C18-Pad1)
- C2 pad 1: 3V3 -> /Ethernet_Controller/ETH_3V3
- C22 pad 1: LT9611_VCC33_IO -> /HDMI_converter/LT9611_VCC33_IO
- C23 pad 1: LT9611_VCC33_IO -> /HDMI_converter/LT9611_VCC33_IO
- C24 pad 1: LT9611_VCC33_IO -> /HDMI_converter/LT9611_VCC33_IO
- C25 pad 1: LT9611_VCC33_IO -> /HDMI_converter/LT9611_VCC33_IO
- C26 pad 1: LT9611_VCC33_RX -> /HDMI_converter/LT9611_VCC33_RX
- C27 pad 1: LT9611_VCC33_RX -> /HDMI_converter/LT9611_VCC33_RX
- C28 pad 1: RST_N -> /HDMI_converter/RST_N
- C29 pad 1: LT9611_VCC33_RX -> /HDMI_converter/LT9611_VCC33_RX
- C3 pad 1: 3V3 -> /Ethernet_Controller/ETH_3V3
- C30 pad 1: LT9611_VCC33_RX -> /HDMI_converter/LT9611_VCC33_RX
- C31 pad 1: LT9611_VCC33_TX -> /HDMI_converter/LT9611_VCC33_TX
- C32 pad 1: LT9611_VCC33_TX -> /HDMI_converter/LT9611_VCC33_TX
- C4 pad 1: 3V3 -> /Ethernet_Controller/ETH_3V3
- C42 pad 1: 1V8 -> 3V3_SYS
- C43 pad 1: /HDMI_converter/XTALI -> /HDMI_converter/XTALO
- C46 pad 2: 3V3 -> VREG_S4A_1V8
- C47 pad 1: /HDMI_converter/XTALO -> /HDMI_converter/XTALI
- C48 pad 1: 1V8 -> /Ethernet_Controller/ETH_3V3
- C49 pad 2: TX_CLK_N -> /HDMI_converter/TX_D2_P
- C5 pad 1: 3V3 -> /Ethernet_Controller/ETH_3V3
- C50 pad 2: TX_CLK_P -> /HDMI_converter/TX_D2_N
- C51 pad 2: TX_D0_N -> /HDMI_converter/TX_D1_P
- C52 pad 2: TX_D0_P -> /HDMI_converter/TX_D1_N
- C53 pad 2: TX_D1_N -> /HDMI_converter/TX_D0_P
- C54 pad 2: TX_D1_P -> /HDMI_converter/TX_D0_N
- C55 pad 2: TX_D2_N -> /HDMI_converter/TX_CLK_P
- C56 pad 2: TX_D2_P -> /HDMI_converter/TX_CLK_N
- C57 pad 1: VCOM -> /HDMI_converter/VCOM
- C60 pad 1: 5V -> 5V_SYS
- C61 pad 1: 5V -> 5V_SYS
- C62 pad 1: 5V -> 5V_SYS
- C63 pad 1: 5V -> 5V_SYS
- C66 pad 1: USB_VBUS -> Net-(C66-Pad1)
- C68 pad 1: USB_VBUS -> GND
- C68 pad 2: GND -> USB_VBUS
- C84 pad 1: 3V3 -> 3V3_SYS
- C85 pad 1: 3V3 -> 3V3_SYS
- C86 pad 1: 3V3 -> 3V3_SYS
- C87 pad 1: 3V3 -> 3V3_SYS
- C88 pad 1: 1V8 -> 1V8_SYS
- C89 pad 1: 5V -> 5V_SYS
- C9 pad 1: 5V -> VDD
- C96 pad 1: 3V3 -> /Ethernet_Controller/ETH_3V3
- C97 pad 1: 3V3 -> VREG_S4A_1V8
- C98 pad 1: 1V8 -> 3V3_SYS
- C99 pad 1: Net-(C100-Pad1) -> /PoE/VDD_POE
- D11 pad 1: /USB-C_Interface /USB_CC1 -> AUX_VDD_VALID
- D13 pad 1: /USB-C_Interface /USB_CC2 -> PD_VDD_VALID
- D23 pad 1: Net-(D23-Pad1) -> /USB-PD/PD_CC2
- D23 pad 2: Net-(D23-Pad2) -> /USB-PD/PD_CC1
- D26 pad A: 5V -> (no net)
- D3 pad A: 3V3 -> 3V3_SYS
- D7 pad A: GND -> /HDMI_converter/5V_HDMI_FB_D
- IC1 pad 8: (no net) -> /PoE/APD
- J10 pad 1: (no net) -> /PSU/AUX_VDD
- J11 pad A5: Net-(D23-Pad1) -> /USB-PD/PD_CC1
- J11 pad B5: Net-(D23-Pad2) -> /USB-PD/PD_CC2
- J2 pad 19: 5V -> /HDMI_converter/5V_HDMI
- J3 pad A10: USB_VBUS -> Net-(C66-Pad1)
- J3 pad A5: /USB-C_Interface /USB_CC1 -> /USB-C_Interface /USB1_CC1
- J3 pad A8: /USB-C_Interface /USB_SBU1 -> (no net)
- J3 pad B5: /USB-C_Interface /USB_CC2 -> /USB-C_Interface /USB1_CC2
- J3 pad B8: /USB-C_Interface /USB_SBU2 -> (no net)
- J5 pad 11: TP_I2C_SCL -> /LCM/TP_I2C_SCL_3V3
- J5 pad 12: TP_I2C_SDA -> /LCM/TP_I2C_SDA_3V3
- J5 pad 14: 3V3 -> 3V3_SYS
- J5 pad 15: 3V3 -> 3V3_SYS
- J6 pad 17: TP_I2C_SCL -> /LCM/TP_I2C_SCL_3V3
- J6 pad 18: TP_I2C_SDA -> /LCM/TP_I2C_SDA_3V3
- J6 pad 20: 3V3 -> 3V3_SYS
- J7 pad 1: /SoM/GPIO_25 -> (no net)
- J8 pad 39: /Cameras_Interface/CAM0_SDA -> (no net)
- J8 pad 40: /Cameras_Interface/CAM0_SCL -> (no net)
- J8 pad 41: /Cameras_Interface/CAM1_SDA -> (no net)
- J8 pad 42: /Cameras_Interface/CAM1_SCL -> (no net)
- J8 pad 47: Net-(J8-Pad47) -> /Cameras_Interface/3V3_CAM
- J8 pad 48: Net-(J8-Pad47) -> /Cameras_Interface/3V3_CAM
- J8 pad 49: 5V -> 5V_SYS
- J8 pad 50: 5V -> 5V_SYS
- L1 pad 1: 3V3 -> 3V3_SYS
- L1 pad 2: LT9611_VCC33_IO -> /HDMI_converter/LT9611_VCC33_IO
- L2 pad 1: 3V3 -> 3V3_SYS
- L2 pad 2: LT9611_VCC33_RX -> /HDMI_converter/LT9611_VCC33_RX
- L29 pad 1: Net-(C110-Pad1) -> Net-(C110-Pad2)
- L29 pad 2: 5V -> 5V_SYS
- L3 pad 1: 3V3 -> 3V3_SYS
- L3 pad 2: LT9611_VCC33_TX -> /HDMI_converter/LT9611_VCC33_TX
- L30 pad 2: 3V3 -> 3V8_SYS
- L31 pad 2: 1V8 -> 3V3_SYS
- PS1 pad 3: Net-(C100-Pad1) -> /PoE/VDD_POE
- PS1 pad 4: VDD -> 5V_POE
- Q1 pad 1: CEC_GPIO6 -> VREG_S4A_1V8
- Q1 pad 2: Net-(Q1-Pad2) -> LT9611_GPIO5
- Q1 pad 3: /HDMI_converter/CEC_HDMI -> /HDMI_converter/INTO_GPIO5
- Q2 pad 1: LT9611_GPIO5 -> VREG_S4A_1V8
- Q2 pad 2: 1V8 -> LT9611_RST
- Q2 pad 3: INTO_GPIO5 -> /HDMI_converter/RST_N
- Q3 pad 1: LT9611_RST -> Net-(Q3-Pad1)
- Q3 pad 2: 1V8 -> /HDMI_converter/LT_CEC
- Q3 pad 3: RST_N -> /HDMI_converter/CEC_HDMI
- Q4 pad 1: GND -> Net-(Q4-Pad1)
- Q4 pad 2: Net-(Q4-Pad2) -> GND
- Q4 pad 3: VCOM -> /HDMI_converter/VCOM
- Q5 pad 2: Net-(Q5-Pad2) -> /PSU/BYPASS_EN
- Q6 pad 1: VDD -> /PSU/VS1
- Q6 pad 2: VDD -> Net-(C18-Pad1)
- Q6 pad 3: VDD -> /PSU/VS1
- Q6 pad 4: Net-(Q5-Pad2) -> Net-(C18-Pad1)
- Q6 pad 5: 5V -> VDD
- Q6 pad 6: 5V -> VDD
- Q6 pad 7: 5V -> /PSU/AUX_VDD
- Q6 pad 8: 5V -> /PSU/AUX_VDD
- R1 pad 1: (no net) -> Net-(R1-Pad1)
- R1 pad 2: Net-(R1-Pad2) -> GND
- R100 pad 1: 3V3 -> 3V3_SYS
- R101 pad 1: 3V3 -> 3V3_SYS
- R102 pad 1: 3V3 -> 3V3_SYS
- R103 pad 1: 3V3 -> 3V3_SYS
- R104 pad 1: 1V8 -> VREG_S4A_1V8
- R11 pad 1: 1V8 -> VREG_S4A_1V8
- R11 pad 2: /Ethernet_Controller/PCIE1_WAKE_N -> PCIE1_WAKE_N
- R12 pad 1: 1V8 -> VREG_S4A_1V8
- R12 pad 2: /Ethernet_Controller/PCIE1_RST_N -> PCIE1_CLKREQ_N
- R13 pad 1: 1V8 -> VREG_S4A_1V8
- R13 pad 2: /Ethernet_Controller/PCIE1_CLKREQ_N -> PCIE1_RST_N
- R14 pad 1: 3V3 -> 3V3_SYS
- R15 pad 1: /Ethernet_Controller/XTAL1 -> /Ethernet_Controller/XTAL2
- R15 pad 2: /Ethernet_Controller/XTAL2 -> /Ethernet_Controller/XTAL1
- R17 pad 2: 3V3 -> /Ethernet_Controller/ETH_3V3
- R18 pad 2: 3V3 -> /Ethernet_Controller/ETH_3V3
- R19 pad 1: 3V3 -> 3V3_SYS
- R19 pad 2: Net-(Q1-Pad2) -> Net-(Q3-Pad1)
- R2 pad 1: (no net) -> GND
- R20 pad 1: CEC_GPIO6 -> /HDMI_converter/CEC_HDMI
- R20 pad 2: /HDMI_converter/CEC_HDMI -> /HDMI_converter/LT_CEC
- R22 pad 1: 3V3 -> 3V3_SYS
- R22 pad 2: RST_N -> /HDMI_converter/RST_N
- R23 pad 1: 3V3 -> 3V3_SYS
- R23 pad 2: HDMIOUT_SCL -> /HDMI_converter/INTO_GPIO5
- R24 pad 1: 3V3 -> 3V3_SYS
- R24 pad 2: HDMIOUT_SDA -> /HDMI_converter/HDMIOUT_SCL
- R25 pad 1: 3V3 -> 3V3_SYS
- R25 pad 2: INTO_GPIO5 -> /HDMI_converter/HDMIOUT_SDA
- R26 pad 1: 1V8 -> VREG_S4A_1V8
- R27 pad 1: 1V8 -> VREG_S4A_1V8
- R29 pad 1: 3V3 -> 3V3_SYS
- R29 pad 2: INTO_GPIO5 -> /HDMI_converter/INTO_GPIO5
- R3 pad 1: (no net) -> GND
- R30 pad 1: 3V3 -> 3V3_SYS
- R30 pad 2: RST_N -> /HDMI_converter/RST_N
- R31 pad 1: 5V -> 5V_SYS
- R32 pad 1: 5V -> 5V_SYS
- R35 pad 1: 3V3 -> 3V3_SYS
- R37 pad 1: GND -> I2C4_SCL
- R37 pad 2: Net-(R37-Pad2) -> VREG_S4A_1V8
- R38 pad 1: GND -> I2C4_SDA
- R38 pad 2: Net-(R37-Pad2) -> VREG_S4A_1V8
- R39 pad 1: 3V3 -> /HDMI_converter/LT9611_VCC33_TX
- R39 pad 2: TX_D2_P -> /HDMI_converter/TX_CLK_N
- R4 pad 1: 3V3 -> 3V3_SYS
- R40 pad 1: /HDMI_converter/XTALI -> /HDMI_converter/XTALO
- R40 pad 2: /HDMI_converter/XTALO -> /HDMI_converter/XTALI
- R41 pad 1: 3V3 -> /HDMI_converter/LT9611_VCC33_TX
- R41 pad 2: TX_D2_N -> /HDMI_converter/TX_CLK_P
- R42 pad 1: 3V3 -> /HDMI_converter/LT9611_VCC33_TX
- R42 pad 2: TX_D1_P -> /HDMI_converter/TX_D0_N
- R43 pad 1: 3V3 -> /HDMI_converter/LT9611_VCC33_TX
- R43 pad 2: TX_D1_N -> /HDMI_converter/TX_D0_P
- R44 pad 1: 3V3 -> /HDMI_converter/LT9611_VCC33_TX
- R44 pad 2: TX_D0_P -> /HDMI_converter/TX_D1_N
- R45 pad 1: 3V3 -> /HDMI_converter/LT9611_VCC33_TX
- R45 pad 2: TX_D0_N -> /HDMI_converter/TX_D1_P
- R46 pad 1: 3V3 -> /HDMI_converter/LT9611_VCC33_TX
- R46 pad 2: TX_CLK_P -> /HDMI_converter/TX_D2_N
- R47 pad 1: 1V8 -> /HDMI_converter/HDMIOUT_SDA
- R47 pad 2: Net-(R47-Pad2) -> 3V3_SYS
- R48 pad 1: Net-(R47-Pad2) -> /HDMI_converter/HDMIOUT_SCL
- R48 pad 2: GND -> 3V3_SYS
- R49 pad 1: 1V8 -> TP_I2C_SDA
- R49 pad 2: I2C4_SDA -> LVS1A_1V8
- R5 pad 1: GND -> Net-(R5-Pad1)
- R5 pad 2: Net-(R5-Pad2) -> GND
- R50 pad 1: 1V8 -> TP_I2C_SCL
- R50 pad 2: I2C4_SCL -> LVS1A_1V8
- R51 pad 1: 3V3 -> /HDMI_converter/LT9611_VCC33_TX
- R51 pad 2: TX_CLK_N -> /HDMI_converter/TX_D2_P
- R52 pad 1: /HDMI_converter/HDMI_TX2_P -> Net-(R52-Pad1)
- R52 pad 2: VCOM -> GND
- R53 pad 1: 5V -> /HDMI_converter/5V_HDMI
- R54 pad 1: /HDMI_converter/HDMI_TX2_N -> /HDMI_converter/HDMI_CLK_N
- R54 pad 2: VCOM -> /HDMI_converter/VCOM
- R56 pad 1: /HDMI_converter/HDMI_TX1_P -> /HDMI_converter/HDMI_CLK_P
- R56 pad 2: VCOM -> /HDMI_converter/VCOM
- R57 pad 1: /HDMI_converter/HDMI_TX1_N -> /HDMI_converter/HDMI_TX0_N
- R57 pad 2: VCOM -> /HDMI_converter/VCOM
- R58 pad 2: VCOM -> /HDMI_converter/VCOM
- R59 pad 1: 3V3 -> 3V3_SYS
- R59 pad 2: Net-(Q4-Pad2) -> Net-(Q4-Pad1)
- R60 pad 1: /HDMI_converter/HDMI_TX0_N -> /HDMI_converter/HDMI_TX1_N
- R60 pad 2: VCOM -> /HDMI_converter/VCOM
- R61 pad 1: /HDMI_converter/HDMI_CLK_P -> /HDMI_converter/HDMI_TX1_P
- R61 pad 2: VCOM -> /HDMI_converter/VCOM
- R62 pad 1: /HDMI_converter/HDMI_CLK_N -> /HDMI_converter/HDMI_TX2_N
- R62 pad 2: VCOM -> /HDMI_converter/VCOM
- R64 pad 2: 5V -> 5V_SYS
- R65 pad 2: 5V -> 5V_SYS
- R66 pad 2: 5V -> 5V_SYS
- R68 pad 2: 1V8 -> VREG_S4A_1V8
- R70 pad 2: 3V3 -> 3V3_SYS
- R71 pad 1: TP_I2C_SDA -> /LCM/TP_I2C_SCL_3V3
- R71 pad 2: 3V3 -> 3V3_SYS
- R72 pad 1: TP_I2C_SCL -> /LCM/TP_I2C_SDA_3V3
- R72 pad 2: 3V3 -> 3V3_SYS
- R77 pad 1: 1V8 -> CCI1_I2C_SDA
- R77 pad 2: Net-(R77-Pad2) -> LVS1A_1V8
- R78 pad 1: Net-(R77-Pad2) -> CCI0_I2C_SDA
- R78 pad 2: GND -> LVS1A_1V8
- R79 pad 1: CCI0_I2C_SCL -> CCI1_I2C_SCL
- R79 pad 2: /Cameras_Interface/CAM0_SCL -> LVS1A_1V8
- R8 pad 1: 1V8 -> GND
- R80 pad 1: CCI0_I2C_SDA -> CCI0_I2C_SCL
- R80 pad 2: /Cameras_Interface/CAM0_SDA -> LVS1A_1V8
- R81 pad 1: CCI1_I2C_SCL -> /Cameras_Interface/CCI1_I2C_SCL_3V3
- R81 pad 2: /Cameras_Interface/CAM1_SCL -> /Cameras_Interface/3V3_CAM
- R82 pad 1: CCI1_I2C_SDA -> /Cameras_Interface/CCI0_I2C_SCL_3V3
- R82 pad 2: /Cameras_Interface/CAM1_SDA -> /Cameras_Interface/3V3_CAM
- R85 pad 2: VDD -> 5V_POE
- R87 pad 1: VDD -> GNDD
- R87 pad 2: GNDD -> (no net)
- R9 pad 2: Net-(R8-Pad2) -> Net-(R154-Pad2)
- R95 pad 1: Net-(Q5-Pad2) -> /PSU/BYPASS_EN
- R97 pad 1: 5V -> 5V_SYS
- U1 pad 11: 3V3 -> /Ethernet_Controller/ETH_3V3
- U1 pad 12: /Ethernet_Controller/PCIE1_CLKREQ_N -> PCIE1_CLKREQ_N
- U1 pad 19: /Ethernet_Controller/PCIE1_RST_N -> PCIE1_RST_N
- U1 pad 21: /Ethernet_Controller/PCIE1_WAKE_N -> PCIE1_WAKE_N
- U1 pad 23: 3V3 -> /Ethernet_Controller/ETH_3V3
- U1 pad 31: Net-(R5-Pad2) -> Net-(R5-Pad1)
- U1 pad 32: 3V3 -> /Ethernet_Controller/ETH_3V3
- U10 pad 1_107: (no net) -> PCIE1_RST_N
- U10 pad 1_109: (no net) -> PCIE1_CLKREQ_N
- U10 pad 1_111: (no net) -> PCIE1_WAKE_N
- U10 pad 1_134: (no net) -> Net-(R1-Pad1)
- U10 pad 1_149: (no net) -> LVS1A_1V8
- U10 pad 1_159: VBAT -> 3V8_SYS
- U10 pad 1_160: VBAT -> 3V8_SYS
- U10 pad 1_161: VBAT -> 3V8_SYS
- U10 pad 1_162: VBAT -> 3V8_SYS
- U10 pad 1_163: VBAT -> 3V8_SYS
- U10 pad 1_164: VBAT -> 3V8_SYS
- U10 pad 1_165: VBAT -> 3V8_SYS
- U10 pad 1_166: VBAT -> 3V8_SYS
- U10 pad 1_167: VBAT -> 3V8_SYS
- U10 pad 1_168: VBAT -> 3V8_SYS
- U10 pad 2_124: 1V8 -> VREG_S4A_1V8
- U10 pad 2_126: 1V8 -> VREG_S4A_1V8
- U10 pad 2_128: 1V8 -> VREG_S4A_1V8
- U10 pad 2_148: 1V8 -> (no net)
- U10 pad 2_159: CS_N -> (no net)
- U10 pad 2_163: CS_N -> (no net)
- U10 pad 2_165: CS_N -> (no net)
- U10 pad 2_2: /SoM/GPIO_25 -> (no net)
- U12 pad 12: 3V3 -> 3V3_SYS
- U12 pad 14: 3V3 -> 3V3_SYS
- U12 pad 16: 3V3 -> 3V3_SYS
- U12 pad 18: 3V3 -> 3V3_SYS
- U12 pad 2: 3V3 -> 3V3_SYS
- U12 pad 4: 3V3 -> 3V3_SYS
- U12 pad 70: 3V3 -> 3V3_SYS
- U12 pad 72: 3V3 -> 3V3_SYS
- U12 pad 74: 3V3 -> 3V3_SYS
- U13 pad 3: 5V -> VDD
- U13 pad 4: Net-(R4-Pad2) -> Net-(R154-Pad2)
- U13 pad 5: Net-(R1-Pad2) -> Net-(R151-Pad2)
- U14 pad 3: 5V -> VDD
- U14 pad 4: Net-(R8-Pad2) -> Net-(R4-Pad2)
- U14 pad 5: Net-(R2-Pad2) -> Net-(R148-Pad2)
- U15 pad 3: 5V -> VDD
- U15 pad 5: Net-(R3-Pad2) -> Net-(R149-Pad2)
- U17 pad 2: Net-(C110-Pad1) -> Net-(C110-Pad2)
- U17 pad 6: Net-(C110-Pad2) -> Net-(C110-Pad1)
- U18 pad 1: Net-(D23-Pad1) -> /USB-PD/PD_CC1
- U18 pad 10: (no net) -> GND
- U18 pad 11: (no net) -> STUSB4500_ATTACH
- U18 pad 12: (no net) -> Net-(R121-Pad2)
- U18 pad 13: (no net) -> Net-(R122-Pad2)
- U18 pad 14: (no net) -> /USB-PD/STUSB4500_PWR_OK3
- U18 pad 15: (no net) -> STUSB4500_GPIO
- U18 pad 17: (no net) -> STUSB4500_AB_SIDE
- U18 pad 19: (no net) -> STUSB4500_ALERT
- U18 pad 2: Net-(D23-Pad1) -> /USB-PD/PD_CC1
- U18 pad 20: (no net) -> /USB-PD/STUSB4500_PWR_OK2
- U18 pad 21: Net-(C138-Pad1) -> /USB-PD/VREG_1V2
- U18 pad 23: /USB-PD/2V7 -> /USB-PD/VREG_2V7
- U18 pad 24: /USB-PD/PD_VBUS -> /USB-PD/STUSB_VDD
- U18 pad 25: (no net) -> GND
- U18 pad 4: Net-(D23-Pad2) -> /USB-PD/PD_CC2
- U18 pad 5: Net-(D23-Pad2) -> /USB-PD/PD_CC2
- U18 pad 7: (no net) -> STUSB4500_SCL
- U18 pad 8: (no net) -> STUSB4500_SDA
- U2 pad 17: RST_N -> /HDMI_converter/RST_N
- U2 pad 18: HDMIOUT_SCL -> /HDMI_converter/HDMIOUT_SCL
- U2 pad 19: HDMIOUT_SDA -> /HDMI_converter/HDMIOUT_SDA
- U2 pad 23: INTO_GPIO5 -> /HDMI_converter/INTO_GPIO5
- U2 pad 24: CEC_GPIO6 -> /HDMI_converter/LT_CEC
- U2 pad 26: LT9611_VCC33_IO -> /HDMI_converter/LT9611_VCC33_RX
- U2 pad 3: LT9611_VCC33_RX -> /HDMI_converter/LT9611_VCC33_IO
- U2 pad 34: LT9611_VCC33_IO -> /HDMI_converter/LT9611_VCC33_RX
- U2 pad 38: TX_CLK_N -> /HDMI_converter/TX_CLK_N
- U2 pad 39: TX_CLK_P -> /HDMI_converter/TX_CLK_P
- U2 pad 40: TX_D0_N -> /HDMI_converter/TX_D0_N
- U2 pad 41: TX_D0_P -> /HDMI_converter/TX_D0_P
- U2 pad 42: VCOM -> /HDMI_converter/VCOM
- U2 pad 43: LT9611_VCC33_TX -> /HDMI_converter/LT9611_VCC33_TX
- U2 pad 45: TX_D1_N -> /HDMI_converter/TX_D1_N
- U2 pad 46: TX_D1_P -> /HDMI_converter/TX_D1_P
- U2 pad 47: TX_D2_N -> /HDMI_converter/TX_D2_N
- U2 pad 48: TX_D2_P -> /HDMI_converter/TX_D2_P
- U2 pad 51: LT9611_VCC33_RX -> /HDMI_converter/LT9611_VCC33_IO
- U2 pad 52: Net-(R28-Pad2) -> Net-(R52-Pad1)
- U2 pad 55: LT9611_VCC33_RX -> /HDMI_converter/LT9611_VCC33_IO
- U3 pad 1: 1V8 -> VREG_S4A_1V8
- U3 pad 11: 3V3 -> 3V3_SYS
- U3 pad 12: Net-(R37-Pad2) -> VREG_S4A_1V8
- U5 pad 1: 5V -> 5V_SYS
- U5 pad 2: 5V -> 5V_SYS
- U6 pad 10: 3V3 -> 3V3_SYS
- U7 pad 1: 1V8 -> 1V8_SYS
- U7 pad 14: 5V -> 5V_SYS
- U7 pad 8: 5V -> 1V8_SYS
- U8 pad 1: 3V3 -> 3V3_SYS
- U8 pad 10: 3V3 -> 3V3_SYS
- U8 pad 6: 3V3 -> 3V3_SYS
- Y2 pad 1: /HDMI_converter/XTALI -> /HDMI_converter/XTALO
- Y2 pad 3: /HDMI_converter/XTALO -> /HDMI_converter/XTALI

Commit message: Loclib
Parts:
- C106, C150: footprint antmicro-footprints:0805-cap -> sa800u-baseboard-hw-footprints:0805-cap
- D11, D13, D19: footprint antmicro-footprints:LED_0603 -> sa800u-baseboard-hw-footprints:LED_0603
- R1, R134, R135, R136, R137, R138, R139, R140, R141, R142, R143, R154, R2, R28, R3, R54, R56, R57, R58, R60, R61, R62, R8: footprint antmicro-footprints:0402-res -> sa800u-baseboard-hw-footprints:0402-res
- R155, R156: footprint antmicro-footprints:0603-res -> sa800u-baseboard-hw-footprints:0603-res
- SP2, SP3, SP4, SP5: footprint antmicro-footprints:9774060151 -> sa800u-baseboard-hw-footprints:9774060151
- U22: footprint antmicro-footprints:SOT-223 -> sa800u-baseboard-hw-footprints:SOT-223
