File: USB-PD.sch (KiCad schematic (older format))
At the start: 24 parts, among them J11 WE_632723300011, Q7 IRF7404TRPBF, U18 STUSB4500QTR

Commit message: add OD signaling pins with pullups network
Parts:
- added R? (x6): R_4k7_0402, antmicro-footprints:0402-res, symbol antmicroResistors0402:R_4k7_0402
Connections:
- net labels added: STUSB4500_AB_SIDE, STUSB4500_ALERT, STUSB4500_ATTACH, STUSB4500_GPIO, STUSB4500_PWR_OK2, STUSB4500_PWR_OK3
- wire segments 114 -> 146
Other:
- note added: "I2C pullups (ALERT is I2C interrupt)"
- note added: "OD pins pullups"
- note added: "Pull - up to SoM's voltage."
Changed lines of the file:
@@
 Wire Wire Line
 	6350 4950 6700 4950
-Text GLabel 5000 6400 0    50   Input ~ 0
+Text GLabel 5250 6750 0    50   Input ~ 0
 STUSB4500_SDA
-Text GLabel 5000 6300 0    50   Input ~ 0
+Text GLabel 5250 6650 0    50   Input ~ 0
 STUSB4500_SCL
 Wire Wire Line
-	5000 6300 5200 6300
-Wire Wire Line
-	5750 6300 5750 6150
-Wire Wire Line
-	5850 6400 5850 6150
-Wire Wire Line
-	5000 6400 5200 6400
-Text GLabel 5750 6150 1    50   Input ~ 0
+	5250 6650 5450 6650
+Wire Wire Line
+	6000 6650 6000 6500
+Wire Wire Line
+	6100 6750 6100 6500
+Wire Wire Line
+	5250 6750 5450 6750
+Text GLabel 6200 6350 1    50   Input ~ 0
 1V8
-Text GLabel 5850 6150 1    50   Input ~ 0
+$Comp
+L antmicroResistors0402:R_4k7_0402 R?
+U 1 1 61F8049E
+P 5600 6650
+F 0 "R?" H 5400 6700 60  0000 C CNN
+F 1 "R_4k7_0402" H 5600 6500 60  0001 C CNN
+F 2 "antmicro-footprints:0402-res" H 5800 6850 60  0001 L CNN
+F 3 "" H 5600 6650 50  0001 C CNN
+F 4 "VISHAY" H 5800 7050 60  0001 L CNN "Manufacturer"
+F 5 "MCS04020C4701FE000" H 5800 6950 60  0001 L CNN "MPN"
+F 6 "4k7" H 5600 6650 50  0000 C CNN "Val"
+	1    5600 6650
+	1    0    0    -1
+$EndComp
+Wire Wire Line
+	5750 6650 6000 6650
+$Comp
+L antmicroResistors0402:R_4k7_0402 R?
+U 1 1 61F80835
+P 5600 6750
+F 0 "R?" H 5400 6800 60  0000 C CNN
+F 1 "R_4k7_0402" H 5600 6600 60  0001 C CNN
+F 2 "antmicro-footprints:0402-res" H 5800 6950 60  0001 L CNN
+F 3 "" H 5600 6750 50  0001 C CNN
+F 4 "VISHAY" H 5800 7150 60  0001 L CNN "Manufacturer"
+F 5 "MCS04020C4701FE000" H 5800 7050 60  0001 L CNN "MPN"
+F 6 "4k7" H 5600 6750 50  0000 C CNN "Val"
+	1    5600 6750
+	1    0    0    -1
+$EndComp
+Wire Wire Line
+	5750 6750 6100 6750
+Text GLabel 6350 5050 0    50   Input ~ 0
+STUSB4500_ALERT
+Wire Wire Line
+	6700 5050 6350 5050
+Text Notes 3100 7150 0    50   ~ 0
+Pull - up to SoM's voltage.
+Text GLabel 5250 6850 0    50   Input ~ 0
+STUSB4500_ALERT
+Wire Wire Line
+	5250 6850 5450 6850
+Wire Wire Line
+	6200 6850 6200 6500
+Wire Wire Line
+	6000 6500 6100 6500
+Connection ~ 6100 6500
+Wire Wire Line
+	6100 6500 6200 6500
+Wire Wire Line
+	6200 6500 6200 6350
+$Comp
+L antmicroResistors0402:R_4k7_0402 R?
+U 1 1 61FA2102
+P 5600 6850
+F 0 "R?" H 5400 6900 60  0000 C CNN
+F 1 "R_4k7_0402" H 5600 6700 60  0001 C CNN
+F 2 "antmicro-footprints:0402-res" H 5800 7050 60  0001 L CNN
+F 3 "" H 5600 6850 50  0001 C CNN
+F 4 "VISHAY" H 5800 7250 60  0001 L CNN "Manufacturer"
+F 5 "MCS04020C4701FE000" H 5800 7150 60  0001 L CNN "MPN"
+F 6 "4k7" H 5600 6850 50  0000 C CNN "Val"
+	1    5600 6850
+	1    0    0    -1
+$EndComp
+Wire Wire Line
+	5750 6850 6200 6850
+Wire Wire Line
+	8500 4550 8700 4550
+Text GLabel 8700 4550 2    50   Input ~ 0
+STUSB4500_ATTACH
+Text GLabel 8700 4650 2    50   Input ~ 0
+STUSB4500_PWR_OK2
+Text GLabel 8700 4750 2    50   Input ~ 0
+STUSB4500_PWR_OK3
+Wire Wire Line
+	8700 4650 8500 4650
+Wire Wire Line
+	8500 4750 8700 4750
+Text GLabel 8700 4950 2    50   Input ~ 0
+STUSB4500_GPIO
+Wire Wire Line
+	8500 4950 8700 4950
+Text GLabel 8700 5150 2    50   Input ~ 0
+STUSB4500_AB_SIDE
+Wire Wire Line
+	8700 5150 8500 5150
+Text Notes 4500 6500 0    50   ~ 0
+I2C pullups (ALERT is I2C interrupt)
+Text GLabel 5250 7850 0    50   Input ~ 0
+STUSB4500_ATTACH
+Text GLabel 5250 7750 0    50   Input ~ 0
+STUSB4500_PWR_OK2
+Text GLabel 5250 7650 0    50   Input ~ 0
+STUSB4500_PWR_OK3
+Text GLabel 5250 7550 0    50   Input ~ 0
+STUSB4500_GPIO
+Text GLabel 5250 7450 0    50   Input ~ 0
+STUSB4500_AB_SIDE
+Wire Wire Line
+	5750 7450 5750 7300
+Wire Wire Line
+	5850 7550 5850 7300
+Text GLabel 6150 7150 1    50   Input ~ 0
 1V8
-$Comp
-L antmicroResistors0402:R_4k7_0402 R?
-U 1 1 61F8049E
-P 5350 6300
-F 0 "R?" H 5350 6513 60  0000 C CNN
-F 1 "R_4k7_0402" H 5350 6150 60  0001 C CNN
-F 2 "antmicro-footprints:0402-res" H 5550 6500 60  0001 L CNN
-F 3 "" H 5350 6300 50  0001 C CNN
-F 4 "VISHAY" H 5550 6700 60  0001 L CNN "Manufacturer"
-F 5 "MCS04020C4701FE000" H 5550 6600 60  0001 L CNN "MPN"
-F 6 "4k7" H 5350 6415 50  0000 C CNN "Val"
-	1    5350 6300
-	1    0    0    -1
-$EndComp
-Wire Wire Line
-	5500 6300 5750 6300
-$Comp
-L antmicroResistors0402:R_4k7_0402 R?
-U 1 1 61F80835
-P 5350 6400
-F 0 "R?" H 5350 6200 60  0000 C CNN
-F 1 "R_4k7_0402" H 5350 6250 60  0001 C CNN
-F 2 "antmicro-footprints:0402-res" H 5550 6600 60  0001 L CNN
-F 3 "" H 5350 6400 50  0001 C CNN
-F 4 "VISHAY" H 5550 6800 60  0001 L CNN "Manufacturer"
-F 5 "MCS04020C4701FE000" H 5550 6700 60  0001 L CNN "MPN"
-F 6 "4k7" H 5350 6300 50  0000 C CNN "Val"
-	1    5350 6400
-	1    0    0    -1
-$EndComp
-Wire Wire Line
-	5500 6400 5850 6400
+Wire Wire Line
+	5250 7450 5400 7450
+Wire Wire Line
+	5250 7550 5400 7550
+Wire Wire Line
+	5950 7650 5950 7300
+Wire Wire Line
+	5750 7300 5850 7300
+Connection ~ 5850 7300
+Wire Wire Line
+	5850 7300 5950 7300
+Wire Wire Line
+	6150 7300 6150 7150
+Wire Wire Line
+	5250 7650 5400 7650
+Wire Wire Line
+	5950 7300 6050 7300
+Wire Wire Line
+	6050 7300 6050 7750
+Wire Wire Line
+	6050 7750 5700 7750
+Connection ~ 5950 7300
+Wire Wire Line
+	6050 7300 6150 7300
+Wire Wire Line
+	6150 7300 6150 7850
+Wire Wire Line
+	6150 7850 5700 7850
+Connection ~ 6050 7300
+Connection ~ 6150 7300
+Connection ~ 6200 6500
+Text Notes 4900 7300 0    50   ~ 0
+OD pins pullups
+$Comp
+L antmicroResistors0402:R_4k7_0402 R?
+U 1 1 62072163
+P 5550 7450
+F 0 "R?" H 5350 7500 60  0000 C CNN
+F 1 "R_4k7_0402" H 5550 7300 60  0001 C CNN
+F 2 "antmicro-footprints:0402-res" H 5750 7650 60  0001 L CNN
+F 3 "" H 5550 7450 50  0001 C CNN
+F 4 "VISHAY" H 5750 7850 60  0001 L CNN "Manufacturer"
+F 5 "MCS04020C4701FE000" H 5750 7750 60  0001 L CNN "MPN"
+F 6 "4k7" H 5550 7450 50  0000 C CNN "Val"
+	1    5550 7450
+	1    0    0    -1
+$EndComp
+Wire Wire Line
+	5700 7450 5750 7450
+$Comp
+L antmicroResistors0402:R_4k7_0402 R?
+U 1 1 62072928
+P 5550 7550
+F 0 "R?" H 5350 7600 60  0000 C CNN
+F 1 "R_4k7_0402" H 5550 7400 60  0001 C CNN
+F 2 "antmicro-footprints:0402-res" H 5750 7750 60  0001 L CNN
+F 3 "" H 5550 7550 50  0001 C CNN
+F 4 "VISHAY" H 5750 7950 60  0001 L CNN "Manufacturer"
+F 5 "MCS04020C4701FE000" H 5750 7850 60  0001 L CNN "MPN"
+F 6 "4k7" H 5550 7550 50  0000 C CNN "Val"
+	1    5550 7550
+	1    0    0    -1
+$EndComp
+Wire Wire Line
+	5700 7550 5850 7550
+$Comp
+L antmicroResistors0402:R_4k7_0402 R?
+U 1 1 62072AB9
+P 5550 7650
+F 0 "R?" H 5350 7700 60  0000 C CNN
+F 1 "R_4k7_0402" H 5550 7500 60  0001 C CNN
+F 2 "antmicro-footprints:0402-res" H 5750 7850 60  0001 L CNN
+F 3 "" H 5550 7650 50  0001 C CNN
+F 4 "VISHAY" H 5750 8050 60  0001 L CNN "Manufacturer"
+F 5 "MCS04020C4701FE000" H 5750 7950 60  0001 L CNN "MPN"
+F 6 "4k7" H 5550 7650 50  0000 C CNN "Val"
+	1    5550 7650
+	1    0    0    -1
+$EndComp
+Wire Wire Line
+	5700 7650 5950 7650
+$Comp
+L antmicroResistors0402:R_4k7_0402 R?
+U 1 1 62072BBE
+P 5550 7750
+F 0 "R?" H 5350 7800 60  0000 C CNN
+F 1 "R_4k7_0402" H 5550 7600 60  0001 C CNN
+F 2 "antmicro-footprints:0402-res" H 5750 7950 60  0001 L CNN
+F 3 "" H 5550 7750 50  0001 C CNN
+F 4 "VISHAY" H 5750 8150 60  0001 L CNN "Manufacturer"
+F 5 "MCS04020C4701FE000" H 5750 8050 60  0001 L CNN "MPN"
+F 6 "4k7" H 5550 7750 50  0000 C CNN "Val"
+	1    5550 7750
+	1    0    0    -1
+$EndComp
+Wire Wire Line
+	5400 7750 5250 7750
+$Comp
+L antmicroResistors0402:R_4k7_0402 R?
+U 1 1 62072D97
+P 5550 7850
+F 0 "R?" H 5350 7900 60  0000 C CNN
+F 1 "R_4k7_0402" H 5550 7700 60  0001 C CNN
+F 2 "antmicro-footprints:0402-res" H 5750 8050 60  0001 L CNN
+F 3 "" H 5550 7850 50  0001 C CNN
+F 4 "VISHAY" H 5750 8250 60  0001 L CNN "Manufacturer"
+F 5 "MCS04020C4701FE000" H 5750 8150 60  0001 L CNN "MPN"
+F 6 "4k7" H 5550 7850 50  0000 C CNN "Val"
+	1    5550 7850
+	1    0    0    -1
+$EndComp
+Wire Wire Line
+	5400 7850 5250 7850
 $EndSCHEMATC
