File: USB-PD.sch (KiCad schematic (older format))
At the start: 30 parts, among them J11 WE_632723300011, Q7 IRF7404TRPBF, U18 STUSB4500QTR

Commit message: finished USB-PD
Parts:
- removed R? (x2): R_4k7_0402, antmicro-footprints:0402-res, symbol antmicroResistors0402:R_4k7_0402
- added D?: ASMB-TTF0-0A20B, antmicro-footprints:PLCC6_3.5x3.7mm, symbol antmicroLEDIndicationDiscrete:ASMB-TTF0-0A20B
- added R?: R_590R_0402, antmicro-footprints:0402-res, symbol antmicroResistors0402:R_590R_0402
- added R?: R_150R_0402, antmicro-footprints:0402-res, symbol antmicroResistors0402:R_150R_0402
- added R?: R_100R_0402, antmicro-footprints:0402-res, symbol antmicroResistors0402:R_100R_0402
Connections:
- net labels added: 5V
- wire segments 146 -> 148
Other:
- note added: "R G B\n50 30 30 [mA]\n2.1 2.9 2.9 [V]"
- note removed: "WORK IN PROGRESS"
Changed lines of the file:
@@
 This diode has Vrm (standoff voltage) = 24V\nCCx pins are rated for up to 22V. But identical\ndiode was used in reference and in dev board.
 Connection ~ 6200 1750
-Text Notes 7200 3350 0    50   ~ 0
-WORK IN PROGRESS
 $Comp
 L sa800u-baseboard-hw:GND #PWR0213
 U 1 1 61DF321E
-P 9650 4450
-F 0 "#PWR0213" H 9650 4200 50  0001 C CNN
-F 1 "GND" V 9655 4322 50  0000 R CNN
-F 2 "" H 9650 4450 50  0001 C CNN
-F 3 "" H 9650 4450 50  0001 C CNN
-	1    9650 4450
-	1    0    0    -1
+P 9850 4350
+F 0 "#PWR0213" H 9850 4100 50  0001 C CNN
+F 1 "GND" V 9855 4222 50  0000 R CNN
+F 2 "" H 9850 4350 50  0001 C CNN
+F 3 "" H 9850 4350 50  0001 C CNN
+	1    9850 4350
+	0    -1   -1   0
 $EndComp
 $Comp
@@
 	9650 3950 9650 4250
 Wire Wire Line
-	9650 4450 9650 4350
+	9850 4350 9650 4350
 Connection ~ 9650 4350
 $Comp
@@
 Wire Wire Line
 	6450 5250 6700 5250
-Text Notes 12450 1550 0    50   ~ 0
-WORK IN PROGRESS
 Wire Wire Line
 	12350 1750 12350 1850
@@
 $EndComp
 Wire Wire Line
-	13200 1750 14050 1750
+	13200 1750 13650 1750
 Wire Wire Line
 	14050 1750 14050 1800
@@
 Text GLabel 8700 4550 2    50   Input ~ 0
 STUSB4500_ATTACH
-Text GLabel 8700 4650 2    50   Input ~ 0
-STUSB4500_PWR_OK2
-Text GLabel 8700 4750 2    50   Input ~ 0
-STUSB4500_PWR_OK3
-Wire Wire Line
-	8700 4650 8500 4650
-Wire Wire Line
-	8500 4750 8700 4750
+Wire Wire Line
+	9500 4650 8500 4650
+Wire Wire Line
+	8500 4750 9500 4750
 Text GLabel 8700 4950 2    50   Input ~ 0
 STUSB4500_GPIO
@@
 Text Notes 4500 6500 0    50   ~ 0
 I2C pullups (ALERT is I2C interrupt)
-Text GLabel 5250 7850 0    50   Input ~ 0
+Text GLabel 5450 7650 0    50   Input ~ 0
 STUSB4500_ATTACH
-Text GLabel 5250 7750 0    50   Input ~ 0
-STUSB4500_PWR_OK2
-Text GLabel 5250 7650 0    50   Input ~ 0
-STUSB4500_PWR_OK3
-Text GLabel 5250 7550 0    50   Input ~ 0
+Text GLabel 5450 7550 0    50   Input ~ 0
 STUSB4500_GPIO
-Text GLabel 5250 7450 0    50   Input ~ 0
+Text GLabel 5450 7450 0    50   Input ~ 0
 STUSB4500_AB_SIDE
 Wire Wire Line
-	5750 7450 5750 7300
-Wire Wire Line
-	5850 7550 5850 7300
+	5950 7450 5950 7300
+Wire Wire Line
+	6050 7550 6050 7300
 Text GLabel 6150 7150 1    50   Input ~ 0
 1V8
 Wire Wire Line
-	5250 7450 5400 7450
-Wire Wire Line
-	5250 7550 5400 7550
-Wire Wire Line
-	5950 7650 5950 7300
-Wire Wire Line
-	5750 7300 5850 7300
-Connection ~ 5850 7300
-Wire Wire Line
-	5850 7300 5950 7300
+	5450 7450 5600 7450
+Wire Wire Line
+	5450 7550 5600 7550
+Wire Wire Line
+	6150 7650 6150 7300
 Wire Wire Line
 	6150 7300 6150 7150
 Wire Wire Line
-	5250 7650 5400 7650
-Wire Wire Line
-	5950 7300 6050 7300
-Wire Wire Line
-	6050 7300 6050 7750
-Wire Wire Line
-	6050 7750 5700 7750
-Connection ~ 5950 7300
-Wire Wire Line
-	6050 7300 6150 7300
-Wire Wire Line
-	6150 7300 6150 7850
-Wire Wire Line
-	6150 7850 5700 7850
-Connection ~ 6050 7300
-Connection ~ 6150 7300
+	5450 7650 5600 7650
 Connection ~ 6200 6500
 Text Notes 4900 7300 0    50   ~ 0
@@
 L antmicroResistors0402:R_4k7_0402 R?
 U 1 1 62072163
-P 5550 7450
-F 0 "R?" H 5350 7500 60  0000 C CNN
-F 1 "R_4k7_0402" H 5550 7300 60  0001 C CNN
-F 2 "antmicro-footprints:0402-res" H 5750 7650 60  0001 L CNN
-F 3 "" H 5550 7450 50  0001 C CNN
-F 4 "VISHAY" H 5750 7850 60  0001 L CNN "Manufacturer"
-F 5 "MCS04020C4701FE000" H 5750 7750 60  0001 L CNN "MPN"
-F 6 "4k7" H 5550 7450 50  0000 C CNN "Val"
-	1    5550 7450
-	1    0    0    -1
-$EndComp
-Wire Wire Line
-	5700 7450 5750 7450
+P 5750 7450
+F 0 "R?" H 5550 7500 60  0000 C CNN
+F 1 "R_4k7_0402" H 5750 7300 60  0001 C CNN
+F 2 "antmicro-footprints:0402-res" H 5950 7650 60  0001 L CNN
+F 3 "" H 5750 7450 50  0001 C CNN
+F 4 "VISHAY" H 5950 7850 60  0001 L CNN "Manufacturer"
+F 5 "MCS04020C4701FE000" H 5950 7750 60  0001 L CNN "MPN"
+F 6 "4k7" H 5750 7450 50  0000 C CNN "Val"
+	1    5750 7450
+	1    0    0    -1
+$EndComp
+Wire Wire Line
+	5900 7450 5950 7450
 $Comp
 L antmicroResistors0402:R_4k7_0402 R?
 U 1 1 62072928
-P 5550 7550
-F 0 "R?" H 5350 7600 60  0000 C CNN
-F 1 "R_4k7_0402" H 5550 7400 60  0001 C CNN
-F 2 "antmicro-footprints:0402-res" H 5750 7750 60  0001 L CNN
-F 3 "" H 5550 7550 50  0001 C CNN
-F 4 "VISHAY" H 5750 7950 60  0001 L CNN "Manufacturer"
-F 5 "MCS04020C4701FE000" H 5750 7850 60  0001 L CNN "MPN"
-F 6 "4k7" H 5550 7550 50  0000 C CNN "Val"
-	1    5550 7550
-	1    0    0    -1
-$EndComp
-Wire Wire Line
-	5700 7550 5850 7550
+P 5750 7550
+F 0 "R?" H 5550 7600 60  0000 C CNN
+F 1 "R_4k7_0402" H 5750 7400 60  0001 C CNN
+F 2 "antmicro-footprints:0402-res" H 5950 7750 60  0001 L CNN
+F 3 "" H 5750 7550 50  0001 C CNN
+F 4 "VISHAY" H 5950 7950 60  0001 L CNN "Manufacturer"
+F 5 "MCS04020C4701FE000" H 5950 7850 60  0001 L CNN "MPN"
+F 6 "4k7" H 5750 7550 50  0000 C CNN "Val"
+	1    5750 7550
+	1    0    0    -1
+$EndComp
+Wire Wire Line
+	5900 7550 6050 7550
 $Comp
 L antmicroResistors0402:R_4k7_0402 R?
 U 1 1 62072AB9
-P 5550 7650
-F 0 "R?" H 5350 7700 60  0000 C CNN
-F 1 "R_4k7_0402" H 5550 7500 60  0001 C CNN
-F 2 "antmicro-footprints:0402-res" H 5750 7850 60  0001 L CNN
-F 3 "" H 5550 7650 50  0001 C CNN
-F 4 "VISHAY" H 5750 8050 60  0001 L CNN "Manufacturer"
-F 5 "MCS04020C4701FE000" H 5750 7950 60  0001 L CNN "MPN"
-F 6 "4k7" H 5550 7650 50  0000 C CNN "Val"
-	1    5550 7650
-	1    0    0    -1
-$EndComp
-Wire Wire Line
-	5700 7650 5950 7650
-$Comp
-L antmicroResistors0402:R_4k7_0402 R?
-U 1 1 62072BBE
-P 5550 7750
-F 0 "R?" H 5350 7800 60  0000 C CNN
-F 1 "R_4k7_0402" H 5550 7600 60  0001 C CNN
-F 2 "antmicro-footprints:0402-res" H 5750 7950 60  0001 L CNN
-F 3 "" H 5550 7750 50  0001 C CNN
-F 4 "VISHAY" H 5750 8150 60  0001 L CNN "Manufacturer"
-F 5 "MCS04020C4701FE000" H 5750 8050 60  0001 L CNN "MPN"
-F 6 "4k7" H 5550 7750 50  0000 C CNN "Val"
-	1    5550 7750
-	1    0    0    -1
-$EndComp
-Wire Wire Line
-	5400 7750 5250 7750
-$Comp
-L antmicroResistors0402:R_4k7_0402 R?
-U 1 1 62072D97
-P 5550 7850
-F 0 "R?" H 5350 7900 60  0000 C CNN
-F 1 "R_4k7_0402" H 5550 7700 60  0001 C CNN
-F 2 "antmicro-footprints:0402-res" H 5750 8050 60  0001 L CNN
-F 3 "" H 5550 7850 50  0001 C CNN
-F 4 "VISHAY" H 5750 8250 60  0001 L CNN "Manufacturer"
-F 5 "MCS04020C4701FE000" H 5750 8150 60  0001 L CNN "MPN"
-F 6 "4k7" H 5550 7850 50  0000 C CNN "Val"
-	1    5550 7850
-	1    0    0    -1
-$EndComp
-Wire Wire Line
-	5400 7850 5250 7850
+P 5750 7650
+F 0 "R?" H 5550 7700 60  0000 C CNN
+F 1 "R_4k7_0402" H 5750 7500 60  0001 C CNN
+F 2 "antmicro-footprints:0402-res" H 5950 7850 60  0001 L CNN
+F 3 "" H 5750 7650 50  0001 C CNN
+F 4 "VISHAY" H 5950 8050 60  0001 L CNN "Manufacturer"
+F 5 "MCS04020C4701FE000" H 5950 7950 60  0001 L CNN "MPN"
+F 6 "4k7" H 5750 7650 50  0000 C CNN "Val"
+	1    5750 7650
+	1    0    0    -1
+$EndComp
+Wire Wire Line
+	5900 7650 6150 7650
+Connection ~ 13650 1750
+Wire Wire Line
+	13650 1750 14050 1750
+Text Notes 14100 4550 0    50   ~ 0
+R   G   B\n50  30 30 [mA]\n2.1 2.9 2.9 [V]
+Wire Wire Line
+	13650 1750 13650 4500
+Text GLabel 13450 4200 1    50   Input ~ 0
+5V
+Text GLabel 13850 4200 1    50   Input ~ 0
+5V
+Wire Wire Line
+	13450 4200 13450 4500
+Wire Wire Line
+	13850 4200 13850 4500
+$Comp
+L antmicroLEDIndicationDiscrete:ASMB-TTF0-0A20B D?
+U 1 1 620BAED1
+P 13650 4750
+F 0 "D?" V 13597 4372 60  0000 R CNN
+F 1 "ASMB-TTF0-0A20B" V 13703 4372 60  0000 R CNN
+F 2 "antmicro-footprints:PLCC6_3.5x3.7mm" H 13250 4050 60  0001 L CNN
+F 3 "https://docs.broadcom.com/doc/ASMB-TTF0-0A20B-DS101" H 13850 5050 60  0001 L CNN
+F 4 "ASMB-TTF0-0A20B" H 13200 4150 60  0001 L CNN "MPN"
+F 5 "Broadcom" H 13500 4250 60  0001 L CNN "Manufacturer"
+	1    13650 4750
+	0    -1   1    0
+$EndComp
+$Comp
+L antmicroResistors0402:R_590R_0402 R?
+U 1 1 621057A9
+P 13650 5350
+F 0 "R?" H 13400 5300 60  0000 L CNN
+F 1 "R_590R_0402" H 13650 5200 60  0001 C CNN
+F 2 "antmicro-footprints:0402-res" H 13850 5550 60  0001 L CNN
+F 3 "" H 13650 5350 50  0001 C CNN
+F 4 "PANASONIC_ELECTRONIC_COMPONENTS" H 13850 5750 60  0001 L CNN "Manufacturer"
+F 5 "ERJ2RKF5900X" H 13850 5650 60  0001 L CNN "MPN"
+F 6 "590R" H 13550 5350 50  0000 L CNN "Val"
+	1    13650 5350
+	0    1    1    0
+$EndComp
+Wire Wire Line
+	13650 5200 13650 5000
+$Comp
+L power:GND #PWR?
+U 1 1 62113B31
+P 13650 5700
+F 0 "#PWR?" H 13650 5450 50  0001 C CNN
+F 1 "GND" H 13655 5527 50  0000 C CNN
+F 2 "" H 13650 5700 50  0001 C CNN
+F 3 "" H 13650 5700 50  0001 C CNN
+	1    13650 5700
+	1    0    0    -1
+$EndComp
+Wire Wire Line
+	13450 5000 13450 5200
+Wire Wire Line
+	13850 5200 13850 5000
+Wire Wire Line
+	13650 5500 13650 5700
+Wire Wire Line
+	13450 5500 13450 5700
+Wire Wire Line
+	13850 5500 13850 5700
+Text Label 9500 4650 0    50   ~ 0
+STUSB4500_PWR_OK2
+Text Label 9500 4750 0    50   ~ 0
+STUSB4500_PWR_OK3
+Text Label 13450 5700 3    50   ~ 0
+STUSB4500_PWR_OK2
+Text Label 13850 5700 3    50   ~ 0
+STUSB4500_PWR_OK3
+Wire Wire Line
+	5950 7300 6050 7300
+Connection ~ 6050 7300
+Wire Wire Line
+	6050 7300 6150 7300
+Connection ~ 6150 7300
+$Comp
+L antmicroResistors0402:R_150R_0402 R?
+U 1 1 62198F27
+P 13450 5350
+F 0 "R?" H 13200 5300 60  0000 L CNN
+F 1 "R_150R_0402" H 13450 5200 60  0001 C CNN
+F 2 "antmicro-footprints:0402-res" H 13650 5550 60  0001 L CNN
+F 3 "" H 13450 5350 50  0001 C CNN
+F 4 "VISHAY" H 13650 5750 60  0001 L CNN "Manufacturer"
+F 5 "CRCW0402150RFKED" H 13650 5650 60  0001 L CNN "MPN"
+F 6 "150R" H 13350 5350 50  0000 L CNN "Val"
+	1    13450 5350
+	0    1    1    0
+$EndComp
+$Comp
+L antmicroResistors0402:R_100R_0402 R?
+U 1 1 6219BF48
+P 13850 5350
+F 0 "R?" H 13600 5300 60  0000 L CNN
+F 1 "R_100R_0402" H 13850 5200 60  0001 C CNN
+F 2 "antmicro-footprints:0402-res" H 14050 5550 60  0001 L CNN
+F 3 "" H 13850 5350 50  0001 C CNN
+F 4 "BOURNS" H 14050 5750 60  0001 L CNN "Manufacturer"
+F 5 "CR0402-FX-1000GLF" H 14050 5650 60  0001 L CNN "MPN"
+F 6 "100R" H 13750 5350 50  0000 L CNN "Val"
+	1    13850 5350
+	0    1    1    0
+$EndComp
 $EndSCHEMATC

Commit message: Loclib
Parts:
- D?: footprint antmicro-footprints:ESD144B1W0201E6327XTSA1 -> sa800u-baseboard-hw-footprints:ESD144B1W0201E6327XTSA1; symbol antmicroTVSDiodes:ESD144B1W0201E6327XTSA1 -> sa800u-baseboard-hw:ESD144B1W0201E6327XTSA1
- D?: footprint antmicro-footprints:PLCC6_3.5x3.7mm -> sa800u-baseboard-hw-footprints:PLCC6_3.5x3.7mm; symbol antmicroLEDIndicationDiscrete:ASMB-TTF0-0A20B -> sa800u-baseboard-hw:ASMB-TTF0-0A20B
- R? (x4): footprint antmicro-footprints:0402-res -> sa800u-baseboard-hw-footprints:0402-res; symbol antmicroResistors0402:R_100k_0402 -> sa800u-baseboard-hw:R_100k_0402
- R? (x6): footprint antmicro-footprints:0402-res -> sa800u-baseboard-hw-footprints:0402-res; symbol antmicroResistors0402:R_4k7_0402 -> sa800u-baseboard-hw:R_4k7_0402
- R?: footprint antmicro-footprints:0402-res -> sa800u-baseboard-hw-footprints:0402-res; symbol antmicroResistors0402:R_590R_0402 -> sa800u-baseboard-hw:R_590R_0402
- R?: footprint antmicro-footprints:0402-res -> sa800u-baseboard-hw-footprints:0402-res; symbol antmicroResistors0402:R_150R_0402 -> sa800u-baseboard-hw:R_150R_0402
- R?: footprint antmicro-footprints:0402-res -> sa800u-baseboard-hw-footprints:0402-res; symbol antmicroResistors0402:R_100R_0402 -> sa800u-baseboard-hw:R_100R_0402
Changed lines of the file:
@@
 Connection ~ 12350 1850
 $Comp
-L antmicroTVSDiodes:ESD144B1W0201E6327XTSA1 D?
+L sa800u-baseboard-hw:ESD144B1W0201E6327XTSA1 D?
 U 1 1 61ED3FD6
 P 14050 2150
 F 0 "D?" V 14004 2228 50  0000 L CNN
 F 1 "ESD144B1W0201E6327XTSA1" V 14095 2228 50  0000 L CNN
-F 2 "antmicro-footprints:ESD144B1W0201E6327XTSA1" H 14050 2150 50  0001 C CNN
+F 2 "sa800u-baseboard-hw-footprints:ESD144B1W0201E6327XTSA1" H 14050 2150 50  0001 C CNN
 F 3 "https://www.infineon.com/dgdl/Infineon-ESD144-B1-W0201-DataSheet-v02_00-EN.pdf?fileId=5546d462677d0f4601679886a2a8707c" H 14050 2150 50  0001 C CNN
 F 4 "ESD144B1W0201E6327XTSA1" H 14050 2150 50  0001 C CNN "MPN"
@@
 	14050 2500 14050 2550
 $Comp
-L power:GND #PWR?
+L sa800u-baseboard-hw:GND #PWR?
 U 1 1 61EDB438
 P 14050 2550
@@
 2V7
 $Comp
-L antmicroResistors0402:R_100k_0402 R?
+L sa800u-baseboard-hw:R_100k_0402 R?
 U 1 1 61EEDDB8
 P 5100 4650
 F 0 "R?" H 4950 4750 60  0000 C CNN
 F 1 "R_100k_0402" H 5100 4500 60  0001 C CNN
-F 2 "antmicro-footprints:0402-res" H 5300 4850 60  0001 L CNN
+F 2 "sa800u-baseboard-hw-footprints:0402-res" H 5300 4850 60  0001 L CNN
 F 3 "" H 5100 4650 50  0001 C CNN
 F 4 "VISHAY" H 5300 5050 60  0001 L CNN "Manufacturer"
@@
 	4950 4650 4650 4650
 $Comp
-L antmicroResistors0402:R_100k_0402 R?
+L sa800u-baseboard-hw:R_100k_0402 R?
 U 1 1 61EEE353
 P 5100 4750
 F 0 "R?" H 4950 4650 60  0000 C CNN
 F 1 "R_100k_0402" H 5100 4600 60  0001 C CNN
-F 2 "antmicro-footprints:0402-res" H 5300 4950 60  0001 L CNN
+F 2 "sa800u-baseboard-hw-footprints:0402-res" H 5300 4950 60  0001 L CNN
 F 3 "" H 5100 4750 50  0001 C CNN
 F 4 "VISHAY" H 5300 5150 60  0001 L CNN "Manufacturer"
@@
 Connection ~ 5450 4750
 $Comp
-L power:GND #PWR?
+L sa800u-baseboard-hw:GND #PWR?
 U 1 1 61EF35F3
 P 5350 5150
@@
 $EndComp
 $Comp
-L power:GND #PWR?
+L sa800u-baseboard-hw:GND #PWR?
 U 1 1 61EF3823
 P 5450 5150
@@
 $EndComp
 $Comp
-L antmicroResistors0402:R_100k_0402 R?
+L sa800u-baseboard-hw:R_100k_0402 R?
 U 1 1 61EF8DE3
 P 5350 4950
 F 0 "R?" H 5350 4850 60  0000 C CNN
 F 1 "R_100k_0402" H 5350 4800 60  0001 C CNN
-F 2 "antmicro-footprints:0402-res" H 5550 5150 60  0001 L CNN
+F 2 "sa800u-baseboard-hw-footprints:0402-res" H 5550 5150 60  0001 L CNN
 F 3 "" H 5350 4950 50  0001 C CNN
 F 4 "VISHAY" H 5550 5350 60  0001 L CNN "Manufacturer"
@@
 	5350 5100 5350 5150
 $Comp
-L antmicroResistors0402:R_100k_0402 R?
+L sa800u-baseboard-hw:R_100k_0402 R?
 U 1 1 61F02819
 P 5450 4950
 F 0 "R?" H 5450 5050 60  0000 C CNN
 F 1 "R_100k_0402" H 5450 4800 60  0001 C CNN
-F 2 "antmicro-footprints:0402-res" H 5650 5150 60  0001 L CNN
+F 2 "sa800u-baseboard-hw-footprints:0402-res" H 5650 5150 60  0001 L CNN
 F 3 "" H 5450 4950 50  0001 C CNN
 F 4 "VISHAY" H 5650 5350 60  0001 L CNN "Manufacturer"
@@
 Connection ~ 8850 6150
 $Comp
-L power:GND #PWR?
+L sa800u-baseboard-hw:GND #PWR?
 U 1 1 61F1871C
 P 8850 6250
@@
 1V8
 $Comp
-L antmicroResistors0402:R_4k7_0402 R?
+L sa800u-baseboard-hw:R_4k7_0402 R?
 U 1 1 61F8049E
 P 5600 6650
 F 0 "R?" H 5400 6700 60  0000 C CNN
 F 1 "R_4k7_0402" H 5600 6500 60  0001 C CNN
-F 2 "antmicro-footprints:0402-res" H 5800 6850 60  0001 L CNN
+F 2 "sa800u-baseboard-hw-footprints:0402-res" H 5800 6850 60  0001 L CNN
 F 3 "" H 5600 6650 50  0001 C CNN
 F 4 "VISHAY" H 5800 7050 60  0001 L CNN "Manufacturer"
@@
 	5750 6650 6000 6650
 $Comp
-L antmicroResistors0402:R_4k7_0402 R?
+L sa800u-baseboard-hw:R_4k7_0402 R?
 U 1 1 61F80835
 P 5600 6750
 F 0 "R?" H 5400 6800 60  0000 C CNN
 F 1 "R_4k7_0402" H 5600 6600 60  0001 C CNN
-F 2 "antmicro-footprints:0402-res" H 5800 6950 60  0001 L CNN
+F 2 "sa800u-baseboard-hw-footprints:0402-res" H 5800 6950 60  0001 L CNN
 F 3 "" H 5600 6750 50  0001 C CNN
 F 4 "VISHAY" H 5800 7150 60  0001 L CNN "Manufacturer"
@@
 	6200 6500 6200 6350
 $Comp
-L antmicroResistors0402:R_4k7_0402 R?
+L sa800u-baseboard-hw:R_4k7_0402 R?
 U 1 1 61FA2102
 P 5600 6850
 F 0 "R?" H 5400 6900 60  0000 C CNN
 F 1 "R_4k7_0402" H 5600 6700 60  0001 C CNN
-F 2 "antmicro-footprints:0402-res" H 5800 7050 60  0001 L CNN
+F 2 "sa800u-baseboard-hw-footprints:0402-res" H 5800 7050 60  0001 L CNN
 F 3 "" H 5600 6850 50  0001 C CNN
 F 4 "VISHAY" H 5800 7250 60  0001 L CNN "Manufacturer"
@@
 OD pins pullups
 $Comp
-L antmicroResistors0402:R_4k7_0402 R?
+L sa800u-baseboard-hw:R_4k7_0402 R?
 U 1 1 62072163
 P 5750 7450
 F 0 "R?" H 5550 7500 60  0000 C CNN
 F 1 "R_4k7_0402" H 5750 7300 60  0001 C CNN
-F 2 "antmicro-footprints:0402-res" H 5950 7650 60  0001 L CNN
+F 2 "sa800u-baseboard-hw-footprints:0402-res" H 5950 7650 60  0001 L CNN
 F 3 "" H 5750 7450 50  0001 C CNN
 F 4 "VISHAY" H 5950 7850 60  0001 L CNN "Manufacturer"
@@
 	5900 7450 5950 7450
 $Comp
-L antmicroResistors0402:R_4k7_0402 R?
+L sa800u-baseboard-hw:R_4k7_0402 R?
 U 1 1 62072928
 P 5750 7550
 F 0 "R?" H 5550 7600 60  0000 C CNN
 F 1 "R_4k7_0402" H 5750 7400 60  0001 C CNN
-F 2 "antmicro-footprints:0402-res" H 5950 7750 60  0001 L CNN
+F 2 "sa800u-baseboard-hw-footprints:0402-res" H 5950 7750 60  0001 L CNN
 F 3 "" H 5750 7550 50  0001 C CNN
 F 4 "VISHAY" H 5950 7950 60  0001 L CNN "Manufacturer"
@@
 	5900 7550 6050 7550
 $Comp
-L antmicroResistors0402:R_4k7_0402 R?
+L sa800u-baseboard-hw:R_4k7_0402 R?
 U 1 1 62072AB9
 P 5750 7650
 F 0 "R?" H 5550 7700 60  0000 C CNN
 F 1 "R_4k7_0402" H 5750 7500 60  0001 C CNN
-F 2 "antmicro-footprints:0402-res" H 5950 7850 60  0001 L CNN
+F 2 "sa800u-baseboard-hw-footprints:0402-res" H 5950 7850 60  0001 L CNN
 F 3 "" H 5750 7650 50  0001 C CNN
 F 4 "VISHAY" H 5950 8050 60  0001 L CNN "Manufacturer"
@@
 	13850 4200 13850 4500
 $Comp
-L antmicroLEDIndicationDiscrete:ASMB-TTF0-0A20B D?
+L sa800u-baseboard-hw:ASMB-TTF0-0A20B D?
 U 1 1 620BAED1
 P 13650 4750
 F 0 "D?" V 13597 4372 60  0000 R CNN
 F 1 "ASMB-TTF0-0A20B" V 13703 4372 60  0000 R CNN
-F 2 "antmicro-footprints:PLCC6_3.5x3.7mm" H 13250 4050 60  0001 L CNN
+F 2 "sa800u-baseboard-hw-footprints:PLCC6_3.5x3.7mm" H 13250 4050 60  0001 L CNN
 F 3 "https://docs.broadcom.com/doc/ASMB-TTF0-0A20B-DS101" H 13850 5050 60  0001 L CNN
 F 4 "ASMB-TTF0-0A20B" H 13200 4150 60  0001 L CNN "MPN"
@@
 $EndComp
 $Comp
-L antmicroResistors0402:R_590R_0402 R?
+L sa800u-baseboard-hw:R_590R_0402 R?
 U 1 1 621057A9
 P 13650 5350
 F 0 "R?" H 13400 5300 60  0000 L CNN
 F 1 "R_590R_0402" H 13650 5200 60  0001 C CNN
-F 2 "antmicro-footprints:0402-res" H 13850 5550 60  0001 L CNN
+F 2 "sa800u-baseboard-hw-footprints:0402-res" H 13850 5550 60  0001 L CNN
 F 3 "" H 13650 5350 50  0001 C CNN
 F 4 "PANASONIC_ELECTRONIC_COMPONENTS" H 13850 5750 60  0001 L CNN "Manufacturer"
@@
 	13650 5200 13650 5000
 $Comp
-L power:GND #PWR?
+L sa800u-baseboard-hw:GND #PWR?
 U 1 1 62113B31
 P 13650 5700
@@
 Connection ~ 6150 7300
 $Comp
-L antmicroResistors0402:R_150R_0402 R?
+L sa800u-baseboard-hw:R_150R_0402 R?
 U 1 1 62198F27
 P 13450 5350
 F 0 "R?" H 13200 5300 60  0000 L CNN
 F 1 "R_150R_0402" H 13450 5200 60  0001 C CNN
-F 2 "antmicro-footprints:0402-res" H 13650 5550 60  0001 L CNN
+F 2 "sa800u-baseboard-hw-footprints:0402-res" H 13650 5550 60  0001 L CNN
 F 3 "" H 13450 5350 50  0001 C CNN
 F 4 "VISHAY" H 13650 5750 60  0001 L CNN "Manufacturer"
@@
 $EndComp
 $Comp
-L antmicroResistors0402:R_100R_0402 R?
+L sa800u-baseboard-hw:R_100R_0402 R?
 U 1 1 6219BF48
 P 13850 5350
 F 0 "R?" H 13600 5300 60  0000 L CNN
 F 1 "R_100R_0402" H 13850 5200 60  0001 C CNN
-F 2 "antmicro-footprints:0402-res" H 14050 5550 60  0001 L CNN
+F 2 "sa800u-baseboard-hw-footprints:0402-res" H 14050 5550 60  0001 L CNN
 F 3 "" H 13850 5350 50  0001 C CNN
 F 4 "BOURNS" H 14050 5750 60  0001 L CNN "Manufacturer"
