File: LCM.sch (KiCad schematic (older format))
At the start: 12 parts, among them J7 3-84952-0, J8 F52R-1A7H1-11020

Commit message: annotations
Parts:
- renumbered J7 to J5, J8 to J6, L1 to L11, L2 to L12, L3 to L13, L4 to L14, L5 to L15, L6 to L16, L7 to L17, L8 to L18, R46 to R71, R47 to R72
Changed lines of the file:
@@
 Connection ~ 2650 2350
 $Comp
-L power:+3V3 #PWR035
+L power:+3V3 #PWR062
 U 1 1 61BD4928
 P 2600 2350
-F 0 "#PWR035" H 2600 2200 50  0001 C CNN
+F 0 "#PWR062" H 2600 2200 50  0001 C CNN
 F 1 "+3V3" V 2615 2478 50  0000 L CNN
 F 2 "" H 2600 2350 50  0001 C CNN
@@
 Connection ~ 2750 2150
 $Comp
-L power:GND #PWR036
+L power:GND #PWR063
 U 1 1 61BD6C0B
 P 2750 2500
-F 0 "#PWR036" H 2750 2250 50  0001 C CNN
+F 0 "#PWR063" H 2750 2250 50  0001 C CNN
 F 1 "GND" H 2755 2327 50  0000 C CNN
 F 2 "" H 2750 2500 50  0001 C CNN
@@
 Connection ~ 9050 2500
 $Comp
-L power:+3V3 #PWR040
+L power:+3V3 #PWR065
 U 1 1 61BE8457
 P 8700 2900
-F 0 "#PWR040" H 8700 2750 50  0001 C CNN
+F 0 "#PWR065" H 8700 2750 50  0001 C CNN
 F 1 "+3V3" V 8715 3028 50  0000 L CNN
 F 2 "" H 8700 2900 50  0001 C CNN
@@
 Connection ~ 9050 2800
 $Comp
-L power:GND #PWR041
+L power:GND #PWR066
 U 1 1 61BEA7A9
 P 9050 3050
-F 0 "#PWR041" H 9050 2800 50  0001 C CNN
+F 0 "#PWR066" H 9050 2800 50  0001 C CNN
 F 1 "GND" H 9055 2877 50  0000 C CNN
 F 2 "" H 9050 3050 50  0001 C CNN
@@
 DSI0_CLK_P
 $Comp
-L antmicroResistors0402:R_4k7_0402 R47
+L antmicroResistors0402:R_4k7_0402 R72
 U 1 1 619BC4E7
 P 1750 2350
-F 0 "R47" V 1705 2420 60  0000 L CNN
+F 0 "R72" V 1705 2420 60  0000 L CNN
 F 1 "R_4k7_0402" H 1750 2200 60  0001 C CNN
 F 2 "antmicro-footprints:0402-res" H 1950 2550 60  0001 L CNN
@@
 $EndComp
 $Comp
-L antmicroResistors0402:R_4k7_0402 R46
+L antmicroResistors0402:R_4k7_0402 R71
 U 1 1 619BDFE3
 P 1500 2350
-F 0 "R46" V 1455 2420 60  0000 L CNN
+F 0 "R71" V 1455 2420 60  0000 L CNN
 F 1 "R_4k7_0402" H 1500 2200 60  0001 C CNN
 F 2 "antmicro-footprints:0402-res" H 1700 2550 60  0001 L CNN
@@
 	1500 2500 1500 2600
 $Comp
-L power:+3V3 #PWR033
+L power:+3V3 #PWR060
 U 1 1 619CDB8C
 P 1500 2600
-F 0 "#PWR033" H 1500 2450 50  0001 C CNN
+F 0 "#PWR060" H 1500 2450 50  0001 C CNN
 F 1 "+3V3" V 1515 2728 50  0000 L CNN
 F 2 "" H 1500 2600 50  0001 C CNN
@@
 $EndComp
 $Comp
-L power:+3V3 #PWR034
+L power:+3V3 #PWR061
 U 1 1 619CE012
 P 1750 2600
-F 0 "#PWR034" H 1750 2450 50  0001 C CNN
+F 0 "#PWR061" H 1750 2450 50  0001 C CNN
 F 1 "+3V3" V 1765 2728 50  0000 L CNN
 F 2 "" H 1750 2600 50  0001 C CNN
@@
 $EndComp
 $Comp
-L antmicroFCCConnectors:3-84952-0 J7
+L antmicroFCCConnectors:3-84952-0 J5
 U 1 1 619D8F59
 P 3350 2350
-F 0 "J7" H 3580 2337 50  0000 L CNN
+F 0 "J5" H 3580 2337 50  0000 L CNN
 F 1 "3-84952-0" H 3580 2246 50  0000 L CNN
 F 2 "antmicro-footprints:TE_3-84952-0" H 4150 2250 50  0001 L BNN
@@
 NoConn ~ 2950 3850
 $Comp
-L power:GND #PWR037
+L power:GND #PWR064
 U 1 1 61A1358A
 P 2950 4200
-F 0 "#PWR037" H 2950 3950 50  0001 C CNN
+F 0 "#PWR064" H 2950 3950 50  0001 C CNN
 F 1 "GND" H 2955 4027 50  0000 C CNN
 F 2 "" H 2950 4200 50  0001 C CNN
@@
 General purpose DSI for LCD
 $Comp
-L antmicroFCCConnectors:F52R-1A7H1-11020 J8
+L antmicroFCCConnectors:F52R-1A7H1-11020 J6
 U 1 1 61ADF1E8
 P 9500 900
-F 0 "J8" H 9828 -13 50  0000 L CNN
+F 0 "J6" H 9828 -13 50  0000 L CNN
 F 1 "F52R-1A7H1-11020" H 9828 -104 50  0000 L CNN
 F 2 "antmicro-footprints:F52R-1A7H1-11020" H 9500 900 50  0001 C CNN
@@
 P 1550 1100
 AR Path="/61B9B38A" Ref="L?"  Part="1"
-AR Path="/61BD2CC1/61B9B38A" Ref="L1"  Part="1"
-F 0 "L1" H 1900 1200 50  0000 C CNN
+AR Path="/61BD2CC1/61B9B38A" Ref="L11"  Part="1"
+F 0 "L11" H 1900 1200 50  0000 C CNN
 F 1 "NFP0QHB242HS2D" H 2200 1000 50  0000 C CNN
 F 2 "antmicro-footprints:FIL_NFP0QHB242HS2D" H 1550 1100 50  0001 C CNN
@@
 P 1550 1400
 AR Path="/61C048CC" Ref="L?"  Part="1"
-AR Path="/61BD2CC1/61C048CC" Ref="L2"  Part="1"
-F 0 "L2" H 1900 1500 50  0000 C CNN
+AR Path="/61BD2CC1/61C048CC" Ref="L12"  Part="1"
+F 0 "L12" H 1900 1500 50  0000 C CNN
 F 1 "NFP0QHB242HS2D" H 2200 1300 50  0000 C CNN
 F 2 "antmicro-footprints:FIL_NFP0QHB242HS2D" H 1550 1400 50  0001 C CNN
@@
 P 1550 1700
 AR Path="/61C3A309" Ref="L?"  Part="1"
-AR Path="/61BD2CC1/61C3A309" Ref="L3"  Part="1"
-F 0 "L3" H 1900 1800 50  0000 C CNN
+AR Path="/61BD2CC1/61C3A309" Ref="L13"  Part="1"
+F 0 "L13" H 1900 1800 50  0000 C CNN
 F 1 "NFP0QHB242HS2D" H 2200 1600 50  0000 C CNN
 F 2 "antmicro-footprints:FIL_NFP0QHB242HS2D" H 1550 1700 50  0001 C CNN
@@
 P 7000 1150
 AR Path="/61C65B0C" Ref="L?"  Part="1"
-AR Path="/61BD2CC1/61C65B0C" Ref="L4"  Part="1"
-F 0 "L4" H 7350 1250 50  0000 C CNN
+AR Path="/61BD2CC1/61C65B0C" Ref="L14"  Part="1"
+F 0 "L14" H 7350 1250 50  0000 C CNN
 F 1 "NFP0QHB242HS2D" H 7650 1050 50  0000 C CNN
 F 2 "antmicro-footprints:FIL_NFP0QHB242HS2D" H 7000 1150 50  0001 C CNN
@@
 P 7000 1450
 AR Path="/61C82351" Ref="L?"  Part="1"
-AR Path="/61BD2CC1/61C82351" Ref="L5"  Part="1"
-F 0 "L5" H 7350 1550 50  0000 C CNN
+AR Path="/61BD2CC1/61C82351" Ref="L15"  Part="1"
+F 0 "L15" H 7350 1550 50  0000 C CNN
 F 1 "NFP0QHB242HS2D" H 7650 1350 50  0000 C CNN
 F 2 "antmicro-footprints:FIL_NFP0QHB242HS2D" H 7000 1450 50  0001 C CNN
@@
 P 7000 1750
 AR Path="/61C82CCB" Ref="L?"  Part="1"
-AR Path="/61BD2CC1/61C82CCB" Ref="L6"  Part="1"
-F 0 "L6" H 7350 1850 50  0000 C CNN
+AR Path="/61BD2CC1/61C82CCB" Ref="L16"  Part="1"
+F 0 "L16" H 7350 1850 50  0000 C CNN
 F 1 "NFP0QHB242HS2D" H 7650 1650 50  0000 C CNN
 F 2 "antmicro-footprints:FIL_NFP0QHB242HS2D" H 7000 1750 50  0001 C CNN
@@
 P 7000 2050
 AR Path="/61C832C1" Ref="L?"  Part="1"
-AR Path="/61BD2CC1/61C832C1" Ref="L7"  Part="1"
-F 0 "L7" H 7350 2150 50  0000 C CNN
+AR Path="/61BD2CC1/61C832C1" Ref="L17"  Part="1"
+F 0 "L17" H 7350 2150 50  0000 C CNN
 F 1 "NFP0QHB242HS2D" H 7650 1950 50  0000 C CNN
 F 2 "antmicro-footprints:FIL_NFP0QHB242HS2D" H 7000 2050 50  0001 C CNN
@@
 P 7000 2350
 AR Path="/61C83C74" Ref="L?"  Part="1"
-AR Path="/61BD2CC1/61C83C74" Ref="L8"  Part="1"
-F 0 "L8" H 7350 2450 50  0000 C CNN
+AR Path="/61BD2CC1/61C83C74" Ref="L18"  Part="1"
+F 0 "L18" H 7350 2450 50  0000 C CNN
 F 1 "NFP0QHB242HS2D" H 7650 2250 50  0000 C CNN
 F 2 "antmicro-footprints:FIL_NFP0QHB242HS2D" H 7000 2350 50  0001 C CNN
@@
 	6200 2700 9300 2700
 $Comp
-L power:PWR_FLAG #FLG0102
+L power:PWR_FLAG #FLG02
 U 1 1 62BD2011
 P 1500 2600
-F 0 "#FLG0102" H 1500 2675 50  0001 C CNN
+F 0 "#FLG02" H 1500 2675 50  0001 C CNN
 F 1 "PWR_FLAG" V 1500 2728 50  0000 L CNN
 F 2 "" H 1500 2600 50  0001 C CNN

Commit message: Add local libs to fix CI
Parts:
- J5: footprint antmicro-footprints:TE_3-84952-0 -> sa800u-baseboard-hw-footprints:TE_3-84952-0; symbol antmicroFCCConnectors:3-84952-0 -> sa800u-baseboard-hw:3-84952-0
- J6: footprint antmicro-footprints:F52R-1A7H1-11020 -> sa800u-baseboard-hw-footprints:F52R-1A7H1-11020; symbol antmicroFCCConnectors:F52R-1A7H1-11020 -> sa800u-baseboard-hw:F52R-1A7H1-11020
- L11, L12, L13, L14, L15, L16, L17, L18: footprint antmicro-footprints:FIL_NFP0QHB242HS2D -> sa800u-baseboard-hw-footprints:FIL_NFP0QHB242HS2D; symbol antmicroFixedInductors:NFP0QHB242HS2D -> sa800u-baseboard-hw:NFP0QHB242HS2D
- R71, R72: footprint antmicro-footprints:0402-res -> sa800u-baseboard-hw-footprints:0402-res; symbol antmicroResistors0402:R_4k7_0402 -> sa800u-baseboard-hw:R_4k7_0402
Changed lines of the file:
@@
 Connection ~ 2650 2350
 $Comp
-L power:+3V3 #PWR062
+L sa800u-baseboard-hw:+3V3 #PWR062
 U 1 1 61BD4928
 P 2600 2350
@@
 Connection ~ 2750 2150
 $Comp
-L power:GND #PWR063
+L sa800u-baseboard-hw:GND #PWR063
 U 1 1 61BD6C0B
 P 2750 2500
@@
 Connection ~ 9050 2500
 $Comp
-L power:+3V3 #PWR065
+L sa800u-baseboard-hw:+3V3 #PWR065
 U 1 1 61BE8457
 P 8700 2900
@@
 Connection ~ 9050 2800
 $Comp
-L power:GND #PWR066
+L sa800u-baseboard-hw:GND #PWR066
 U 1 1 61BEA7A9
 P 9050 3050
@@
 DSI0_CLK_P
 $Comp
-L antmicroResistors0402:R_4k7_0402 R72
+L sa800u-baseboard-hw:R_4k7_0402 R72
 U 1 1 619BC4E7
 P 1750 2350
 F 0 "R72" V 1705 2420 60  0000 L CNN
 F 1 "R_4k7_0402" H 1750 2200 60  0001 C CNN
-F 2 "antmicro-footprints:0402-res" H 1950 2550 60  0001 L CNN
+F 2 "sa800u-baseboard-hw-footprints:0402-res" H 1950 2550 60  0001 L CNN
 F 3 "" H 1750 2350 50  0001 C CNN
 F 4 "VISHAY" H 1950 2750 60  0001 L CNN "Manufacturer"
@@
 $EndComp
 $Comp
-L antmicroResistors0402:R_4k7_0402 R71
+L sa800u-baseboard-hw:R_4k7_0402 R71
 U 1 1 619BDFE3
 P 1500 2350
 F 0 "R71" V 1455 2420 60  0000 L CNN
 F 1 "R_4k7_0402" H 1500 2200 60  0001 C CNN
-F 2 "antmicro-footprints:0402-res" H 1700 2550 60  0001 L CNN
+F 2 "sa800u-baseboard-hw-footprints:0402-res" H 1700 2550 60  0001 L CNN
 F 3 "" H 1500 2350 50  0001 C CNN
 F 4 "VISHAY" H 1700 2750 60  0001 L CNN "Manufacturer"
@@
 	1500 2500 1500 2600
 $Comp
-L power:+3V3 #PWR060
+L sa800u-baseboard-hw:+3V3 #PWR060
 U 1 1 619CDB8C
 P 1500 2600
@@
 $EndComp
 $Comp
-L power:+3V3 #PWR061
+L sa800u-baseboard-hw:+3V3 #PWR061
 U 1 1 619CE012
 P 1750 2600
@@
 $EndComp
 $Comp
-L antmicroFCCConnectors:3-84952-0 J5
+L sa800u-baseboard-hw:3-84952-0 J5
 U 1 1 619D8F59
 P 3350 2350
 F 0 "J5" H 3580 2337 50  0000 L CNN
 F 1 "3-84952-0" H 3580 2246 50  0000 L CNN
-F 2 "antmicro-footprints:TE_3-84952-0" H 4150 2250 50  0001 L BNN
+F 2 "sa800u-baseboard-hw-footprints:TE_3-84952-0" H 4150 2250 50  0001 L BNN
 F 3 "https://www.te.com/commerce/DocumentDelivery/DDEController?Action=showdoc&DocId=Data+Sheet%7F1-1773959-6-flexible-printed-circuit-con%7F0919%7Fpdf%7FEnglish%7FENG_DS_1-1773959-6-flexible-printed-circuit-con_0919.pdf%7F3-84952-0" H 4150 2250 50  0001 L BNN
 F 4 "3-84952-0" H 3580 2155 50  0001 L CNN "MPN"
@@
 NoConn ~ 2950 3850
 $Comp
-L power:GND #PWR064
+L sa800u-baseboard-hw:GND #PWR064
 U 1 1 61A1358A
 P 2950 4200
@@
 General purpose DSI for LCD
 $Comp
-L antmicroFCCConnectors:F52R-1A7H1-11020 J6
+L sa800u-baseboard-hw:F52R-1A7H1-11020 J6
 U 1 1 61ADF1E8
 P 9500 900
 F 0 "J6" H 9828 -13 50  0000 L CNN
 F 1 "F52R-1A7H1-11020" H 9828 -104 50  0000 L CNN
-F 2 "antmicro-footprints:F52R-1A7H1-11020" H 9500 900 50  0001 C CNN
+F 2 "sa800u-baseboard-hw-footprints:F52R-1A7H1-11020" H 9500 900 50  0001 C CNN
 F 3 "https://www.snapeda.com/parts/F52R-1A7H1-11020/Amphenol%20ICC%20(FCI)/datasheet/" H 9500 900 50  0001 C CNN
 F 4 "F52R-1A7H1-11020" H 9828 -195 50  0001 L CNN "MPN"
@@
 $EndComp
 $Comp
-L antmicroFixedInductors:NFP0QHB242HS2D L?
+L sa800u-baseboard-hw:NFP0QHB242HS2D L?
 U 1 1 61B9B38A
 P 1550 1100
@@
 F 0 "L11" H 1900 1200 50  0000 C CNN
 F 1 "NFP0QHB242HS2D" H 2200 1000 50  0000 C CNN
-F 2 "antmicro-footprints:FIL_NFP0QHB242HS2D" H 1550 1100 50  0001 C CNN
+F 2 "sa800u-baseboard-hw-footprints:FIL_NFP0QHB242HS2D" H 1550 1100 50  0001 C CNN
 F 3 "https://www.farnell.com/datasheets/2616945.pdf" H 1550 1100 50  0001 C CNN
 F 4 "NFP0QHB242HS2D" H 1550 1517 50  0001 C CNN "MPN"
@@
 	1250 1200 1250 1150
 $Comp
-L antmicroFixedInductors:NFP0QHB242HS2D L?
+L sa800u-baseboard-hw:NFP0QHB242HS2D L?
 U 1 1 61C048CC
 P 1550 1400
@@
 F 0 "L12" H 1900 1500 50  0000 C CNN
 F 1 "NFP0QHB242HS2D" H 2200 1300 50  0000 C CNN
-F 2 "antmicro-footprints:FIL_NFP0QHB242HS2D" H 1550 1400 50  0001 C CNN
+F 2 "sa800u-baseboard-hw-footprints:FIL_NFP0QHB242HS2D" H 1550 1400 50  0001 C CNN
 F 3 "https://www.farnell.com/datasheets/2616945.pdf" H 1550 1400 50  0001 C CNN
 F 4 "NFP0QHB242HS2D" H 1550 1817 50  0001 C CNN "MPN"
@@
 	1250 1350 700  1350
 $Comp
-L antmicroFixedInductors:NFP0QHB242HS2D L?
+L sa800u-baseboard-hw:NFP0QHB242HS2D L?
 U 1 1 61C3A309
 P 1550 1700
@@
 F 0 "L13" H 1900 1800 50  0000 C CNN
 F 1 "NFP0QHB242HS2D" H 2200 1600 50  0000 C CNN
-F 2 "antmicro-footprints:FIL_NFP0QHB242HS2D" H 1550 1700 50  0001 C CNN
+F 2 "sa800u-baseboard-hw-footprints:FIL_NFP0QHB242HS2D" H 1550 1700 50  0001 C CNN
 F 3 "https://www.farnell.com/datasheets/2616945.pdf" H 1550 1700 50  0001 C CNN
 F 4 "NFP0QHB242HS2D" H 1550 2117 50  0001 C CNN "MPN"
@@
 	1250 1750 700  1750
 $Comp
-L antmicroFixedInductors:NFP0QHB242HS2D L?
+L sa800u-baseboard-hw:NFP0QHB242HS2D L?
 U 1 1 61C65B0C
 P 7000 1150
@@
 F 0 "L14" H 7350 1250 50  0000 C CNN
 F 1 "NFP0QHB242HS2D" H 7650 1050 50  0000 C CNN
-F 2 "antmicro-footprints:FIL_NFP0QHB242HS2D" H 7000 1150 50  0001 C CNN
+F 2 "sa800u-baseboard-hw-footprints:FIL_NFP0QHB242HS2D" H 7000 1150 50  0001 C CNN
 F 3 "https://www.farnell.com/datasheets/2616945.pdf" H 7000 1150 50  0001 C CNN
 F 4 "NFP0QHB242HS2D" H 7000 1567 50  0001 C CNN "MPN"
@@
 $EndComp
 $Comp
-L antmicroFixedInductors:NFP0QHB242HS2D L?
+L sa800u-baseboard-hw:NFP0QHB242HS2D L?
 U 1 1 61C82351
 P 7000 1450
@@
 F 0 "L15" H 7350 1550 50  0000 C CNN
 F 1 "NFP0QHB242HS2D" H 7650 1350 50  0000 C CNN
-F 2 "antmicro-footprints:FIL_NFP0QHB242HS2D" H 7000 1450 50  0001 C CNN
+F 2 "sa800u-baseboard-hw-footprints:FIL_NFP0QHB242HS2D" H 7000 1450 50  0001 C CNN
 F 3 "https://www.farnell.com/datasheets/2616945.pdf" H 7000 1450 50  0001 C CNN
 F 4 "NFP0QHB242HS2D" H 7000 1867 50  0001 C CNN "MPN"
@@
 $EndComp
 $Comp
-L antmicroFixedInductors:NFP0QHB242HS2D L?
+L sa800u-baseboard-hw:NFP0QHB242HS2D L?
 U 1 1 61C82CCB
 P 7000 1750
@@
 F 0 "L16" H 7350 1850 50  0000 C CNN
 F 1 "NFP0QHB242HS2D" H 7650 1650 50  0000 C CNN
-F 2 "antmicro-footprints:FIL_NFP0QHB242HS2D" H 7000 1750 50  0001 C CNN
+F 2 "sa800u-baseboard-hw-footprints:FIL_NFP0QHB242HS2D" H 7000 1750 50  0001 C CNN
 F 3 "https://www.farnell.com/datasheets/2616945.pdf" H 7000 1750 50  0001 C CNN
 F 4 "NFP0QHB242HS2D" H 7000 2167 50  0001 C CNN "MPN"
@@
 $EndComp
 $Comp
-L antmicroFixedInductors:NFP0QHB242HS2D L?
+L sa800u-baseboard-hw:NFP0QHB242HS2D L?
 U 1 1 61C832C1
 P 7000 2050
@@
 F 0 "L17" H 7350 2150 50  0000 C CNN
 F 1 "NFP0QHB242HS2D" H 7650 1950 50  0000 C CNN
-F 2 "antmicro-footprints:FIL_NFP0QHB242HS2D" H 7000 2050 50  0001 C CNN
+F 2 "sa800u-baseboard-hw-footprints:FIL_NFP0QHB242HS2D" H 7000 2050 50  0001 C CNN
 F 3 "https://www.farnell.com/datasheets/2616945.pdf" H 7000 2050 50  0001 C CNN
 F 4 "NFP0QHB242HS2D" H 7000 2467 50  0001 C CNN "MPN"
@@
 $EndComp
 $Comp
-L antmicroFixedInductors:NFP0QHB242HS2D L?
+L sa800u-baseboard-hw:NFP0QHB242HS2D L?
 U 1 1 61C83C74
 P 7000 2350
@@
 F 0 "L18" H 7350 2450 50  0000 C CNN
 F 1 "NFP0QHB242HS2D" H 7650 2250 50  0000 C CNN
-F 2 "antmicro-footprints:FIL_NFP0QHB242HS2D" H 7000 2350 50  0001 C CNN
+F 2 "sa800u-baseboard-hw-footprints:FIL_NFP0QHB242HS2D" H 7000 2350 50  0001 C CNN
 F 3 "https://www.farnell.com/datasheets/2616945.pdf" H 7000 2350 50  0001 C CNN
 F 4 "NFP0QHB242HS2D" H 7000 2767 50  0001 C CNN "MPN"
@@
 	6200 2700 9300 2700
 $Comp
-L power:PWR_FLAG #FLG02
+L sa800u-baseboard-hw:PWR_FLAG #FLG02
 U 1 1 62BD2011
 P 1500 2600

Commit message: fixing ERC errors
Connections:
- net labels added: 3V3
- net labels removed: +3V3
Other:
- note added: "Add some TVS diodes for protection."
Changed lines of the file:
@@
 	2650 2350 2600 2350
 Connection ~ 2650 2350
-$Comp
-L sa800u-baseboard-hw:+3V3 #PWR062
-U 1 1 61BD4928
-P 2600 2350
-F 0 "#PWR062" H 2600 2200 50  0001 C CNN
-F 1 "+3V3" V 2615 2478 50  0000 L CNN
-F 2 "" H 2600 2350 50  0001 C CNN
-F 3 "" H 2600 2350 50  0001 C CNN
-	1    2600 2350
-	0    -1   -1   0
-$EndComp
 Wire Wire Line
 	2750 2150 2750 2500
@@
 	1    0    0    -1
 $EndComp
-Text Label 700  1150 0    50   ~ 0
-DSI0_LN1_P
-Text Label 700  1050 0    50   ~ 0
-DSI0_LN1_N
-Text Label 700  1650 0    50   ~ 0
-DSI0_LN0_N
-Text Label 700  1750 0    50   ~ 0
-DSI0_LN0_P
-Text Label 700  1450 0    50   ~ 0
-DSI0_CLK_P
-Text Label 700  1350 0    50   ~ 0
-DSI0_CLK_N
-Text Label 550  2050 0    50   ~ 0
-TP_I2C_SDA
-Text Label 550  1950 0    50   ~ 0
-TP_I2C_SCL
-Text Label 6000 1200 0    50   ~ 0
-DSI0_LN3_P
-Text Label 6000 1100 0    50   ~ 0
-DSI0_LN3_N
-Text Label 6000 1500 0    50   ~ 0
-DSI0_LN2_P
-Text Label 6000 1400 0    50   ~ 0
-DSI0_LN2_N
-Text Label 6000 1700 0    50   ~ 0
-DSI0_LN1_N
-Text Label 6000 1800 0    50   ~ 0
-DSI0_LN1_P
-Text Label 6000 2000 0    50   ~ 0
-DSI0_LN0_N
-Text Label 6000 2100 0    50   ~ 0
-DSI0_LN0_P
 Wire Wire Line
 	9300 1000 9050 1000
@@
 Wire Wire Line
 	9050 2200 9300 2200
-Text Label 6200 2600 0    50   ~ 0
-TP_I2C_SCL
-Text Label 6200 2700 0    50   ~ 0
-TP_I2C_SDA
 Wire Wire Line
 	9050 2200 9050 2500
@@
 	9050 2800 9300 2800
 Connection ~ 9050 2500
-$Comp
-L sa800u-baseboard-hw:+3V3 #PWR065
-U 1 1 61BE8457
-P 8700 2900
-F 0 "#PWR065" H 8700 2750 50  0001 C CNN
-F 1 "+3V3" V 8715 3028 50  0000 L CNN
-F 2 "" H 8700 2900 50  0001 C CNN
-F 3 "" H 8700 2900 50  0001 C CNN
-	1    8700 2900
-	0    -1   -1   0
-$EndComp
 Wire Wire Line
 	8700 2900 9300 2900
@@
 Wire Wire Line
 	7300 2400 9300 2400
-Text Label 6000 2300 0    50   ~ 0
-DSI0_CLK_N
-Text Label 6000 2400 0    50   ~ 0
-DSI0_CLK_P
 $Comp
 L sa800u-baseboard-hw:R_4k7_0402 R72
@@
 Wire Wire Line
 	1500 2500 1500 2600
-$Comp
-L sa800u-baseboard-hw:+3V3 #PWR060
-U 1 1 619CDB8C
-P 1500 2600
-F 0 "#PWR060" H 1500 2450 50  0001 C CNN
-F 1 "+3V3" V 1515 2728 50  0000 L CNN
-F 2 "" H 1500 2600 50  0001 C CNN
-F 3 "" H 1500 2600 50  0001 C CNN
-	1    1500 2600
-	-1   0    0    1
-$EndComp
-$Comp
-L sa800u-baseboard-hw:+3V3 #PWR061
-U 1 1 619CE012
-P 1750 2600
-F 0 "#PWR061" H 1750 2450 50  0001 C CNN
-F 1 "+3V3" V 1765 2728 50  0000 L CNN
-F 2 "" H 1750 2600 50  0001 C CNN
-F 3 "" H 1750 2600 50  0001 C CNN
-	1    1750 2600
-	-1   0    0    1
-$EndComp
 $Comp
 L sa800u-baseboard-hw:3-84952-0 J5
@@
 	0    1    1    0
 $EndComp
-Connection ~ 1500 2600
+Text GLabel 700  1050 0    50   Input ~ 0
+DSI0_LN1_N
+Text GLabel 700  1150 0    50   Input ~ 0
+DSI0_LN1_P
+Text GLabel 700  1350 0    50   Input ~ 0
+DSI0_CLK_N
+Text GLabel 700  1450 0    50   Input ~ 0
+DSI0_CLK_P
+Text GLabel 700  1650 0    50   Input ~ 0
+DSI0_LN0_N
+Text GLabel 700  1750 0    50   Input ~ 0
+DSI0_LN0_P
+Text GLabel 550  1950 0    50   Input ~ 0
+TP_I2C_SCL
+Text GLabel 550  2050 0    50   Input ~ 0
+TP_I2C_SDA
+Text GLabel 1500 2600 3    50   Input ~ 0
+3V3
+Text GLabel 1750 2600 3    50   Input ~ 0
+3V3
+Text GLabel 2600 2350 0    50   Input ~ 0
+3V3
+Text GLabel 6000 1100 0    50   Input ~ 0
+DSI0_LN3_N
+Text GLabel 6000 1200 0    50   Input ~ 0
+DSI0_LN3_P
+Text GLabel 6000 1400 0    50   Input ~ 0
+DSI0_LN2_N
+Text GLabel 6000 1500 0    50   Input ~ 0
+DSI0_LN2_P
+Text GLabel 6000 1700 0    50   Input ~ 0
+DSI0_LN1_N
+Text GLabel 6000 1800 0    50   Input ~ 0
+DSI0_LN1_P
+Text GLabel 6000 2000 0    50   Input ~ 0
+DSI0_LN0_N
+Text GLabel 6000 2100 0    50   Input ~ 0
+DSI0_LN0_P
+Text GLabel 6000 2300 0    50   Input ~ 0
+DSI0_CLK_N
+Text GLabel 6000 2400 0    50   Input ~ 0
+DSI0_CLK_P
+Text GLabel 6200 2600 0    50   Input ~ 0
+TP_I2C_SCL
+Text GLabel 6200 2700 0    50   Input ~ 0
+TP_I2C_SDA
+Text GLabel 8700 2900 0    50   Input ~ 0
+3V3
+Text Notes 3600 3300 0    50   ~ 0
+Add some TVS diodes for protection.
 $EndSCHEMATC

Commit message: Cleanup LCM, add voltage translator to LCM I2C
Parts:
- removed R71, R72: R_4k7_0402, sa800u-baseboard-hw-footprints:0402-res, symbol sa800u-baseboard-hw:R_4k7_0402
- added C? (x2): C_100n_0402, sa800u-baseboard-hw-footprints:0402-cap, symbol sa800u-baseboard-hw:C_100n_0402
- added R? (x4): R_2k_0402, antmicro-footprints:0402-res, symbol antmicroResistors0402:R_2k_0402
- added U?: NTS0102GT, antmicro-footprints:PSON50P100X195X50-8N, symbol antmicroLogicTranslatorsLevelShifters:NTS0102GT
Connections:
- net labels added: 3V3_SYS, LVS1A_1V8, TP_I2C_SCL_3V3, TP_I2C_SDA_3V3
- net labels removed: 3V3
- wire segments 104 -> 133
Other:
- moved on the sheet: J5, J6, L11, L12, L13, L14, L15, L16, L17, L18

Commit message: Loclib
Parts:
- R? (x4): footprint antmicro-footprints:0402-res -> sa800u-baseboard-hw-footprints:0402-res; symbol antmicroResistors0402:R_2k_0402 -> sa800u-baseboard-hw:R_2k_0402
- U?: footprint antmicro-footprints:PSON50P100X195X50-8N -> sa800u-baseboard-hw-footprints:PSON50P100X195X50-8N; symbol antmicroLogicTranslatorsLevelShifters:NTS0102GT -> sa800u-baseboard-hw:NTS0102GT
Changed lines of the file:
@@
 Add some TVS diodes for protection.
 $Comp
-L antmicroLogicTranslatorsLevelShifters:NTS0102GT U?
+L sa800u-baseboard-hw:NTS0102GT U?
 U 1 1 65E71148
 P 3675 7675
 F 0 "U?" H 3675 8190 50  0000 C CNN
 F 1 "NTS0102GT" H 3675 8099 50  0000 C CNN
-F 2 "antmicro-footprints:PSON50P100X195X50-8N" H 3575 8175 50  0001 C CNN
+F 2 "sa800u-baseboard-hw-footprints:PSON50P100X195X50-8N" H 3575 8175 50  0001 C CNN
 F 3 "http://www.farnell.com/datasheets/1760723.pdf" H 4325 8425 50  0001 C CNN
 F 4 "NTS0102GT" H 3675 8190 50  0001 C CNN "MPN"
@@
 $EndComp
 $Comp
-L antmicroResistors0402:R_2k_0402 R?
+L sa800u-baseboard-hw:R_2k_0402 R?
 U 1 1 6605EB55
 P 2800 7325
 F 0 "R?" V 2845 7255 60  0000 R CNN
 F 1 "R_2k_0402" H 2800 7175 60  0001 C CNN
-F 2 "antmicro-footprints:0402-res" H 3000 7525 60  0001 L CNN
+F 2 "sa800u-baseboard-hw-footprints:0402-res" H 3000 7525 60  0001 L CNN
 F 3 "" H 2800 7325 50  0001 C CNN
 F 4 "VISHAY" H 3000 7725 60  0001 L CNN "Manufacturer"
@@
 	2700 7475 2700 7625
 $Comp
-L antmicroResistors0402:R_2k_0402 R?
+L sa800u-baseboard-hw:R_2k_0402 R?
 U 1 1 6605EB4C
 P 2700 7325
 F 0 "R?" V 2745 7394 60  0000 L CNN
 F 1 "R_2k_0402" H 2700 7175 60  0001 C CNN
-F 2 "antmicro-footprints:0402-res" H 2900 7525 60  0001 L CNN
+F 2 "sa800u-baseboard-hw-footprints:0402-res" H 2900 7525 60  0001 L CNN
 F 3 "" H 2700 7325 50  0001 C CNN
 F 4 "VISHAY" H 2900 7725 60  0001 L CNN "Manufacturer"
@@
 	4550 7475 4550 7525
 $Comp
-L antmicroResistors0402:R_2k_0402 R?
+L sa800u-baseboard-hw:R_2k_0402 R?
 U 1 1 660892CF
 P 4550 7325
 F 0 "R?" V 4595 7255 60  0000 R CNN
 F 1 "R_2k_0402" H 4550 7175 60  0001 C CNN
-F 2 "antmicro-footprints:0402-res" H 4750 7525 60  0001 L CNN
+F 2 "sa800u-baseboard-hw-footprints:0402-res" H 4750 7525 60  0001 L CNN
 F 3 "" H 4550 7325 50  0001 C CNN
 F 4 "VISHAY" H 4750 7725 60  0001 L CNN "Manufacturer"
@@
 $EndComp
 $Comp
-L antmicroResistors0402:R_2k_0402 R?
+L sa800u-baseboard-hw:R_2k_0402 R?
 U 1 1 660892C6
 P 4650 7325
 F 0 "R?" V 4695 7394 60  0000 L CNN
 F 1 "R_2k_0402" H 4650 7175 60  0001 C CNN
-F 2 "antmicro-footprints:0402-res" H 4850 7525 60  0001 L CNN
+F 2 "sa800u-baseboard-hw-footprints:0402-res" H 4850 7525 60  0001 L CNN
 F 3 "" H 4650 7325 50  0001 C CNN
 F 4 "VISHAY" H 4850 7725 60  0001 L CNN "Manufacturer"
