File: usb-pd.sch (KiCad schematic (older format))
At the start: 39 parts, among them J12 12401598E4_2A, Q7 SQS401EN-T1_BE3, U18 STUSB4500QTR

Commit message: Enumerate parts
Parts:
- gave numbers to parts that had none: 2
Changed lines of the file:
@@
 I2C10_SDA
 $Comp
-L sa800u-baseboard-hw:GND #PWR?
+L sa800u-baseboard-hw:GND #PWR0197
 U 1 1 629F9470
 P 4850 5225
-F 0 "#PWR?" H 4850 4975 50  0001 C CNN
+F 0 "#PWR0197" H 4850 4975 50  0001 C CNN
 F 1 "GND" H 4855 5052 50  0000 C CNN
 F 2 "" H 4850 5225 50  0001 C CNN
@@
 $EndComp
 $Comp
-L sa800u-baseboard-hw:PESD18VF1BSFYL D?
+L sa800u-baseboard-hw:PESD18VF1BSFYL D31
 U 1 1 629F9478
 P 4850 4975
-F 0 "D?" V 4809 5078 60  0000 L CNN
+F 0 "D31" V 4809 5078 60  0000 L CNN
 F 1 "PESD18VF1BSFYL" V 4915 5078 60  0000 L CNN
 F 2 "sa800u-baseboard-hw-footprints:RESC0603X26N" H 4850 4525 100 0001 L CNN
@@
 $EndComp
 $Comp
-L sa800u-baseboard-hw:GND #PWR?
+L sa800u-baseboard-hw:GND #PWR0275
 U 1 1 62A0542C
 P 4650 5250
-F 0 "#PWR?" H 4650 5000 50  0001 C CNN
+F 0 "#PWR0275" H 4650 5000 50  0001 C CNN
 F 1 "GND" H 4655 5077 50  0000 C CNN
 F 2 "" H 4650 5250 50  0001 C CNN
@@
 $EndComp
 $Comp
-L sa800u-baseboard-hw:PESD18VF1BSFYL D?
+L sa800u-baseboard-hw:PESD18VF1BSFYL D23
 U 1 1 62A05434
 P 4650 5000
-F 0 "D?" V 4609 4897 60  0000 R CNN
+F 0 "D23" V 4609 4897 60  0000 R CNN
 F 1 "PESD18VF1BSFYL" V 4715 4897 60  0000 R CNN
 F 2 "sa800u-baseboard-hw-footprints:RESC0603X26N" H 4650 4550 100 0001 L CNN
