File: psu.kicad_sch (KiCad schematic)
At the start: 116 parts, among them J10 Molex_Nano-Fit-1053xx_xx02-ho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, Q10 BSS84, Q11 Si7223DN, Q12 Si7223DN, Q13 BSS84, Q14 BSS84, Q15 BSS84PH6327XTSA2, Q16 SQS401EN-T1_BE3, Q8 BSS84, Q9 Si7223DN, U17 LTC4417IUF, U18 LMV431IM5, U22 AP62301WU-7

Commit message: Introduce component standardization
Parts:
- C121, C122, C126, C127, C131: footprint sa800u-baseboard-hw-footprints:0603-cap -> sa800u-baseboard-hw-footprints:C_0603_1608Metric; Author (none) -> Antmicro; License (none) -> Apache-2.0
- C123, C124, C125, C138: footprint sa800u-baseboard-hw-footprints:0402-cap -> sa800u-baseboard-hw-footprints:C_0402_1005Metric; Author (none) -> Antmicro; Dielectric (none) -> X5R; License (none) -> Apache-2.0; Voltage (none) -> 50V
- C128, C129, C130, C135, C136, C137, C139, C140, C141: value (none) -> C_22u_0603; footprint (none) -> sa800u-baseboard-hw-footprints:C_0603_1608Metric; Author (none) -> Antmicro; License (none) -> Apache-2.0; Manufacturer MURATA -> Murata
- C132, C133, C134: renamed from C?; value (none) -> C_100n_0402; footprint (none) -> sa800u-baseboard-hw-footprints:C_0402_1005Metric; Author (none) -> Antmicro; Dielectric (none) -> X5R; License (none) -> Apache-2.0; MPN 0402X104K6R3CT -> GRM155R61H104KE14D; Manufacturer Walsin -> Murata; Voltage (none) -> 50V
- C142, C143: footprint sa800u-baseboard-hw-footprints:0603-cap -> sa800u-baseboard-hw-footprints:C_0603_1608Metric; Author (none) -> Antmicro; License (none) -> Apache-2.0; Manufacturer MURATA -> Murata
- D24, D25, D26, D27, D28: footprint sa800u-baseboard-hw-footprints:LED_0603 -> sa800u-baseboard-hw-footprints:LED_0603_1608Metric_G; symbol sa800u-baseboard-hw:KP-1608EC -> sa800u-baseboard-hw:LED_G_0603_KP-1608ZGC; Author (none) -> Antmicro; License (none) -> Apache-2.0; MPN KP-1608EC -> KP-1608ZGC; Manufacturer KINGBRIGHT -> Kingbright
- J10: value Molex_Nano-Fit-1053xx_xx02-horizontal_vertical -> Conn_Molex_NanoFit_1053131202; footprint sa800u-baseboard-hw-footprints:Molex_Nano-Fit_1053xx-xx02_1x02_P2.50mm_Horizontal -> sa800u-baseboard-hw-footprints:Conn_Molex_NanoFit_1053131202; symbol sa800u-baseboard-hw:Molex_Nano-Fit-1053xx_xx02-horizontal_vertical -> sa800u-baseboard-hw:Conn_Molex_NanoFit_1053131202; Author (none) -> Antmicro; License (none) -> Apache-2.0
- L26, L27, L28: value XEL4030-222MEC -> L_2u2_6.1A_XEL4030; footprint sa800u-baseboard-hw-footprints:Coilcraft-XEL4030 -> sa800u-baseboard-hw-footprints:L_Coilcraft_XEL4030; symbol sa800u-baseboard-hw:XEL4030-222MEC -> sa800u-baseboard-hw:L_2u2_6.1A_XEL4030; Author (none) -> Antmicro; License (none) -> Apache-2.0
- L29: renamed from L?; value (none) -> L_2u2_6.1A_XEL4030; footprint (none) -> sa800u-baseboard-hw-footprints:L_Coilcraft_XEL4030; symbol sa800u-baseboard-hw:XEL4030-222MEC -> sa800u-baseboard-hw:L_2u2_6.1A_XEL4030; Author (none) -> Antmicro; License (none) -> Apache-2.0
- Q10, Q13, Q14, Q16, Q8: Author (none) -> Antmicro; License (none) -> Apache-2.0
- Q11, Q12, Q9: Author (none) -> Antmicro; License (none) -> Apache-2.0; Manufacturer VISHAY -> Vishay
- Q15: Author (none) -> Antmicro; License (none) -> Apache-2.0; Manufacturer INFINEON -> Infineon Technologies
- R105, R108, R112: footprint sa800u-baseboard-hw-footprints:0402-res -> sa800u-baseboard-hw-footprints:R_0402_1005Metric; Author (none) -> Antmicro; License (none) -> Apache-2.0; MPN RC0402FR-07200KL -> CR0402-FX-2003GLF; Manufacturer YAGEO_(PHYCOMP) -> Bourns; Tolerance (none) -> 1%
- R106, R109, R113: footprint sa800u-baseboard-hw-footprints:0402-res -> sa800u-baseboard-hw-footprints:R_0402_1005Metric; Author (none) -> Antmicro; License (none) -> Apache-2.0; MPN MCWR04X3902FTL -> CR0402-FX-3902GLF; Manufacturer MULTICOMP -> Bourns; Tolerance (none) -> 1%
- R107, R110, R114: footprint sa800u-baseboard-hw-footprints:0402-res -> sa800u-baseboard-hw-footprints:R_0402_1005Metric; Author (none) -> Antmicro; License (none) -> Apache-2.0; Tolerance (none) -> 1%
- R111, R115, R116, R121, R122, R127, R128, R130, R131, R132, R133, R134, R138, R139, R142: footprint sa800u-baseboard-hw-footprints:0402-res -> sa800u-baseboard-hw-footprints:R_0402_1005Metric; Author (none) -> Antmicro; License (none) -> Apache-2.0; MPN CRCW040210K0FKEDHP -> CR0402-FX-1002GLF; Manufacturer VISHAY -> Bourns; Tolerance (none) -> 1%
- R117: footprint sa800u-baseboard-hw-footprints:0402-res -> sa800u-baseboard-hw-footprints:R_0402_1005Metric; Author (none) -> Antmicro; License (none) -> Apache-2.0; MPN ERJ-2RKF2553X -> CR0402-FX-2553GLF; Manufacturer PANASONIC_ELECTRONIC_COMPONENTS -> Bourns; Tolerance (none) -> 1%
- R118, R119, R120: value R_1M0_0402 -> R_1M_0402; footprint sa800u-baseboard-hw-footprints:0402-res -> sa800u-baseboard-hw-footprints:R_0402_1005Metric; symbol sa800u-baseboard-hw:R_1M0_0402 -> sa800u-baseboard-hw:R_1M_0402; Author (none) -> Antmicro; License (none) -> Apache-2.0; MPN CRG0402F1M0 -> CR0402-FX-1004GLF; Manufacturer TE CONNECTIVITY -> Bourns; Tolerance (none) -> 1%; Val 1M0 -> 1M
- R123: footprint sa800u-baseboard-hw-footprints:0402-res -> sa800u-baseboard-hw-footprints:R_0402_1005Metric; Author (none) -> Antmicro; License (none) -> Apache-2.0; MPN RC0402FR-077K5L -> CR0402-FX-7501GLF; Manufacturer YAGEO -> Bourns; Tolerance (none) -> 1%
- R124, R125: footprint sa800u-baseboard-hw-footprints:0402-res -> sa800u-baseboard-hw-footprints:R_0402_1005Metric; Author (none) -> Antmicro; License (none) -> Apache-2.0; MPN RC0402FR-072K2L -> CR0402-FX-2201GLF; Manufacturer YAGEO -> Bourns; Tolerance (none) -> 1%
- R126: footprint sa800u-baseboard-hw-footprints:0402-res -> sa800u-baseboard-hw-footprints:R_0402_1005Metric; Author (none) -> Antmicro; License (none) -> Apache-2.0; Manufacturer BOURNS -> Bourns; Tolerance (none) -> 1%
- R129: footprint sa800u-baseboard-hw-footprints:0402-res -> sa800u-baseboard-hw-footprints:R_0402_1005Metric; Author (none) -> Antmicro; License (none) -> Apache-2.0; MPN CRCW040225K5FKED -> CR0402-FX-2552GLF; Manufacturer Vishay -> Bourns; Tolerance (none) -> 1%
- R135: footprint sa800u-baseboard-hw-footprints:0402-res -> sa800u-baseboard-hw-footprints:R_0402_1005Metric; Author (none) -> Antmicro; License (none) -> Apache-2.0; MPN MCWR04X7502FTL -> CR0402-FX-7502GLF; Manufacturer MULTICOMP -> Bourns; Tolerance (none) -> 1%
- R136, R140: footprint sa800u-baseboard-hw-footprints:0402-res -> sa800u-baseboard-hw-footprints:R_0402_1005Metric; Author (none) -> Antmicro; License (none) -> Apache-2.0; MPN CRCW040220K0FKED -> CR0402-FX-2002GLF; Manufacturer VISHAY -> Bourns; Tolerance (none) -> 1%
- R137: footprint sa800u-baseboard-hw-footprints:0402-res -> sa800u-baseboard-hw-footprints:R_0402_1005Metric; Author (none) -> Antmicro; License (none) -> Apache-2.0; MPN CRCW040231K6FKEDC -> CR0402-FX-3162GLF; Manufacturer Vishay -> Bourns; Tolerance (none) -> 1%
- R141: footprint sa800u-baseboard-hw-footprints:0402-res -> sa800u-baseboard-hw-footprints:R_0402_1005Metric; Author (none) -> Antmicro; License (none) -> Apache-2.0; MPN ERJ-2RKF5232X -> CR0402-FX-5232GLF; Manufacturer Panasonic -> Bourns; Tolerance (none) -> 1%
- TP48, TP49, TP50, TP51, TP52, TP53, TP54, TP55, TP57, TP59, TP60, TP64, TP65, TP66, TP67, TP69: value TP_SMD_0_75MM -> TP_0.75mm_SMD; footprint sa800u-baseboard-hw-footprints:Testpoint_smd_0_75mm -> sa800u-baseboard-hw-footprints:TP_SMD_0.75mm; symbol sa800u-baseboard-hw:TP_SMD_0_75MM -> sa800u-baseboard-hw:TP_0.75mm_SMD; Author (none) -> Antmicro; License (none) -> Apache-2.0
- TP56, TP58, TP61, TP62, TP63, TP68, TP70, TP71, TP72, TP73, TP74, TP75, TP76, TP77: renamed from TP?; value (none) -> TP_0.75mm_SMD; footprint (none) -> sa800u-baseboard-hw-footprints:TP_SMD_0.75mm; symbol sa800u-baseboard-hw:TP -> sa800u-baseboard-hw:TP_0.75mm_SMD; Author (none) -> Antmicro; License (none) -> Apache-2.0
- U17: value LTC4417IUF -> LTC4417_QFN; footprint sa800u-baseboard-hw-footprints:LTC4417IUF-TRPBF -> sa800u-baseboard-hw-footprints:QFN-24-1EP_4x4mm_EP2.1x2.1mm; symbol sa800u-baseboard-hw:LTC4417IUF -> sa800u-baseboard-hw:LTC4417_QFN; Author (none) -> Antmicro; License (none) -> Apache-2.0
- U18: value LMV431IM5 -> LMV431_SOT-23-5; symbol sa800u-baseboard-hw:LMV431IM5 -> sa800u-baseboard-hw:LMV431_SOT-23-5; Author (none) -> Antmicro; License (none) -> Apache-2.0
- U19, U20, U21: value (none) -> AP62301WU-7; footprint (none) -> sa800u-baseboard-hw-footprints:AP62301WU-7-TSOT23-6; Author (none) -> Antmicro; License (none) -> Apache-2.0
- U22: footprint sa800u-baseboard-hw-footprints:TSOT23-6 -> sa800u-baseboard-hw-footprints:AP62301WU-7-TSOT23-6; Author (none) -> Antmicro; License (none) -> Apache-2.0
Connections:
- net at L27.1, U20.2 (SW): now also C133.2; no longer C133.1
- net at U20.6 (BST): now also C133.1; no longer C133.2
- net at L26.1, U19.2 (SW): now also C132.2; no longer C132.1
- net at U19.6 (BST): now also C132.1; no longer C132.2
- net at L28.1, U21.2 (SW): now also C134.2; no longer C134.1
- net at U21.6 (BST): now also C134.1; no longer C134.2
- net G3: now reaches C125.1, Q12.2 (G1), Q12.4 (G2), TP53.1, U17.13 (G3)
- net G2: now reaches C124.1, Q11.2 (G1), Q11.4 (G2), TP52.1, U17.15 (G2)
- net G1: now reaches C123.1, Q9.2 (G1), Q9.4 (G2), TP51.1, U17.17 (G1)
Other:
- moved on the sheet: C121, C122, C123, C124, C125, C126, C127, C128, C129, C130, C131, C132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

Commit message: Add OHP assets
Other:
- company: (none) -> Antmicro Ltd.
Changed lines of the file:
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@@
   (title_block
     (title "SA800U (Snapdragon 845) Baseboard")
-    (date "2023-07-27")
-    (rev "1.0.2")
+    (date "2023-10-19")
+    (rev "1.0.3")
+    (company "Antmicro Ltd.")
     (comment 1 "www.antmicro.com")
-    (comment 2 "Antmicro Ltd.")
   )
   (junction (at 325.628 221.615) (diameter 0) (color 0 0 0 0)
@@
     (pin "2")
   )
-  (symbol (lib_id "sa800u-baseboard-hw:L_2u2_6.1A_XEL4030") (at 326.39 186.69 0) (unit 1)
+  (symbol (lib_name "L_2u2_6.1A_XEL4030_3") (lib_id "sa800u-baseboard-hw:L_2u2_6.1A_XEL4030") (at 326.39 186.69 0) (unit 1)
     (in_bom yes) (on_board yes) (fields_autoplaced)
     (property "Reference" "L27" (id 0) (at 328.93 181.61 0))
@@
     (pin "1")
   )
-  (symbol (lib_id "sa800u-baseboard-hw:L_2u2_6.1A_XEL4030") (at 328.168 151.765 0) (unit 1)
+  (symbol (lib_name "L_2u2_6.1A_XEL4030_2") (lib_id "sa800u-baseboard-hw:L_2u2_6.1A_XEL4030") (at 328.168 151.765 0) (unit 1)
     (in_bom yes) (on_board yes) (fields_autoplaced)
     (property "Reference" "L26" (id 0) (at 330.708 146.05 0))
@@
     (pin "1")
   )
-  (symbol (lib_id "sa800u-baseboard-hw:L_2u2_6.1A_XEL4030") (at 355.092 69.215 0) (unit 1)
+  (symbol (lib_name "L_2u2_6.1A_XEL4030_1") (lib_id "sa800u-baseboard-hw:L_2u2_6.1A_XEL4030") (at 355.092 69.215 0) (unit 1)
     (in_bom yes) (on_board yes) (fields_autoplaced)
     (property "Reference" "L29" (id 0) (at 357.632 63.5 0))
@@
     (pin "9")
   )
-  (symbol (lib_id "sa800u-baseboard-hw:Si7223DN") (at 109.855 72.39 270) (mirror x) (unit 1)
+  (symbol (lib_name "Si7223DN_2") (lib_id "sa800u-baseboard-hw:Si7223DN") (at 109.855 72.39 270) (mirror x) (unit 1)
     (in_bom yes) (on_board yes) (fields_autoplaced)
     (property "Reference" "Q9" (id 0) (at 118.11 64.1349 90)
@@
     (pin "8")
   )
-  (symbol (lib_id "sa800u-baseboard-hw:Si7223DN") (at 135.255 114.3 270) (mirror x) (unit 1)
+  (symbol (lib_name "Si7223DN_1") (lib_id "sa800u-baseboard-hw:Si7223DN") (at 135.255 114.3 270) (mirror x) (unit 1)
     (in_bom yes) (on_board yes) (fields_autoplaced)
     (property "Reference" "Q12" (id 0) (at 143.51 106.0449 90)
