File: som.kicad_sch (KiCad schematic)
At the start: 43 parts, among them M1 SA800U-WF-mechanical_model, SW1 CVS-02B, U11 SA800U-WF

Commit message: Introduce component standardization
Parts:
- BAT1: value MS621FE-FL11E -> Battery_Holder_MS621FE-FL11E; symbol sa800u-baseboard-hw:MS621FE-FL11E -> sa800u-baseboard-hw:Battery_Holder_MS621FE-FL11E; Author (none) -> Antmicro; License (none) -> Apache-2.0
- C100, C101, C99: footprint sa800u-baseboard-hw-footprints:0805-cap -> sa800u-baseboard-hw-footprints:C_0805_2012Metric; Author (none) -> Antmicro; License (none) -> Apache-2.0; Manufacturer MURATA -> Murata
- C102: footprint sa800u-baseboard-hw-footprints:0402-cap -> sa800u-baseboard-hw-footprints:C_0402_1005Metric; Author (none) -> Antmicro; Dielectric (none) -> X5R; License (none) -> Apache-2.0; MPN 0402X104K6R3CT -> GRM155R61H104KE14D; Manufacturer Walsin -> Murata; Voltage (none) -> 50V
- C103: footprint sa800u-baseboard-hw-footprints:0402-cap -> sa800u-baseboard-hw-footprints:C_0402_1005Metric; Author (none) -> Antmicro; License (none) -> Apache-2.0; Manufacturer MULTICOMP -> Multicomp
- C104: footprint sa800u-baseboard-hw-footprints:0402-cap -> sa800u-baseboard-hw-footprints:C_0402_1005Metric; Author (none) -> Antmicro; Dielectric (none) -> C0G; License (none) -> Apache-2.0; MPN MC0402N100D500CT -> GCM1555C1H100GA16D; Manufacturer MULTICOMP -> Murata; Voltage (none) -> 50V
- D13: footprint sa800u-baseboard-hw-footprints:STS321045B502 -> sa800u-baseboard-hw-footprints:SOD-323; Author (none) -> Antmicro; License (none) -> Apache-2.0
- D14, D15, D16: renamed from D?; value (none) -> KP-1608EC; footprint (none) -> sa800u-baseboard-hw-footprints:LED_0603_1608Metric_G; symbol sa800u-baseboard-hw:KP-1608EC -> sa800u-baseboard-hw:LED_G_0603_KP-1608ZGC; Author (none) -> Antmicro; License (none) -> Apache-2.0; MPN KP-1608EC -> KP-1608ZGC; Manufacturer KINGBRIGHT -> Kingbright
- D17, D18, D19, D20: footprint sa800u-baseboard-hw-footprints:RESC0603X26N -> sa800u-baseboard-hw-footprints:D_0201_0603Metric; Author (none) -> Antmicro; License (none) -> Apache-2.0
- D38: Author (none) -> Antmicro; License (none) -> Apache-2.0
- M1: Author (none) -> Antmicro; DNP (none) -> DNP; License (none) -> Apache-2.0
- Q5, Q6, Q7: renamed from Q?; value (none) -> BSS138PW; footprint (none) -> sa800u-baseboard-hw-footprints:SC70-3; symbol sa800u-baseboard-hw:BSS138APW -> sa800u-baseboard-hw:BSS138PW; Author (none) -> Antmicro; License (none) -> Apache-2.0; Manufacturer ON Semiconductor -> Nexperia
- R175, R77, R78, R79: renamed from R?; value (none) -> R_10k_0402; footprint (none) -> sa800u-baseboard-hw-footprints:R_0402_1005Metric; Author (none) -> Antmicro; License (none) -> Apache-2.0; MPN CRCW040210K0FKEDHP -> CR0402-FX-1002GLF; Manufacturer VISHAY -> Bourns; Tolerance (none) -> 1%
- R176, R177, R178, R179: footprint sa800u-baseboard-hw-footprints:0402-res -> sa800u-baseboard-hw-footprints:R_0402_1005Metric; Author (none) -> Antmicro; Current (none) -> 1A; License (none) -> Apache-2.0; Manufacturer PANASONIC -> Panasonic
- R69, R73, R74, R75, R76: footprint sa800u-baseboard-hw-footprints:0402-res -> sa800u-baseboard-hw-footprints:R_0402_1005Metric; Author (none) -> Antmicro; License (none) -> Apache-2.0; Manufacturer BOURNS -> Bourns; Tolerance (none) -> 1%
- R70: footprint sa800u-baseboard-hw-footprints:0402-res -> sa800u-baseboard-hw-footprints:R_0402_1005Metric; Author (none) -> Antmicro; License (none) -> Apache-2.0; MPN MCMR04X4702FTL -> CR0402-FX-4702GLF; Manufacturer MULTICOMP -> Bourns; Tolerance (none) -> 1%
- R71, R72: renamed from R?; value (none) -> R_4k7_0402; footprint (none) -> sa800u-baseboard-hw-footprints:R_0402_1005Metric; Author (none) -> Antmicro; License (none) -> Apache-2.0; MPN MCS04020C4701FE000 -> CR0402-FX-4701GLF; Manufacturer VISHAY -> Bourns; Tolerance (none) -> 1%
- S1, S2, S3, S4: value KMR2 -> SW_SPST_KMR211NGLFS; symbol sa800u-baseboard-hw:KMR2 -> sa800u-baseboard-hw:SW_SPST_KMR211NGLFS; Author (none) -> Antmicro; License (none) -> Apache-2.0; Manufacturer C&K Components -> C&K
- SW1: value CVS-02B -> SW_CVS-02B; symbol sa800u-baseboard-hw:CVS-02B -> sa800u-baseboard-hw:SW_CVS-02B; Author (none) -> Antmicro; License (none) -> Apache-2.0; Manufacturer Nidec Copal -> Nidec
- TP112: renamed from TP?; value (none) -> TP_0.75mm_SMD; footprint (none) -> sa800u-baseboard-hw-footprints:TP_SMD_0.75mm; symbol sa800u-baseboard-hw:TP -> sa800u-baseboard-hw:TP_0.75mm_SMD; Author (none) -> Antmicro; License (none) -> Apache-2.0
- U11: Author (none) -> Antmicro; License (none) -> Apache-2.0; Manufacturer QUECTEL -> Quectel
Connections:
- net GND: now also D13.K (2), SW1.SH; no longer D13.2, U11.1_169 (GND22), U11.1_170 (GND40), U11.2_169 (GND17), U11.2_170 (GND18)
- net VBAT_SOM: now also D13.A (1); no longer D13.1
Other:
- moved on the sheet: C100, C101, C102, C103, C104, C99, M1, R175, R176, R177, R178, R179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

Commit message: Add OHP assets
Parts:
- removed M1: SA800U-WF-mechanical_model, sa800u-baseboard-hw-footprints:SA800U-WF_mechanical_model, symbol sa800u-baseboard-hw:SA800U-WF-mechanical_model
- removed U11: SA800U-WF, sa800u-baseboard-hw-footprints:SA800U-WF, symbol sa800u-baseboard-hw:SA800U-WF
- added A1: SA800U-WF, sa800u-baseboard-hw-footprints:SA800U-WF, symbol sa800u-baseboard-hw:SA800U-WF
- added U11: Receptacle_SA800U-WF, sa800u-baseboard-hw-footprints:Receptacle_SA800U-WF, symbol sa800u-baseboard-hw:Receptacle_SA800U-WF
Connections:
- net 1V2_SYS_EN: now also U11.2_132 (GPIO_128)
- net 3V3_SYS_EN: now also U11.2_134 (GPIO_135)
- net ACCL_INT: now also U11.1_139 (ACCEL_INT)
- net AUTO_ON_N: now also U11.1_134 (CBL_PWR_N)
- net BOOT: now also U11.2_136 (GPIO_129)
- net CAM0_AFVDD_EN: now also U11.1_86 (SDC4_CLK)
- net CAM0_AVDD_EN: now also U11.1_102 (CAM0_AVDD_EN)
- net CAM0_DVDD_EN: now also U11.1_132 (CAM0_DVDD_EN)
- net CAM0_MCLK: now also U11.1_91 (CAM0_MCLK)
- net CAM0_PWDN: now also U11.1_114 (CAM0_PWDN)
- net CAM0_RST: now also U11.1_100 (CAM0_RST)
- net CAM1_AFVDD_EN: now also U11.1_88 (SDC4_DATA2)
- net CAM1_AVDD_EN: now also U11.1_98 (CAM1_AVDD_EN)
- net CAM1_DVDD_EN: now also U11.1_130 (CAM1_DVDD_EN)
- net CAM1_MCLK: now also U11.1_95 (CAM1_MCLK)
- net CAM1_PWDN: now also U11.1_120 (CAM1_PWDN)
- net CAM1_RST: now also U11.1_96 (CAM1_RST)
- net CAM3_MCLK: now also U11.1_103 (CAM3_MCLK)
- net CAM3_RST: now also U11.1_126 (CAM3_RST)
- net CAM3_TRIGGER_IN: now also U11.2_95 (SPI11_MOSI)
- net CAM3_TRIGGER_OUT: now also U11.1_128 (CAM3_DVDD_EN)
- net CAM3_VCC_EN: now also U11.1_108 (CAM3_AVDD_EN)
- net CCI0_I2C_SCL: now also U11.1_142 (CCI0_I2C_SCL)
- net CCI0_I2C_SDA: now also U11.1_144 (CCI0_I2C_SDA)
- net CCI1_I2C_SCL: now also U11.1_148 (CCI1_I2C_SCL)
- net CCI1_I2C_SDA: now also U11.1_146 (CCI1_I2C_SDA)
- net CODEC_INT1: now also U11.2_91 (CODEC_INT1)
- net CODEC_INT2: now also U11.2_93 (CODEC_INT2)
- net CODEC_SPI_MISO: now also U11.2_89 (CODEC_SPI_MISO)
- net CSI0_CLK_N: now also U11.1_30 (CSI0_CLK_N)
- net CSI0_CLK_P: now also U11.1_28 (CSI0_CLK_P)
- net CSI0_LN0_N: now also U11.1_22 (CSI0_LN0_N)
- net CSI0_LN0_P: now also U11.1_24 (CSI0_LN0_P)
- net CSI0_LN1_N: now also U11.1_16 (CSI0_LN1_N)
- net CSI0_LN1_P: now also U11.1_18 (CSI0_LN1_P)
- net CSI0_LN2_N: now also U11.1_10 (CSI0_LN2_N)
- net CSI0_LN2_P: now also U11.1_12 (CSI0_LN2_P)
- net CSI0_LN3_N: now also U11.1_6 (CSI0_LN3_N)
- net CSI0_LN3_P: now also U11.1_4 (CSI0_LN3_P)
- net CSI1_CLK_N: now also U11.1_58 (CSI1_CLK_N)
- net CSI1_CLK_P: now also U11.1_60 (CSI1_CLK_P)
- net CSI1_LN0_N: now also U11.1_52 (CSI1_LN0_N)
- net CSI1_LN0_P: now also U11.1_54 (CSI1_LN0_P)
- net CSI1_LN1_N: now also U11.1_46 (CSI1_LN1_N)
- net CSI1_LN1_P: now also U11.1_48 (CSI1_LN1_P)
- net CSI1_LN2_N: now also U11.1_42 (CSI1_LN2_N)
- net CSI1_LN2_P: now also U11.1_40 (CSI1_LN2_P)
- net CSI1_LN3_N: now also U11.1_34 (CSI1_LN3_N)
- net CSI1_LN3_P: now also U11.1_36 (CSI1_LN3_P)
- net CSI2_CLK_N: now also U11.1_63 (CSI2_CLK_N)
- net CSI2_CLK_P: now also U11.1_61 (CSI2_CLK_P)
- net CSI2_LN0_N: now also U11.1_67 (CSI2_LN0_N)
- net CSI2_LN0_P: now also U11.1_69 (CSI2_LN0_P)
- net CSI2_LN1_N: now also U11.1_66 (CSI2_LN1_N)
- net CSI2_LN1_P: now also U11.1_64 (CSI2_LN1_P)
- net CSI2_LN2_N: now also U11.1_72 (CSI2_LN2_N)
- net CSI2_LN2_P: now also U11.1_70 (CSI2_LN2_P)
- net CSI2_LN3_N: now also U11.1_78 (CSI2_LN3_N)
- net CSI2_LN3_P: now also U11.1_76 (CSI2_LN3_P)
- net CSI3_CLK_N: now also U11.1_85 (CSI3_CLK_N)
- net CSI3_CLK_P: now also U11.1_87 (CSI3_CLK_P)
- net CSI3_LN0_N: now also U11.1_81 (CSI3_LN0_N)
- net CSI3_LN0_P: now also U11.1_79 (CSI3_LN0_P)
- net CSI3_LN1_N: now also U11.1_73 (CSI3_LN1_N)
- net CSI3_LN1_P: now also U11.1_75 (CSI3_LN1_P)
- net DBG_RXD: now also U11.2_135 (DBG_RXD)
- net DBG_TXD: now also U11.2_137 (DBG_TXD)
- net DSI0_CLK_N: now also U11.2_26 (DSI0_CLK_N)
- net DSI0_CLK_P: now also U11.2_28 (DSI0_CLK_P)
- net DSI0_LN0_N: now also U11.2_38 (DSI0_LN0_N)
- net DSI0_LN0_P: now also U11.2_40 (DSI0_LN0_P)
- net DSI0_LN1_N: now also U11.2_32 (DSI0_LN1_N)
- net DSI0_LN1_P: now also U11.2_34 (DSI0_LN1_P)
- net DSI0_LN2_N: now also U11.2_20 (DSI0_LN2_N)
- net DSI0_LN2_P: now also U11.2_22 (DSI0_LN2_P)
- net DSI0_LN3_N: now also U11.2_14 (DSI0_LN3_N)
- net DSI0_LN3_P: now also U11.2_16 (DSI0_LN3_P)
- net DSI1_CLK_N: now also U11.2_21 (DSI1_CLK_N)
- net DSI1_CLK_P: now also U11.2_19 (DSI1_CLK_P)
- net DSI1_LN0_N: now also U11.2_13 (DSI1_LN0_N)
- net DSI1_LN0_P: now also U11.2_15 (DSI1_LN0_P)
- net DSI1_LN1_N: now also U11.2_37 (DSI1_LN1_N)
- net DSI1_LN1_P: now also U11.2_39 (DSI1_LN1_P)
- net DSI1_LN2_N: now also U11.2_27 (DSI1_LN2_N)
- net DSI1_LN2_P: now also U11.2_25 (DSI1_LN2_P)
- net DSI1_LN3_N: now also U11.2_31 (DSI1_LN3_N)
- net DSI1_LN3_P: now also U11.2_33 (DSI1_LN3_P)
- net EDP_AUX_N: now also U11.2_131 (EDP_AUX_N)
- net EDP_AUX_P: now also U11.2_129 (EDP_AUX_P)
- net ETH_3V3_EN: now also U11.2_97 (SPI11_MISO)
- net GND: now also U11.1_101 (GND), U11.1_105 (GND), U11.1_113 (GND), U11.1_119 (GND), U11.1_125 (GND), U11.1_13 (GND), U11.1_131 (GND), U11.1_14 (GND), U11.1_156 (GND), U11.1_157 (GND), U11.1_158 (GND), U11.1_19 (GND), U11.1_2 (GND), U11.1_20 (GND), U11.1_25 (GND), U11.1_26 (GND), U11.1_31 (GND), U11.1_32 (GND), U11.1_37 (GND), U11.1_38 (GND), U11.1_41 (GND), U11.1_44 (GND), U11.1_50 (GND), U11.1_56 (GND), U11.1_59 (GND), U11.1_62 (GND), U11.1_65 (GND), U11.1_68 (GND), U11.1_7 (GND), U11.1_71 (GND), U11.1_74 (GND), U11.1_77 (GND), U11.1_8 (GND), U11.1_80 (GND), U11.1_83 (GND), U11.1_89 (GND), U11.1_93 (GND), U11.1_94 (GND), U11.1_97 (GND), U11.2_103 (GND), U11.2_104 (GND), U11.2_109 (GND), U11.2_11 (GND), U11.2_110 (GND), U11.2_115 (GND), U11.2_116 (GND), U11.2_12 (GND), U11.2_121 (GND), U11.2_122 (GND), U11.2_127 (GND), U11.2_155 (GND), U11.2_158 (GND), U11.2_161 (GND), U11.2_167 (GND), U11.2_17 (GND), U11.2_18 (GND), U11.2_23 (GND), U11.2_24 (GND), U11.2_29 (GND), U11.2_30 (GND), U11.2_35 (GND), U11.2_36 (GND), U11.2_41 (GND), U11.2_42 (GND), U11.2_45 (GND), U11.2_53 (GND), U11.2_98 (GND)
- net GYRO_INT: now also U11.1_137 (GYRO_INT)
- net HDMI1_INTO: now also U11.1_92 (SDC4_CMD)
- net HOME_KEY: now also U11.2_145 (HOME_KEY)
- net I2C10_SCL: now also U11.2_75 (I2C10_SCL)
- net I2C10_SDA: now also U11.2_77 (I2C10_SDA)
- net I2C4_SCL: now also U11.2_6 (I2C4_SCL)
- net I2C4_SDA: now also U11.2_4 (I2C4_SDA)
- net I2S1_DATA0: now also U11.2_87 (I2S1_DATA0)
- net I2S1_MCLK: now also U11.2_81 (I2S1_MCLK)
- net I2S1_SCK: now also U11.2_83 (I2S1_SCK)
- net I2S1_WS: now also U11.2_79 (I2S1_WS)
- net I2S2_DATA0: now also U11.2_59 (I2S2_DATA0)
- net I2S2_DATA1: now also U11.2_61 (I2S2_DATA1)
- net I2S2_SCK: now also U11.2_57 (I2S2_SCK)
- net I2S2_WS: now also U11.2_55 (I2S2_WS)
- net I2S3_DATA0: now also U11.2_69 (I2S3_DATA0)
- net I2S3_SCK: now also U11.2_73 (I2S3_SCK)
- net I2S3_WS: now also U11.2_63 (I2S3_WS)
- net LCM_VDD_EN: now also U11.1_43 (UFS_DET)
- net LDO19A_3V0: now also U11.2_150 (LDO19A_3V0)
- net LT6911_3V3_EN: now also U11.1_106 (CAM2_PWDN)
- net LT6911_RST: now also U11.1_90 (SDC4_DATA3)
- net LT9611_GPIO5: now also U11.2_68 (GPIO_52)
- net LT9611_RST: now also U11.2_70 (GPIO_50)
- net LVS1A_1V8: now also U11.1_149 (LVS1A_1V8)
- net LVS2A_1V8: now also U11.2_148 (LVS2A_1V8)
- net MAG_DRDY_INT: now also U11.1_135 (MAG_DRDY_INT)
- net MAG_INT: now also U11.1_133 (MAG_INT)
- net PCIE0_CLKREQ_N: now also U11.1_5 (PCIE0_CLKREQ_N)
- net PCIE0_REFCLK_N: now also U11.1_17 (PCIE0_REFCLK_M)
- net PCIE0_REFCLK_P: now also U11.1_15 (PCIE0_REFCLK_P)
- net PCIE0_RST_N: now also U11.1_1 (PCIE0_RST_N)
- net PCIE0_RX_N: now also U11.1_23 (PCIE0_RX_M)
- net PCIE0_RX_P: now also U11.1_21 (PCIE0_RX_P)
- net PCIE0_TX_N: now also U11.1_9 (PCIE0_TX_M)
- net PCIE0_TX_P: now also U11.1_11 (PCIE0_TX_P)
- net PCIE0_WAKE_N: now also U11.1_3 (PCIE0_WAKE_N)
- net PCIE1_CLKREQ_N: now also U11.1_109 (PCIE1_CLKREQ_N)
- net PCIE1_REFCLK_N: now also U11.1_123 (PCIE1_REFCLK_M)
- net PCIE1_REFCLK_P: now also U11.1_121 (PCIE1_REFCLK_P)
- net PCIE1_RST_N: now also U11.1_107 (PCIE1_RST_N)
- net PCIE1_RX_N: now also U11.1_117 (PCIE1_RX_M)
- net PCIE1_RX_P: now also U11.1_115 (PCIE1_RX_P)
- net PCIE1_TX_N: now also U11.1_127 (PCIE1_TX_M)
- net PCIE1_TX_P: now also U11.1_129 (PCIE1_TX_P)
- net PCIE1_WAKE_N: now also U11.1_111 (PCIE1_WAKE_N)
- net PWRKEY: now also U11.2_5 (PWRKEY)
- net PWR_OFF: now also U11.1_124 (CAM2_RST)
- net RESET_USBHUB: now also U11.1_110 (CAM2_DVDD_EN)
- net SBU_SW_OE: now also U11.2_1 (SBU_SW_OE)
- net SBU_SW_SEL: now also U11.2_3 (SBU_SW_SEL)
- net SD_CLK: now also U11.1_45 (SD_CLK)
- net SD_CMD: now also U11.1_47 (SD_CMD)
- net SD_DATA0: now also U11.1_51 (SD_DATA0)
- net SD_DATA1: now also U11.1_53 (SD_DATA1)
- net SD_DATA2: now also U11.1_57 (SD_DATA2)
- net SD_DATA3: now also U11.1_55 (SD_DATA3)
- net SD_DET: now also U11.1_49 (SD_DET)
- net SD_LDO21A: now also U11.1_151 (SD_LDO21A), U11.1_153 (SD_LDO21A), U11.1_155 (SD_LDO21A)
- net SLIMBUS_CLK: now also U11.2_51 (SLIMBUS_CLK)
- net SLIMBUS_DATA0: now also U11.2_47 (SLIMBUS_DATA0)
- net SLIMBUS_DATA1: now also U11.2_49 (SLIMBUS_DATA1)
- net SSC_I2C1_SCL: now also U11.2_10 (SSC_I2C1_SCL)
- net SSC_I2C1_SDA: now also U11.2_8 (SSC_I2C1_SDA)
- net STUSB4500_AB_SIDE: now also U11.2_66 (GPIO_44)
- net STUSB4500_ALERT: now also U11.2_64 (GPIO_42)
- net STUSB4500_ATTACH: now also U11.2_74 (GPIO_122)
- net STUSB4500_GPIO: now also U11.2_72 (GPIO_134)
- net TP_I2C_SCL: now also U11.2_44 (TP_I2C_SCL)
- net TP_I2C_SDA: now also U11.2_46 (TP_I2C_SDA)
- net TP_INT: now also U11.2_48 (TP_INT)
- net TP_RST: now also U11.2_50 (TP_RST)
- net USB1_D_N: now also U11.2_117 (USB1_DM)
- net USB1_D_P: now also U11.2_119 (USB1_DP)
- net USB1_SS_RX0_N: now also U11.2_118 (USB1_SS1_RX_M)
- net USB1_SS_RX0_P: now also U11.2_120 (USB1_SS1_RX_P)
- net USB1_SS_RX1_N: now also U11.2_114 (USB1_SS2_RX_M)
- net USB1_SS_RX1_P: now also U11.2_112 (USB1_SS2_RX_P)
- net USB1_SS_TX0_N: now also U11.2_123 (USB1_SS1_TX_M)
- net USB1_SS_TX0_P: now also U11.2_125 (USB1_SS1_TX_P)
- net USB1_SS_TX1_N: now also U11.2_111 (USB1_SS2_TX_M)
- net USB1_SS_TX1_P: now also U11.2_113 (USB1_SS2_TX_P)
- net USB2C_HS_D_N: now also U11.2_107 (USB2_DM)
- net USB2C_HS_D_P: now also U11.2_105 (USB2_DP)
- net USB2_EN: now also U11.2_54 (SPI2_CS)
- net USB2_FAULT: now also U11.1_118 (CAM2_STROBE)
- net USB2_SINK: now also U11.2_80 (SPI0_CS)
- net USB2_SS_RX_N: now also U11.2_100 (USB2_SS_RX_M)
- net USB2_SS_RX_P: now also U11.2_102 (USB2_SS_RX_P)
- net USB2_SS_TX_N: now also U11.2_108 (USB2_SS_TX_M)
- net USB2_SS_TX_P: now also U11.2_106 (USB2_SS_TX_P)
- net USB_BOOT: now also U11.2_130 (USB_BOOT)
- net USB_CC1: now also U11.2_141 (USB_CC1)
- net USB_CC2: now also U11.2_139 (USB_CC2)
- net USB_PD_DISABLE: now also U11.2_76 (GPIO_124)
- net USB_VBUS: now also U11.2_160 (USB_VBUS), U11.2_162 (USB_VBUS), U11.2_164 (USB_VBUS), U11.2_166 (USB_VBUS), U11.2_168 (USB_VBUS)
- net USER_LED: now also U11.2_2 (GPIO_25)
- net VBAT_SOM: now also U11.1_159 (VBAT), U11.1_160 (VBAT), U11.1_161 (VBAT), U11.1_162 (VBAT), U11.1_163 (VBAT), U11.1_164 (VBAT), U11.1_165 (VBAT), U11.1_166 (VBAT), U11.1_167 (VBAT), U11.1_168 (VBAT)
- net VOL_DOWN: now also U11.2_7 (VOL_DOWN)
- net VOL_UP: now also U11.2_9 (VOL_UP_)
- net VREG_S4A_1V8: now also U11.2_124 (VREG_S4A_1V8), U11.2_126 (VREG_S4A_1V8), U11.2_128 (VREG_S4A_1V8)
- net VRTC: now also U11.2_133 (VRTC)
- net WCD_CLK: now also U11.2_43 (WCD_CLK)
- net at R70.1: now also U11.2_143 (BAT_THERM)
- net at R176.1: now also U11.2_157 (CS_P)
- net at R177.1: now also U11.2_159 (CS_M)
- net at R178.1: now also U11.2_163 (BAT_P)
- net at R179.1: now also U11.2_165 (BAT_M)
- no-connect marks 52 -> 111
Other:
- note added: "SoM Module"
- company: (none) -> Antmicro Ltd.
